File: example/БМРЦ/БМРЦ.kicad_sch (KiCad schematic)
At the start: 56 parts

Commit message: Канализация вынесена в отдельный файл
Parts:
- added БШ1: ~, symbol SCB:Ящик_батарейный
- added РШ1: ~, symbol SCB:Шкаф_релейный
- added ЭЦ1: ~, symbol SCB:Пост_ЭЦ
- renumbered ~C9 to C1, ~C7 to C2, ~C11 to C3, Входной2 to Входной1, Входной111 to Выходной1, Входной11 to Выходной2, Входной1 to Выходной3, Входной11 to Выходной4, И11 to Изостык1, И11 to Изостык10, И1111 to Изостык11, И111 to Изостык12, И1111 to Изостык13, И1111 to Изостык14, И111111 to Изостык15, И111 to Изостык16, И11111 to Изостык17, И111111 to Изостык18, И11111 to Изостык19, И11 to Изостык2, И111111 to Изостык20, И111111 to Изостык21, И111111 to Изостык22, И11111 to Изостык23, И111111 to Изостык24, И1 to Изостык3, И1 to Изостык4, И11 to Изостык5, И11 to Изостык6, И11 to Изостык7, И11111 to Изостык8, И111 to Изостык9, Маневровый1111 to Маневровый10, Маневровый111 to Маневровый11, Маневровый1111 to Маневровый12, Маневровый1111 to Маневровый13, Маневровый11 to Маневровый14, Маневровый11111 to Маневровый15, Маневровый11111 to Маневровый16, Маневровый1 to Маневровый2, Маневровый11 to Маневровый2, Маневровый1 to Маневровый3, Маневровый11111 to Маневровый4, Маневровый1 to Маневровый4, Маневровый1 to Маневровый5, Маневровый11 to Маневровый5, Маневровый1111 to Маневровый6, Маневровый111 to Маневровый7, Маневровый11 to Маневровый8, Маневровый1111 to Маневровый9, ~C1 to Стрелка1, ~C4 to Стрелка2, ~C3 to Стрелка3, ~C6 to Стрелка4, ~C5 to Стрелка5, ~C8 to Стрелка6, ~C2 to Стрелка7, ~C10 to Стрелка8
Connections:
- net at Изостык16. (привязка), Стрелка7.1: now also C1.3; no longer C1.1
- net at Изостык20. (привязка): now also C1.2; no longer C1.1
- net at Изостык22. (привязка): now also C2.2; no longer C2.1
- net at Изостык23. (привязка): now also C3.2; no longer C3.1
- net at Изостык24. (привязка): now also C3.3; no longer C3.1
- net at Изостык21. (привязка): now also C2.3; no longer C2.1
- new net: Изостык11. (привязка), Стрелка5.1, Стрелка6.1
- new net: Изостык14. (привязка), Стрелка6.1, Стрелка7.1
- new net: Изостык9. (привязка), Стрелка3.1, Стрелка5.1
- new net: Изостык12. (привязка), Стрелка4.1, Стрелка6.1
- new net: Изостык7. (привязка), Стрелка3.1, Стрелка4.1
- new net: Изостык8. (привязка), Стрелка1.1, Стрелка2.1
- new net: Изостык10. (привязка), Стрелка2.1, Стрелка8.1
- new net: Изостык17. (привязка), Стрелка8.1
- now unconnected: C2.1
Other:
- added sheet Канализация_тягового_тока (канализация.kicad_sch)
- note removed: "БШ"
- note removed: "Пост ЭЦ"
- note removed: "РШ"

Commit message: Обновлены РШ и БШ
Parts:
- БШ1: Ордината (none) -> (720); Тип (none) -> ШМБ-У
- РШ1: Ордината (none) -> (720); Тип (none) -> ШРУ-М
Connections:
- new net: Изостык11. (привязка), Стрелка5.1, Стрелка6.1
- new net: Изостык14. (привязка), Стрелка6.1, Стрелка7.1
- new net: Изостык9. (привязка), Стрелка3.1, Стрелка5.1
- new net: Изостык12. (привязка), Стрелка4.1, Стрелка6.1
- new net: Изостык7. (привязка), Стрелка3.1, Стрелка4.1
- new net: Изостык8. (привязка), Стрелка1.1, Стрелка2.1
- new net: Изостык10. (привязка), Стрелка2.1, Стрелка8.1
Changed lines of the file:
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@@
 		)
 		(property "Шкаф" "РШ"
-			(at 50 226 0)
-			(do_not_autoplace yes)
-			(effects
-				(font
-					(size 3.5 3.5)
-				)
+			(at 50 225 0)
+			(do_not_autoplace yes)
+			(effects
+				(font
+					(size 2.5 2.5)
+				)
+			)
+		)
+		(property "Ордината" "(720)"
+			(at 50 211 0)
+			(effects
+				(font
+					(size 2.5 2.5)
+				)
+				(hide yes)
+			)
+		)
+		(property "Тип" "ШРУ-М"
+			(at 50 215 0)
+			(effects
+				(font
+					(size 2.5 2.5)
+				)
+				(hide yes)
 			)
 		)
@@
 		)
 		(property "Шкаф" "БШ"
-			(at 40 226 0)
-			(do_not_autoplace yes)
-			(effects
-				(font
-					(size 3.5 3.5)
-				)
-			)
-		)
+			(at 40 225 0)
+			(do_not_autoplace yes)
+			(effects
+				(font
+					(size 2.5 2.5)
+				)
+			)
+		)
+		(property "Ордината" "(720)"
+			(at 40 215 0)
+			(effects
+				(font
+					(size 2.5 2.5)
+				)
+				(hide yes)
+			)
+		)
+		(property "Тип" "ШМБ-У"
+			(at 40 210 0)
+			(effects
+				(font
+					(size 2.5 2.5)
+				)
+				(hide yes)
+			)
+		)

Commit message: Упрощены УГО ДТ для фазочувствительных РЦ, скрыты точки для двойных СС
Parts:
- Входной1: now left out of the parts list
Connections:
- new net: Изостык11. (привязка), Стрелка5.1, Стрелка6.1
- new net: Изостык14. (привязка), Стрелка6.1, Стрелка7.1
- new net: Изостык9. (привязка), Стрелка3.1, Стрелка5.1
- new net: Изостык12. (привязка), Стрелка4.1, Стрелка6.1
- new net: Изостык7. (привязка), Стрелка3.1, Стрелка4.1
- new net: Изостык8. (привязка), Стрелка1.1, Стрелка2.1
- new net: Изостык10. (привязка), Стрелка2.1, Стрелка8.1
Changed lines of the file:
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@@
 	)
 	(symbol
+		(lib_name "SCB:Изостык")
 		(lib_id "SCB:Изостык")
 		(at 330 160 0)
@@
 	)
 	(symbol
+		(lib_name "SCB:Изостык")
 		(lib_id "SCB:Изостык")
 		(at 208 190 0)
@@
 	)
 	(symbol
+		(lib_name "SCB:Стрелка_спаренная")
 		(lib_id "SCB:Стрелка_спаренная")
 		(at 284 175 0)
@@
 	)
 	(symbol
+		(lib_name "SCB:Изостык")
 		(lib_id "SCB:Изостык")
 		(at 157 175 0)
@@
 	)
 	(symbol
+		(lib_name "SCB:Изостык")
 		(lib_id "SCB:Изостык")
 		(at 334 130 0)
@@
 	)
 	(symbol
+		(lib_name "SCB:Изостык")
 		(lib_id "SCB:Изостык")
 		(at 226 175 0)
@@
 	)
 	(symbol
+		(lib_name "SCB:Изостык")
 		(lib_id "SCB:Изостык")
 		(at 350 220 0)
@@
 	)
 	(symbol
+		(lib_name "SCB:Изостык")
 		(lib_id "SCB:Изостык")
 		(at 86 160 0)
@@
 	)
 	(symbol
+		(lib_name "SCB:Изостык")
 		(lib_id "SCB:Изостык")
 		(at 279 175 0)
@@
 		(mirror y)
 		(unit 2)
-		(exclude_from_sim no)
-		(in_bom yes)
-		(on_board yes)
+		(exclude_from_sim yes)
+		(in_bom no)
+		(on_board no)
 		(dnp no)
 		(fields_autoplaced yes)
@@
 	)
 	(symbol
+		(lib_name "SCB:Стрелка_спаренная_15")
 		(lib_id "SCB:Стрелка_спаренная_15")
 		(at 148 175 0)
@@
 	)
 	(symbol
+		(lib_name "SCB:Изостык")
 		(lib_id "SCB:Изостык")
 		(at 313 175 0)
@@
 	)
 	(symbol
+		(lib_name "SCB:Стрелка_спаренная_15")
 		(lib_id "SCB:Стрелка_спаренная_15")
 		(at 127 205 0)
@@
 	)
 	(symbol
+		(lib_name "SCB:Изостык")
 		(lib_id "SCB:Изостык")
 		(at 74 190 0)
@@
 	)
 	(symbol
+		(lib_name "SCB:Изостык")
 		(lib_id "SCB:Изостык")
 		(at 249 160 0)
@@
 	)
 	(symbol
+		(lib_name "SCB:Изостык")
 		(lib_id "SCB:Изостык")
 		(at 132 190 0)
@@
 	)
 	(symbol
+		(lib_name "SCB:Изостык")
 		(lib_id "SCB:Изостык")
 		(at 167 205 0)
@@
 	)
 	(symbol
+		(lib_name "SCB:Изостык")
 		(lib_id "SCB:Изостык")
 		(at 350 205 0)
@@
 	)
 	(symbol
+		(lib_name "SCB:Изостык")
 		(lib_id "SCB:Изостык")
 		(at 40 190 0)
@@
 	)
 	(symbol
+		(lib_name "SCB:Изостык")
 		(lib_id "SCB:Изостык")
 		(at 40 205 0)
@@
 	)
 	(symbol
+		(lib_name "SCB:Стрелка_спаренная_15")
 		(lib_id "SCB:Стрелка_спаренная_15")
 		(at 294 205 0)
@@
 	)
 	(symbol
+		(lib_name "SCB:Изостык")
 		(lib_id "SCB:Изостык")
 		(at 375 160 0)
@@
 	)
 	(symbol
+		(lib_name "SCB:Изостык")
 		(lib_id "SCB:Изостык")
 		(at 82 175 0)
@@
 	)
 	(symbol
+		(lib_name "SCB:Стрелка_спаренная_15")
 		(lib_id "SCB:Стрелка_спаренная_15")
 		(at 190 175 0)
@@
 	)
 	(symbol
+		(lib_name "SCB:Стрелка_спаренная_15")
 		(lib_id "SCB:Стрелка_спаренная_15")
 		(at 79 190 0)
@@
 	)
 	(symbol
+		(lib_name "SCB:Изостык")
 		(lib_id "SCB:Изостык")
 		(at 123 205 0)
@@
 	)
 	(symbol
+		(lib_name "SCB:Изостык")
 		(lib_id "SCB:Изостык")
 		(at 307 205 0)
@@
 		(at 40 210 180)
 		(unit 1)
-		(exclude_from_sim no)
-		(in_bom yes)
-		(on_board yes)
+		(exclude_from_sim yes)
+		(in_bom no)
+		(on_board no)
 		(dnp no)
 		(fields_autoplaced yes)
@@
 	)
 	(symbol
+		(lib_name "SCB:Изостык")
 		(lib_id "SCB:Изостык")
 		(at 128 160 0)
@@
 	)
 	(symbol
+		(lib_name "SCB:Изостык")
 		(lib_id "SCB:Изостык")
 		(at 286 190 0)
@@
 	)
 	(symbol
+		(lib_name "SCB:Изостык")
 		(lib_id "SCB:Изостык")
 		(at 290 160 0)
