File: example/БМРЦ/двухниточный.kicad_sch (KiCad schematic)
At the start: 129 parts

Commit message: Канализация вынесена в отдельный файл
Parts:
- ДТ1: renamed from ДТ8; Кодирование1 (none) -> К; Кодирование2 (none) -> К
- ДТ10: renamed from ДТ9; Кодирование1 (none) -> К; Кодирование2 (none) -> К; Секция2 2П -> 5
- ДТ11: renamed from ДТ6; Кодирование1 (none) -> К; Кодирование2 (none) -> К; Секция1 1-9 -> 29; Секция2 2П -> 13-17
- ДТ12: renamed from ДТ4; Кодирование1 (none) -> К; Кодирование2 (none) -> К; Секция1 1-9 -> 29
- ДТ13: renamed from ДТ7; Кодирование1 (none) -> К; Кодирование2 (none) -> К; Секция2 2П -> 29
- ДТ14, ДТ2: renamed from ДТ10; Кодирование1 (none) -> К; Кодирование2 (none) -> К
- ДТ15: renamed from ДТ2; Кодирование1 (none) -> К; Кодирование2 (none) -> К; Секция2 2П -> 29А
- ДТ16, ДТ22: renamed from ДТ12; Кодирование1 (none) -> К; Кодирование2 (none) -> К
- ДТ17: renamed from ДТ7; Кодирование1 (none) -> К; Кодирование2 (none) -> К; Секция2 2П -> 31
- ДТ18: renamed from ДТ5; Кодирование1 (none) -> К; Кодирование2 (none) -> К
- ДТ19: renamed from ДТ1; Кодирование1 (none) -> К; Кодирование2 (none) -> К; Секция2 2П -> 29Б
- ДТ20: renamed from ДТ2; Кодирование1 (none) -> К; Кодирование2 (none) -> К; Секция2 2П -> 37Б
- ДТ21: renamed from ДТ4; Кодирование1 (none) -> К; Кодирование2 (none) -> К; Секция2 2П -> 37А
- ДТ23: renamed from ДТ13; Кодирование1 (none) -> К; Кодирование2 (none) -> К; Секция2 2П -> 35Б
- ДТ24: renamed from ДТ3; Кодирование1 (none) -> К; Секция М8П -> (none); Секция1 (none) -> М8П
- ДТ3: renamed from ДТ8; Кодирование1 (none) -> К; Кодирование2 (none) -> К; Секция2 2П -> М5П
- ДТ4: renamed from ДТ5; Кодирование1 (none) -> К; Кодирование2 (none) -> К; Секция2 2П -> М5П
- ДТ5, ДТ9: renamed from ДТ11; Кодирование1 (none) -> К; Кодирование2 (none) -> К
- ДТ6: renamed from ДТ9; Кодирование1 (none) -> К; Кодирование2 (none) -> К
- ДТ7: renamed from ДТ1; Кодирование1 (none) -> К; Кодирование2 (none) -> К; Секция2 2П -> 5
- ДТ8: renamed from ДТ6; Кодирование1 (none) -> К; Кодирование2 (none) -> К
- ЯП1: renamed from Я9; Секция1 М8П -> 1
- ЯП11-15: renamed from Я10; Секция1 М8П -> 11-15
- ЯП19: renamed from Я2; Секция1 18 -> 19
- ЯП21-25: renamed from Я11; Секция1 М8П -> 21-25
- ЯП23: renamed from Я5; Секция1 18 -> 23
- ЯП27: renamed from Я15; Секция1 М8П -> 27
- ЯП2П: renamed from Я12; Секция1 М8П -> 2П
- ЯП3-7: renamed from Я4; Секция1 18 -> 3-7
- ЯП35: renamed from Я16; Секция1 М8П -> 35
- ЯП37: renamed from Я1; Секция1 18 -> 33; Секция2 2П -> 37
- ЯП4П: renamed from Я6; Секция1 18 -> 4П
- ЯП5: renamed from Я3; Секция1 М8П -> 5
- ЯП9: renamed from Я14; Секция1 М8П -> 9
- ЯПНП: renamed from Я13; Секция1 М8П -> НП
- ЯР1: renamed from Я10; Секция1 М8П -> 1
- ЯР11-15: renamed from Я11; Секция1 М8П -> 11-15
- ЯР13-17: renamed from Я8; Секция1 18 -> 13-17; Секция2 2П -> 3-7
- ЯР19: renamed from Я4; Секция1 18 -> 19
- ЯР1П: renamed from Я16; Секция1 М8П -> 1П
- ЯР21-25: renamed from Я12; Секция1 М8П -> 21-25
- ЯР27: renamed from Я14; Секция1 М8П -> 27
- ЯР31: renamed from Я7; Секция1 18 -> 23; Секция2 2П -> 31
- ЯР33: renamed from Я5; Секция1 18 -> 33
- ЯР35А: renamed from Я15; Секция1 М8П -> 35А
- ЯР3П: renamed from Я17; Секция1 18 -> 3П
- ЯР6П: renamed from Я6; Секция1 18 -> 6П
- ЯР9: renamed from Я13; Секция1 М8П -> 9
- ЯРМ29П: renamed from Я1; Секция1 18 -> М29П
- ЯРМ37П: renamed from Я2; Секция1 18 -> М37П
- ЯРМ5П: renamed from Я3; Секция1 М8П -> М5П
- ЯРНДП: renamed from Я9; Секция1 М8П -> НДП
- renumbered Выходной7 to Выходной5, Выходной8 to Выходной7, Выходной5 to Выходной8, Изостыки4 to Изостыки1, Изостыки5 to Изостыки2, Изостыки1 to Изостыки3, Изостыки8 to Изостыки4, Изостыки6 to Изостыки5, Изостыки2 to Изостыки6, Изостыки9 to Изостыки8, Изостыки3 to Изостыки9, Маневровый32 to Маневровый17, Маневровый28 to Маневровый18, Маневровый23 to Маневровый19, Маневровый35 to Маневровый20, Маневровый31 to Маневровый21, Маневровый21 to Маневровый22, Маневровый26 to Маневровый23, Маневровый29 to Маневровый24, Маневровый34 to Маневровый25, Маневровый33 to Маневровый26, Маневровый24 to Маневровый28, Маневровый30 to Маневровый29, Маневровый22 to Маневровый30, Маневровый36 to Маневровый31, Маневровый25 to Маневровый32, Маневровый4 to Маневровый6, Маневровый6 to Маневровый8, Путь3 to Путь1, Путь4 to Путь2, Путь1 to Путь2, Путь5 to Путь3, Путь2 to Путь4, Путь1 to Путь6, СП12 to СП1, СП2 to СП10, СП15 to СП11, СП3 to СП12, СП16 to СП13, СП9 to СП14, СП10 to СП15, СП18 to СП16, СП4 to СП17, СП19 to СП18, СП5 to СП19, СП1 to СП2, СП11 to СП3, СП6 to СП4, СП17 to СП5, СП7 to СП6, СП13 to СП7, СП14 to СП9, Соединитель12 to Соединитель1, Соединитель14 to Соединитель10, Соединитель4 to Соединитель11, Соединитель1 to Соединитель12, Соединитель16 to Соединитель13, Соединитель11 to Соединитель14, Соединитель8 to Соединитель15, Соединитель18 to Соединитель16, Соединитель19 to Соединитель17, Соединитель5 to Соединитель18, Соединитель2 to Соединитель19, Соединитель3 to Соединитель2, Соединитель9 to Соединитель3, Соединитель17 to Соединитель4, Соединитель6 to Соединитель5, Соединитель10 to Соединитель6, Соединитель15 to Соединитель7, Соединитель7 to Соединитель8, Соединитель13 to Соединитель9, Стрелка15 to Стрелка10, Стрелка20 to Стрелка11, Стрелка19 to Стрелка12, Стрелка18 to Стрелка14, Стрелка11 to Стрелка15, Стрелка9 to Стрелка16, Стрелка16 to Стрелка17, Стрелка14 to Стрелка18, Стрелка12 to Стрелка19, Стрелка10 to Стрелка20, Стрелка17 to Стрелка9, Электротяга4 to Электротяга1, Электротяга1 to Электротяга2, Электротяга2 to Электротяга3, Электротяга3 to Электротяга4
Connections:
- net at ЯП21-25.: now also ДТ10. (П), Соединитель10.2, Стрелка14.2
- net at ЯРМ29П.: now also ДТ19. (П), Электротяга2.2
- net at ЯПНП.: now also ДТ2. (П), ДТ5. (П)
- net at ЯП9.: now also ДТ9. (П), Стрелка11.6
- net at ЯП19.: now also ДТ12. (П), Соединитель11.2, Стрелка15.2
- net at ЯР27.: now also ДТ9. (П), Стрелка14.6
- new net: ДТ23. (П), Путь3. (x2)
- new net: ДТ22. (П), Стрелка15. (x2)
- new net: ДТ16. (П), Стрелка15. (x2)
- new net: ДТ23. (П), Стрелка15. (x2)
- new net: ДТ22. (П), Стрелка15.5, ЯП35.
- new net: ДТ22. (П), Стрелка15.6, ЯП35.
- new net: ДТ21. (П), Путь6. (x2)
- new net: Стрелка13., Стрелка14. (x2)
- new net: ДТ14. (П), Стрелка13. (x2)
- new net: ДТ14. (П), Стрелка13.5, ЯР21-25.
- new net: ДТ14. (П), Стрелка13.6, ЯР21-25.
- new net: Стрелка10., Стрелка10. (x2)
- new net: ДТ4. (П), Стрелка10. (x2)
- new net: ДТ4. (П), Стрелка10.5, ЯП3-7.
- new net: ДТ4. (П), Стрелка10.6, ЯП3-7.
- new net: ДТ1. (П), ДТ3. (П), ЯРНДП. (x2)
- new net: ДТ8. (П), Стрелка10. (x2)
- new net: ДТ10. (П), Стрелка14. (x2)
- new net: ДТ4. (П), Изостыки1.1, Тупик1.1, Электротяга1.1, ЯРМ5П.
- new net: ДТ11. (П), Стрелка17. (x2)
- new net: ДТ13. (П), Стрелка17. (x2)
- new net: ДТ11. (П), Стрелка17.5, ЯП23.
- new net: ДТ11. (П), Стрелка17.6, ЯП23.
- new net: ДТ17. (П), Стрелка18. (x2)
- new net: ДТ17. (П), Путь4. (x2)
- new net: ДТ7. (П), Стрелка9. (x2)
- new net: ДТ24. (П), Стрелка9. (x2)
- new net: ДТ19. (П), Электротяга2.1, ЯРМ29П.
- new net: ДТ2. (П), ДТ5. (П), ЯПНП.
- new net: ДТ11. (П), Стрелка13. (x2)
- new net: Стрелка11., Стрелка13. (x2)
- new net: ДТ14. (П), Путь2. (x2)
- new net: ДТ3. (П), Стрелка9. (x2)
- new net: ДТ6. (П), Стрелка9. (x2)
- new net: ДТ6. (П), Стрелка9.5, ЯР1.
- new net: ДТ6. (П), Стрелка9.6, ЯР1.
- new net: ДТ10. (П), Стрелка12. (x2)
- new net: Стрелка12., Стрелка12. (x2)
- new net: ДТ20. (П), Электротяга3.1, ЯРМ37П.
- new net: ДТ20. (П), Электротяга3.2, ЯРМ37П.
- new net: ДТ22. (П), Путь1. (x2)
- new net: ДТ6. (П), Стрелка12. (x2)
- new net: ДТ6. (П), Стрелка12.5, ЯП11-15.
- new net: ДТ16. (П), Стрелка14. (x2)
- new net: ДТ9. (П), Стрелка11.5, ЯП9.
- new net: ДТ15. (П), Стрелка19.5, ЯР33.
- new net: ДТ15. (П), Стрелка19.6, ЯР33.
- new net: ДТ15. (П), Стрелка19. (x2)
- new net: ДТ7. (П), Стрелка15.5, ЯР19.
- new net: ДТ7. (П), Стрелка15.6, ЯР19.
- new net: ДТ7. (П), Стрелка15. (x2)
- new net: ДТ12. (П), Стрелка15. (x2)
- new net: ДТ9. (П), Стрелка14.5, ЯР27.
- new net: ДТ9. (П), Стрелка11. (x2)
- new net: ДТ5. (П), Стрелка11. (x2)
- new net: ДТ9. (П), Стрелка14. (x2)
- new net: ДТ18. (П), Стрелка19. (x2)
- new net: ДТ8. (П), Стрелка11. (x2)
- new net: ДТ13. (П), Стрелка18. (x2)
- now unconnected: ДТ2. (П), ДТ2. (П), ДТ20. (П), ДТ20. (П), ДТ4. (П), ДТ4. (П), ДТ4. (П), ДТ5. (П), ДТ5. (П), ЯП11-15., ЯП23., ЯП23., ЯП3-7., ЯП3-7., ЯП35., ЯП35., ЯР1., ЯР1., ЯР19., ЯР19., ЯР21-25., ЯР21-25., ЯР33., ЯР33., ЯРМ37П., ЯРМ37П., ЯРМ5П., ЯРНДП., ЯРНДП.
Other:
- note added: "К отсасывающей линии ТП"
- note added: "М29П"
- note added: "М37П"
- note added: "М5П"
- company: (none) -> АТ-451

Commit message: Наведен порядок с рамками
Connections:
- net at ДТ23. (П): now also Стрелка15.4; no longer Путь3.
- net at Стрелка15.: now also ДТ23. (П); no longer ДТ22. (П)
- net at ДТ22. (П): now also Путь1.; no longer Стрелка15.
- net at ДТ16. (П): now also Стрелка14.; no longer Стрелка15.
- net at ДТ21. (П): now also Стрелка20.6
- net at ЯП21-25.: now also ДТ10. (П), Соединитель10.2, Стрелка14.2
- net at Стрелка13.: now also ДТ14. (П)
- net at Стрелка14.: now also ДТ10. (П); no longer Стрелка13.
- net at ДТ14. (П): now also Путь2.; no longer Стрелка13.
- net at Стрелка10.: now also ДТ4. (П)
- net at Стрелка10.: now also ДТ8. (П); no longer Стрелка10.
- net at ДТ4. (П): no longer Стрелка10.
- net at ДТ1. (П): now also Путь1.2
- net at ДТ8. (П): now also Стрелка11.; no longer Стрелка10.
- net at ДТ10. (П): now also Соединитель9.2, Стрелка12.2, ЯР11-15.; no longer Стрелка14.
- net at Стрелка17.: now also ДТ13. (П)
- net at ДТ11. (П): now also Стрелка13.6; no longer Стрелка17.
- net at ДТ13. (П): now also Стрелка18.; no longer Стрелка17.
- net at ДТ17. (П): now also Путь4.; no longer Стрелка18.
- net at Стрелка9.: now also ДТ24. (П)
- net at ДТ7. (П): now also Стрелка15.; no longer Стрелка9.
- net at ДТ24. (П): no longer Стрелка9.
- net at ЯРМ29П.: now also ДТ19. (П), Электротяга2.2
- net at ЯПНП.: now also ДТ2. (П), ДТ5. (П)
- net at Стрелка13.: now also Стрелка11.
- net at Стрелка11.: no longer Стрелка13.
- net at ДТ3. (П): now also Соединитель1.2, Стрелка9.2, ЯП1.
- net at Стрелка9.: now also ДТ6. (П); no longer ДТ3. (П)
- net at ДТ6. (П): now also Стрелка12.6, ЯП11-15.; no longer Стрелка9.
- net at ДТ19. (П): now also Стрелка16.4
- net at Стрелка12.: now also Стрелка12.
- net at Стрелка12.: no longer Стрелка12.
- net at Стрелка14.: now also ДТ9. (П); no longer ДТ16. (П)
- net at ЯП9.: now also ДТ9. (П), Стрелка11.6
- net at ДТ15. (П): now also Стрелка16.6
- net at Стрелка19.: now also ДТ18. (П); no longer ДТ15. (П)
- net at Стрелка15.: no longer ДТ7. (П)
- net at ЯП19.: now also ДТ12. (П), Соединитель11.2, Стрелка15.2
- net at ДТ12. (П): now also Стрелка15.
- net at ЯР27.: now also ДТ9. (П), Стрелка14.6
- net at Стрелка11.: now also ДТ5. (П)
- net at ДТ5. (П): no longer Стрелка11.
- net at ДТ18. (П): no longer Стрелка19.
- new net: ДТ23. (П), Путь3.
- new net: ДТ22. (П), Стрелка15. (x2)
- new net: ДТ16. (П), Стрелка15. (x2)
- new net: ДТ23. (П), Стрелка15.
- new net: ДТ22. (П), Стрелка15.5, ЯП35.
- new net: ДТ22. (П), Стрелка15.6, ЯП35.
- new net: ДТ21. (П), Путь6.
- new net: Стрелка13., Стрелка14. (x2)
- new net: ДТ14. (П), Стрелка13.
- new net: ДТ14. (П), Стрелка13.5, ЯР21-25.
- new net: ДТ14. (П), Стрелка13.6, ЯР21-25.
- new net: Стрелка10., Стрелка10. (x2)
- new net: ДТ4. (П), Стрелка10.
- new net: ДТ4. (П), Стрелка10.5, ЯП3-7.
- new net: ДТ4. (П), Стрелка10.6, ЯП3-7.
- new net: ДТ1. (П), ДТ3. (П), ЯРНДП. (x2)
- new net: ДТ8. (П), Стрелка10.
- new net: ДТ10. (П), Стрелка14.
- new net: ДТ4. (П), Изостыки1.1, Тупик1.1, Электротяга1.1, ЯРМ5П.
- new net: ДТ11. (П), Стрелка17. (x2)
- new net: ДТ13. (П), Стрелка17.
- new net: ДТ11. (П), Стрелка17.5, ЯП23.
- new net: ДТ11. (П), Стрелка17.6, ЯП23.
- new net: ДТ17. (П), Стрелка18. (x2)
- new net: ДТ17. (П), Путь4.
- new net: ДТ7. (П), Стрелка9. (x2)
- new net: ДТ24. (П), Стрелка9.
- new net: ДТ19. (П), Электротяга2.1, ЯРМ29П.
- new net: ДТ2. (П), ДТ5. (П), ЯПНП.
- new net: ДТ11. (П), Стрелка13. (x2)
- new net: Стрелка11., Стрелка13.
- new net: ДТ14. (П), Путь2.
- new net: ДТ3. (П), Стрелка9. (x2)
- new net: ДТ6. (П), Стрелка9.
- new net: ДТ6. (П), Стрелка9.5, ЯР1.
- new net: ДТ6. (П), Стрелка9.6, ЯР1.
- new net: ДТ10. (П), Стрелка12. (x2)
- new net: Стрелка12., Стрелка12.
- new net: ДТ20. (П), Электротяга3.1, ЯРМ37П.
- new net: ДТ20. (П), Электротяга3.2, ЯРМ37П.
- new net: ДТ22. (П), Путь1.
- new net: ДТ6. (П), Стрелка12. (x2)
- new net: ДТ6. (П), Стрелка12.5, ЯП11-15.
- new net: ДТ16. (П), Стрелка14.
- new net: ДТ9. (П), Стрелка11.5, ЯП9.
- new net: ДТ15. (П), Стрелка19.5, ЯР33.
- new net: ДТ15. (П), Стрелка19.6, ЯР33.
- new net: ДТ15. (П), Стрелка19. (x2)
- new net: ДТ7. (П), Стрелка15.5, ЯР19.
- new net: ДТ7. (П), Стрелка15.6, ЯР19.
- new net: ДТ7. (П), Стрелка15.
- new net: ДТ12. (П), Стрелка15.
- new net: ДТ9. (П), Стрелка14.5, ЯР27.
- new net: ДТ9. (П), Стрелка11. (x2)
- new net: ДТ5. (П), Стрелка11.
- new net: ДТ9. (П), Стрелка14.
- new net: ДТ18. (П), Стрелка19.
- new net: ДТ8. (П), Стрелка11.
- new net: ДТ13. (П), Стрелка18.
- now unconnected: ДТ18. (П), ДТ2. (П), ДТ2. (П), ДТ20. (П), ДТ20. (П), ДТ24. (П), ДТ4. (П), ДТ4. (П), ДТ4. (П), ДТ4. (П), ДТ5. (П), ДТ5. (П), ДТ5. (П), Стрелка11., Стрелка11., Стрелка11., Стрелка12., Стрелка12., Стрелка12., Стрелка15., Стрелка15., Стрелка15., ЯП1., ЯП11-15., ЯП11-15., ЯП23., ЯП23., ЯП3-7., ЯП3-7., ЯП35., ЯП35., ЯР1., ЯР1., ЯР11-15., ЯР19., ЯР19., ЯР21-25., ЯР21-25., ЯР33., ЯР33., ЯРМ37П., ЯРМ37П., ЯРМ5П., ЯРНДП., ЯРНДП.

Commit message: В двухнитке ЭЦ проложен кабель СЦБ
Parts:
- added К11, К111 (x3), К1111 (x3), К11111, К111111: ~, symbol SCB_Двухнитка:Муфта_ЭЦ
- added Магистральный_1, Магистральный_2, Магистральный_3, Магистральный_4, Магистральный_5, Магистральный_6, Магистральный_7, Магистральный_8, Магистральный_9, Магистральный_кабель1 (x20): ~, symbol SCB:Магистральный_кабель
- added ЭЦ11: ~, symbol SCB:Пост_ЭЦ
- Путь2: Путь IП -> IIП
- ЯП19, ЯП37, ЯР31: Частота1 (none) -> 420/12; Частота2 (none) -> 720/8
Connections:
- net at ДТ23. (П): now also Стрелка15.4; no longer Путь3.
- net at Стрелка15.: now also ДТ23. (П); no longer ДТ22. (П)
- net at ДТ22. (П): now also Путь1.; no longer Стрелка15.
- net at ДТ16. (П): now also Стрелка14.; no longer Стрелка15.
- net at ДТ21. (П): now also Стрелка20.6
- net at Путь6.: no longer ДТ21. (П)
- net at ЯП21-25.: now also ДТ10. (П), Соединитель10.2, Стрелка14.2
- net at Стрелка13.: now also ДТ14. (П)
- net at Стрелка14.: now also ДТ10. (П); no longer Стрелка13.
- net at ДТ14. (П): now also Путь2.; no longer Стрелка13.
- net at Стрелка10.: now also ДТ4. (П)
- net at Стрелка10.: now also ДТ8. (П); no longer Стрелка10.
- net at ДТ4. (П): no longer Стрелка10.
- net at ДТ1. (П): now also Путь1.2
- net at ДТ8. (П): now also Стрелка11.; no longer Стрелка10.
- net at ДТ10. (П): now also Соединитель9.2, Стрелка12.2, ЯР11-15.; no longer Стрелка14.
- net at Стрелка17.: now also ДТ13. (П)
- net at ДТ11. (П): now also Стрелка13.6; no longer Стрелка17.
- net at ДТ13. (П): now also Стрелка18.; no longer Стрелка17.
- net at ДТ17. (П): now also Путь4.; no longer Стрелка18.
- net at Путь4.: no longer ДТ17. (П)
- net at Стрелка9.: now also ДТ24. (П)
- net at ДТ7. (П): now also Стрелка15.; no longer Стрелка9.
- net at ДТ24. (П): no longer Стрелка9.
- net at ЯРМ29П.: now also ДТ19. (П), Электротяга2.2
- net at ЯПНП.: now also ДТ2. (П), ДТ5. (П)
- net at ДТ2. (П), ДТ5. (П): no longer ЯПНП.
- net at Стрелка13.: now also Стрелка11.
- net at Стрелка11.: no longer Стрелка13.
- net at Путь2.: no longer ДТ14. (П)
- net at ДТ3. (П): now also Соединитель1.2, Стрелка9.2, ЯП1.
- net at Стрелка9.: now also ДТ6. (П); no longer ДТ3. (П)
- net at ДТ6. (П): now also Стрелка12.6, ЯП11-15.; no longer Стрелка9.
- net at ДТ19. (П): now also Стрелка16.4
- net at Стрелка12.: now also Стрелка12.
- net at Стрелка12.: no longer Стрелка12.
- net at ЯР31.: now also ДТ13. (П), Стрелка18.
- net at Стрелка14.: now also ДТ9. (П); no longer ДТ16. (П)
- net at ЯП9.: now also ДТ9. (П), Стрелка11.6
- net at ДТ15. (П): now also Стрелка16.6
- net at Стрелка19.: now also ДТ18. (П); no longer ДТ15. (П)
- net at Стрелка15.: no longer ДТ7. (П)
- net at ЯП19.: now also ДТ12. (П), Соединитель11.2, Стрелка15.2
- net at ДТ12. (П): now also Стрелка15.
- net at ЯР27.: now also ДТ9. (П), Стрелка14.6
- net at Стрелка11.: now also ДТ5. (П)
- net at ДТ18. (П): no longer Стрелка19.
- new net: Магистральный_кабель1. (привязка), Магистральный_кабель1. (привязка) (x13)
- new net: ДТ23. (П), Путь3.
- new net: К111., Магистральный_кабель1. (привязка) (x3)
- new net: ДТ22. (П), Стрелка15. (x2)
- new net: ДТ16. (П), Стрелка15. (x2)
- new net: ДТ23. (П), Стрелка15.
- new net: ДТ22. (П), Стрелка15.5, ЯП35.
- new net: ДТ22. (П), Стрелка15.6, ЯП35.
- new net: Магистральный_9. (привязка), Магистральный_кабель1. (привязка)
- new net: Стрелка13., Стрелка14. (x2)
- new net: ДТ14. (П), Стрелка13.
- new net: ДТ14. (П), Стрелка13.5, ЯР21-25.
- new net: ДТ14. (П), Стрелка13.6, ЯР21-25.
- new net: Стрелка10., Стрелка10. (x2)
- new net: ДТ4. (П), Стрелка10.
- new net: ДТ4. (П), Стрелка10.5, ЯП3-7.
- new net: ДТ4. (П), Стрелка10.6, ЯП3-7.
- new net: ДТ1. (П), ДТ3. (П), ЯРНДП. (x2)
- new net: ДТ1. (П), ДТ3. (П) (x2)
- new net: ДТ8. (П), Стрелка10.
- new net: ДТ10. (П), Стрелка14.
- new net: Магистральный_1. (привязка), Магистральный_3. (привязка)
- new net: Магистральный_1. (привязка), Магистральный_кабель1. (привязка)
- new net: ДТ4. (П), Изостыки1.1, Тупик1.1, Электротяга1.1, ЯРМ5П.
- new net: ДТ11. (П), Стрелка17. (x2)
- new net: ДТ13. (П), Стрелка17.
- new net: ДТ11. (П), Стрелка17.5, ЯП23.
- new net: ДТ11. (П), Стрелка17.6, ЯП23.
- new net: ДТ17. (П), Стрелка18. (x2)
- new net: ДТ17. (П), Путь4.
- new net: ДТ7. (П), Стрелка9. (x2)
- new net: ДТ24. (П), Стрелка9.
- new net: ДТ19. (П), Электротяга2.1, ЯРМ29П.
- new net: ДТ2. (П), ДТ5. (П), ЯПНП.
- new net: ДТ11. (П), Стрелка13. (x2)
- new net: Стрелка11., Стрелка13.
- new net: ДТ14. (П), Путь2.
- new net: ДТ3. (П), Стрелка9. (x2)
- new net: ДТ6. (П), Стрелка9.
- new net: ДТ6. (П), Стрелка9.5, ЯР1.
- new net: ДТ6. (П), Стрелка9.6, ЯР1.
- new net: ДТ10. (П), Стрелка12. (x2)
- new net: Стрелка12., Стрелка12.
- new net: К111111., Магистральный_кабель1. (привязка)
- new net: ДТ20. (П), Электротяга3.1, ЯРМ37П.
- new net: ДТ20. (П), Электротяга3.2, ЯРМ37П.
- new net: ДТ22. (П), Путь1.
- new net: К11111., Магистральный_кабель1. (привязка) (x2)
- new net: ДТ6. (П), Стрелка12. (x2)
- new net: ДТ6. (П), Стрелка12.5, ЯП11-15.
- new net: К11., Магистральный_6. (привязка)
- new net: К11., Магистральный_7. (привязка)
- new net: Магистральный_5. (привязка), Магистральный_6. (привязка)
- new net: ДТ16. (П), Стрелка14.
- new net: ДТ9. (П), Стрелка11.5, ЯП9.
- new net: ДТ15. (П), Стрелка19.5, ЯР33.
- new net: ДТ15. (П), Стрелка19.6, ЯР33.
- new net: ДТ15. (П), Стрелка19. (x2)
- new net: ДТ7. (П), Стрелка15.5, ЯР19.
- new net: ДТ7. (П), Стрелка15.6, ЯР19.
- new net: ДТ7. (П), Стрелка15.
- new net: К1111., Магистральный_кабель1. (привязка) (x3)
- new net: К111111., Магистральный_2. (привязка)
- new net: Магистральный_2. (привязка), Магистральный_кабель1. (привязка)
- new net: ДТ12. (П), Стрелка15.
- new net: ДТ9. (П), Стрелка14.5, ЯР27.
- new net: ДТ9. (П), Стрелка11. (x2)
- new net: ДТ5. (П), Стрелка11.
- new net: Магистральный_4. (привязка), Магистральный_5. (привязка)
- new net: ДТ9. (П), Стрелка14.
- new net: ДТ18. (П), Стрелка19.
- new net: ДТ2. (П), ДТ5. (П)
- new net: Магистральный_3. (привязка), Магистральный_4. (привязка)
- new net: ДТ8. (П), Стрелка11.
- new net: Магистральный_8. (привязка), Магистральный_кабель1. (привязка)
- now unconnected: ДТ18. (П), ДТ20. (П), ДТ20. (П), ДТ24. (П), ДТ4. (П), ДТ4. (П), ДТ4. (П), ДТ4. (П), Путь2., Путь4., Путь6., Стрелка11., Стрелка11., Стрелка11., Стрелка12., Стрелка12., Стрелка12., Стрелка15., Стрелка15., Стрелка15., ЯП1., ЯП11-15., ЯП11-15., ЯП23., ЯП23., ЯП3-7., ЯП3-7., ЯП35., ЯП35., ЯР1., ЯР1., ЯР11-15., ЯР19., ЯР19., ЯР21-25., ЯР21-25., ЯР33., ЯР33., ЯРМ37П., ЯРМ37П., ЯРМ5П., ЯРНДП., ЯРНДП.
Other:
- note added: "Ввод каб.СЦБ"
