File: example/АБТЦ-2003/Схемы/АПСА3.kicad_sch (KiCad schematic)
At the start: 20 parts

Commit message: Шаблон АБТЦ обновлен
Parts:
- R18, R19, R20: Тип C5-35В -> (none)

Commit message: Обновление примера
Parts:
- Н1, Н11, Н111, Н1111, Н11111: symbol SCB_Relay:Контакт_нейтрального_якоря -> SCB_Legacy:Контакт_нейтрального_якоря_бн
- Н1, Н11, Н111, Н1111: symbol SCB_Relay:Контакт_нейтрального_якоря_НЗ -> SCB_Legacy:Контакт_нейтрального_якоря_НЗ_бн
Changed lines of the file:
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@@
 (kicad_sch
-	(version 20231120)
+	(version 20250114)
 	(generator "eeschema")
-	(generator_version "8.0")
+	(generator_version "9.0")
 	(paper "A3")
 	(title_block
@@
 	)
 	(symbol
-		(lib_name "SCB_Relay:Контакт_нейтрального_якоря")
-		(lib_id "SCB_Relay:Контакт_нейтрального_якоря")
+		(lib_name "Контакт_нейтрального_якоря_бн_5")
+		(lib_id "SCB_Legacy:Контакт_нейтрального_якоря_бн")
 		(at 152.4 146.05 0)
 		(unit 3)
@@
 	)
 	(symbol
-		(lib_name "SCB_Relay:Контакт_нейтрального_якоря_НЗ")
-		(lib_id "SCB_Relay:Контакт_нейтрального_якоря_НЗ")
+		(lib_name "Контакт_нейтрального_якоря_НЗ_бн_2")
+		(lib_id "SCB_Legacy:Контакт_нейтрального_якоря_НЗ_бн")
 		(at 279.4 146.05 0)
 		(unit 3)
@@
 	)
 	(symbol
-		(lib_name "SCB_Relay:Контакт_нейтрального_якоря")
-		(lib_id "SCB_Relay:Контакт_нейтрального_якоря")
+		(lib_name "Контакт_нейтрального_якоря_бн_9")
+		(lib_id "SCB_Legacy:Контакт_нейтрального_якоря_бн")
 		(at 298.45 63.5 0)
 		(unit 3)
@@
 	)
 	(symbol
-		(lib_name "SCB_Relay:Контакт_нейтрального_якоря")
-		(lib_id "SCB_Relay:Контакт_нейтрального_якоря")
+		(lib_name "Контакт_нейтрального_якоря_бн_6")
+		(lib_id "SCB_Legacy:Контакт_нейтрального_якоря_бн")
 		(at 349.25 82.55 0)
 		(unit 3)
@@
 	)
 	(symbol
-		(lib_name "SCB_Relay:Контакт_нейтрального_якоря")
-		(lib_id "SCB_Relay:Контакт_нейтрального_якоря")
+		(lib_name "Контакт_нейтрального_якоря_бн_3")
+		(lib_id "SCB_Legacy:Контакт_нейтрального_якоря_бн")
 		(at 127 106.68 0)
 		(unit 3)
@@
 	)
 	(symbol
-		(lib_name "SCB_Relay:Контакт_нейтрального_якоря")
-		(lib_id "SCB_Relay:Контакт_нейтрального_якоря")
+		(lib_name "Контакт_нейтрального_якоря_бн_4")
+		(lib_id "SCB_Legacy:Контакт_нейтрального_якоря_бн")
 		(at 127 82.55 0)
 		(unit 3)
@@
 	)
 	(symbol
-		(lib_name "SCB_Relay:Контакт_нейтрального_якоря_НЗ")
-		(lib_id "SCB_Relay:Контакт_нейтрального_якоря_НЗ")
+		(lib_name "Контакт_нейтрального_якоря_НЗ_бн_3")
+		(lib_id "SCB_Legacy:Контакт_нейтрального_якоря_НЗ_бн")
 		(at 374.65 82.55 0)
 		(unit 2)
@@
 	)
 	(symbol
-		(lib_name "SCB_Relay:Контакт_нейтрального_якоря")
-		(lib_id "SCB_Relay:Контакт_нейтрального_якоря")
+		(lib_name "Контакт_нейтрального_якоря_бн_7")
+		(lib_id "SCB_Legacy:Контакт_нейтрального_якоря_бн")
 		(at 152.4 82.55 0)
 		(unit 3)
@@
 	)
 	(symbol
-		(lib_name "SCB_Relay:Контакт_нейтрального_якоря")
-		(lib_id "SCB_Relay:Контакт_нейтрального_якоря")
+		(lib_name "Контакт_нейтрального_якоря_бн_13")
+		(lib_id "SCB_Legacy:Контакт_нейтрального_якоря_бн")
 		(at 101.6 63.5 0)
 		(unit 2)
@@
 	)
 	(symbol
-		(lib_name "SCB_Relay:Контакт_нейтрального_якоря")
-		(lib_id "SCB_Relay:Контакт_нейтрального_якоря")
+		(lib_name "Контакт_нейтрального_якоря_бн_8")
+		(lib_id "SCB_Legacy:Контакт_нейтрального_якоря_бн")
 		(at 228.6 146.05 0)
 		(unit 2)
@@
 	)
 	(symbol
-		(lib_name "SCB_Relay:Контакт_нейтрального_якоря")
-		(lib_id "SCB_Relay:Контакт_нейтрального_якоря")
+		(lib_name "Контакт_нейтрального_якоря_бн_12")
+		(lib_id "SCB_Legacy:Контакт_нейтрального_якоря_бн")
 		(at 177.8 82.55 0)
 		(unit 3)
@@
 	)
 	(symbol
-		(lib_name "SCB_Relay:Контакт_нейтрального_якоря_НЗ")
-		(lib_id "SCB_Relay:Контакт_нейтрального_якоря_НЗ")
+		(lib_name "Контакт_нейтрального_якоря_НЗ_бн_1")
+		(lib_id "SCB_Legacy:Контакт_нейтрального_якоря_НЗ_бн")
 		(at 254 146.05 0)
 		(unit 3)
@@
 	)
 	(symbol
-		(lib_name "SCB_Relay:Контакт_нейтрального_якоря")
-		(lib_id "SCB_Relay:Контакт_нейтрального_якоря")
+		(lib_name "Контакт_нейтрального_якоря_бн_15")
+		(lib_id "SCB_Legacy:Контакт_нейтрального_якоря_бн")
 		(at 177.8 146.05 0)
 		(unit 2)
@@
 	)
 	(symbol
-		(lib_name "SCB_Relay:Контакт_нейтрального_якоря_НЗ")
-		(lib_id "SCB_Relay:Контакт_нейтрального_якоря_НЗ")
+		(lib_name "Контакт_нейтрального_якоря_НЗ_бн_4")
+		(lib_id "SCB_Legacy:Контакт_нейтрального_якоря_НЗ_бн")
 		(at 203.2 82.55 0)
 		(unit 3)
@@
 	)
 	(symbol
-		(lib_name "SCB_Relay:Контакт_нейтрального_якоря_НЗ")
-		(lib_id "SCB_Relay:Контакт_нейтрального_якоря_НЗ")
+		(lib_name "Контакт_нейтрального_якоря_НЗ_бн_5")
+		(lib_id "SCB_Legacy:Контакт_нейтрального_якоря_НЗ_бн")
 		(at 304.8 146.05 0)
 		(unit 2)
@@
 	)
 	(symbol
-		(lib_name "SCB_Relay:Контакт_нейтрального_якоря")
-		(lib_id "SCB_Relay:Контакт_нейтрального_якоря")
+		(lib_name "Контакт_нейтрального_якоря_бн_1")
+		(lib_id "SCB_Legacy:Контакт_нейтрального_якоря_бн")
 		(at 298.45 31.75 0)
 		(unit 3)
@@
 	)
 	(symbol
-		(lib_name "SCB_Relay:Контакт_нейтрального_якоря")
-		(lib_id "SCB_Relay:Контакт_нейтрального_якоря")
+		(lib_name "Контакт_нейтрального_якоря_бн_10")
+		(lib_id "SCB_Legacy:Контакт_нейтрального_якоря_бн")
 		(at 86.36 146.05 0)
 		(mirror y)
@@
 	)
 	(symbol
-		(lib_name "SCB_Relay:Контакт_нейтрального_якоря")
-		(lib_id "SCB_Relay:Контакт_нейтрального_якоря")
+		(lib_name "Контакт_нейтрального_якоря_бн_14")
+		(lib_id "SCB_Legacy:Контакт_нейтрального_якоря_бн")
 		(at 203.2 146.05 0)
 		(unit 1)
@@
 	)
 	(symbol
-		(lib_name "SCB_Relay:Контакт_нейтрального_якоря")
-		(lib_id "SCB_Relay:Контакт_нейтрального_якоря")
+		(lib_id "SCB_Legacy:Контакт_нейтрального_якоря_бн")
 		(at 234.95 31.75 0)
 		(mirror y)
@@
 	)
 	(symbol
-		(lib_name "SCB_Relay:Контакт_нейтрального_якоря_НЗ")
-		(lib_id "SCB_Relay:Контакт_нейтрального_якоря_НЗ")
+		(lib_id "SCB_Legacy:Контакт_нейтрального_якоря_НЗ_бн")
 		(at 152.4 106.68 0)
 		(unit 2)
@@
 	)
 	(symbol
-		(lib_name "SCB_Relay:Контакт_нейтрального_якоря")
-		(lib_id "SCB_Relay:Контакт_нейтрального_якоря")
+		(lib_name "Контакт_нейтрального_якоря_бн_11")
+		(lib_id "SCB_Legacy:Контакт_нейтрального_якоря_бн")
 		(at 152.4 63.5 0)
 		(unit 3)
@@
 	)
 	(symbol
-		(lib_name "SCB_Relay:Контакт_нейтрального_якоря")
-		(lib_id "SCB_Relay:Контакт_нейтрального_якоря")
+		(lib_name "Контакт_нейтрального_якоря_бн_2")
+		(lib_id "SCB_Legacy:Контакт_нейтрального_якоря_бн")
 		(at 127 146.05 0)
 		(unit 3)
