File: example/АБТЦ-2003/Схемы/ПЗ26-32.kicad_sch (KiCad schematic)
At the start: 85 parts

Commit message: Шаблон АБТЦ обновлен
Parts:
- removed Генератор111111101111, Генератор11111111, Генератор1111111111, Генератор11111111111, Генератор111111111111, Генератор111111121111, Генератор11111121111, Генератор11111131111, Генератор11111141111, Генератор11111151111, Генератор11111161111, Генератор11111171111, Генератор11111181111, Генератор11111191111, Генератор1111121111: ~, symbol SCB:Генератор_Нитки
- removed И111111, И1111111: ~, symbol SCB:Изостык
- removed Приемник11111101111, Приемник11111111, Приемник1111111111, Приемник11111111111, Приемник11111121111, Приемник1111121111, Приемник1111131111, Приемник1111141111, Приемник1111151111, Приемник1111161111, Приемник1111171111, Приемник1111181111, Приемник1111191111, Приемник11121111: ~, symbol SCB:Приемник_Нитки
- removed Светофор111111, Светофор1111111, Светофор11111111, Светофор11121111, Светофор11131111, Светофор1121111, Светофор11211111, Светофор1131111, Светофор121111, Светофор1211111, Светофор131111, Светофор1311111: ~, symbol SCB:Светофор
- removed УКСПС111111, УКСПС112111, УКСПС121111, УКСПС131111: ~, symbol SCB:УКСПС
- added Генератор11111, Генератор1111111, Генератор111111101, Генератор11111111, Генератор111111111, Генератор111111121, Генератор11111121, Генератор11111131, Генератор11111141, Генератор11111151, Генератор11111161, Генератор11111171, Генератор11111181, Генератор11111191, Генератор1111121: ~, symbol SCB_АБТЦ:Генератор_Нитки
- added И111, И1111: ~, symbol SCB:Изостык
- added Приемник11111, Приемник11111101, Приемник1111111, Приемник11111111, Приемник11111121, Приемник1111121, Приемник1111131, Приемник1111141, Приемник1111151, Приемник1111161, Приемник1111171, Приемник1111181, Приемник1111191, Приемник11121: ~, symbol SCB_АБТЦ:Приемник_Нитки
- added Светофор111, Светофор1111, Светофор11111, Светофор11121, Светофор11131, Светофор1121, Светофор11211, Светофор1131, Светофор121, Светофор1211, Светофор131, Светофор1311: ~, symbol SCB:Светофор
- added УКСПС111, УКСПС112, УКСПС121, УКСПС131: ~, symbol SCB:УКСПС
Connections:
- new net: Генератор11111171., Приемник1111181.
- new net: Генератор11111171., Приемник1111171.
- new net: Генератор111111111., Приемник1111111.
- new net: Генератор1111121., Приемник1111111.
- new net: Генератор111111111., Приемник11111111.
- new net: Генератор11111141., Приемник1111151.
- new net: Генератор11111151., Приемник1111151.
- new net: Генератор111111101., И1111. (привязка)
- new net: Генератор111111121., Приемник11111121.
- new net: Генератор111111121., Приемник1111121.
- new net: Генератор11111121., Приемник11111121.
- new net: Генератор11111., Приемник11111.
- new net: Генератор11111., И111. (привязка)
- new net: Генератор11111161., Приемник1111161.
- new net: Генератор11111161., Приемник1111171.
- new net: Генератор11111191., Приемник11111101.
- new net: Генератор11111191., Приемник1111191.
- new net: Генератор11111131., Приемник1111131.
- new net: Генератор11111121., Приемник1111131.
- new net: Генератор11111111., Приемник11111111.
- new net: Генератор11111111., Приемник1111121.
- new net: Генератор11111141., Приемник1111141.
- new net: Генератор11111181., Приемник1111181.
- new net: Генератор11111181., Приемник1111191.
- new net: Генератор11111131., Приемник1111141.
- new net: Генератор111111101., Приемник11111101.
- new net: Генератор1111111., Приемник11111.
- new net: Генератор11111151., Приемник1111161.
- new net: Генератор1111121., Приемник11121.
- new net: Генератор1111111., Приемник11121.

Commit message: Обновление примера
Parts:
- Н112, Н1121, Н11211, Н112111, Н1121111, Н11211111, Н112111111, Н1121111111, Н11211111111, Н11231, Н112311, Н1123111: symbol SCB_Relay:Контакт_нейтрального_якоря -> SCB_Legacy:Контакт_нейтрального_якоря_бн
- Н113, Н1131, Н11311, Н113111, Н1131111, Н1311, Н13111, Н131111, Н1311111, Н13111111, Н131111111: symbol SCB_Relay:Контакт_нейтрального_якоря_НЗ -> SCB_Legacy:Контакт_нейтрального_якоря_НЗ_бн
Connections:
- net at Генератор11111171.: now also Приемник1111171.; no longer Приемник1111181.
- net at Приемник1111171.: now also Генератор11111161.; no longer Генератор11111171.
- net at Приемник1111111.: now also Генератор1111121.; no longer Генератор111111111.
- net at Генератор1111121.: now also Приемник11121.; no longer Приемник1111111.
- net at Приемник1111151.: now also Генератор11111151.; no longer Генератор11111141.
- net at Генератор11111151.: now also Приемник1111161.; no longer Приемник1111151.
- net at И1111.: now also Генератор111111101.
- net at Генератор111111101.: now also Приемник11111101.; no longer И1111. (привязка)
- net at Генератор111111121.: now also Приемник1111121.; no longer Приемник11111121.
- net at Приемник1111121.: now also Генератор11111111.; no longer Генератор111111121.
- net at Генератор11111.: now also И111.; no longer Приемник11111.
- net at И111.: no longer Генератор11111.
- net at Генератор11111191.: now also Приемник1111191.; no longer Приемник11111101.
- net at Приемник1111191.: now also Генератор11111181.; no longer Генератор11111191.
- net at Приемник1111131.: now also Генератор11111121.; no longer Генератор11111131.
- net at Приемник11121.: now also Генератор1111111.; no longer Генератор1111121.
- new net: Генератор11111171., Приемник1111181.
- new net: Генератор111111111., Приемник1111111.
- new net: Генератор11111141., Приемник1111151.
- new net: Генератор111111121., Приемник11111121.
- new net: Генератор11111., Приемник11111.
- new net: Генератор11111161., Приемник1111161.
- new net: Генератор11111191., Приемник11111101.
- new net: Генератор11111131., Приемник1111131.
