File: example/АБТЦ-2003/Схемы/ПО2-8.kicad_sch (KiCad schematic)
At the start: 77 parts

Commit message: Шаблон АБТЦ обновлен
Parts:
- removed Генератор1111111, Генератор11111110111, Генератор111111111, Генератор1111111111, Генератор11111111111, Генератор11111112111, Генератор1111112111, Генератор1111113111, Генератор1111114111, Генератор1111115111, Генератор1111116111, Генератор1111117111, Генератор1111118111, Генератор1111119111, Генератор111112111: ~, symbol SCB:Генератор_Нитки
- removed И11111, И111111: ~, symbol SCB:Изостык
- removed Приемник1111110111, Приемник1111111, Приемник111111111, Приемник1111111111, Приемник1111112111, Приемник111112111, Приемник111113111, Приемник111114111, Приемник111115111, Приемник111116111, Приемник111117111, Приемник111118111, Приемник111119111, Приемник1112111: ~, symbol SCB:Приемник_Нитки
- removed Светофор111111, Светофор1111111, Светофор1112111, Светофор1113111, Светофор112111, Светофор1121111, Светофор113111, Светофор12111, Светофор121111, Светофор13111, Светофор131111: ~, symbol SCB:Светофор
- removed УКСПС11111, УКСПС11211, УКСПС12111, УКСПС13111: ~, symbol SCB:УКСПС
- added Генератор11111, Генератор1111111, Генератор111111101, Генератор11111111, Генератор111111111, Генератор111111121, Генератор11111121, Генератор11111131, Генератор11111141, Генератор11111151, Генератор11111161, Генератор11111171, Генератор11111181, Генератор11111191, Генератор1111121: ~, symbol SCB_АБТЦ:Генератор_Нитки
- added И111, И1111: ~, symbol SCB:Изостык
- added Приемник11111, Приемник11111101, Приемник1111111, Приемник11111111, Приемник11111121, Приемник1111121, Приемник1111131, Приемник1111141, Приемник1111151, Приемник1111161, Приемник1111171, Приемник1111181, Приемник1111191, Приемник11121: ~, symbol SCB_АБТЦ:Приемник_Нитки
- added Светофор111, Светофор1111, Светофор11121, Светофор11131, Светофор1121, Светофор11211, Светофор1131, Светофор121, Светофор1211, Светофор131, Светофор1311: ~, symbol SCB:Светофор
- added УКСПС111 (x2), УКСПС121, УКСПС131: ~, symbol SCB:УКСПС
- Светофор11111: Литера Ч -> 5
Connections:
- new net: Генератор11111181., Приемник1111181.
- new net: Генератор11111171., Приемник1111181.
- new net: Генератор11111111., Приемник11111111.
- new net: Генератор11111111., Приемник1111121.
- new net: Генератор111111101., И1111. (привязка)
- new net: Генератор111111101., Приемник11111101.
- new net: Генератор11111131., Приемник1111141.
- new net: Генератор11111141., Приемник1111141.
- new net: Генератор11111131., Приемник1111131.
- new net: Генератор11111121., Приемник11111121.
- new net: Генератор111111121., Приемник11111121.
- new net: Генератор11111151., Приемник1111161.
- new net: Генератор11111151., Приемник1111151.
- new net: Генератор1111121., Приемник1111111.
- new net: Генератор1111121., Приемник11121.
- new net: Генератор11111191., Приемник1111191.
- new net: Генератор11111181., Приемник1111191.
- new net: Генератор111111111., Приемник11111111.
- new net: Генератор11111161., Приемник1111161.
- new net: Генератор11111., И111. (привязка)
- new net: Генератор111111111., Приемник1111111.
- new net: Генератор11111161., Приемник1111171.
- new net: Генератор111111121., Приемник1111121.
- new net: Генератор11111191., Приемник11111101.
- new net: Генератор11111121., Приемник1111131.
- new net: Генератор11111., Приемник11111.
- new net: Генератор11111171., Приемник1111171.
- new net: Генератор1111111., Приемник11111.
- new net: Генератор1111111., Приемник11121.
- new net: Генератор11111141., Приемник1111151.

Commit message: Обновление примера
Parts:
- Н1, Н11, Н111, Н1111, Н11111, Н112, Н1121, Н11211, Н12: symbol SCB_Relay:Контакт_нейтрального_якоря -> SCB_Legacy:Контакт_нейтрального_якоря_бн
- Н1, Н11, Н111, Н1111, Н11111, Н111111, Н13, Н131, Н1311, Н13111, Н131111, Н1311111: symbol SCB_Relay:Контакт_нейтрального_якоря_НЗ -> SCB_Legacy:Контакт_нейтрального_якоря_НЗ_бн
Connections:
- net at Приемник1111181.: now also Генератор11111171.; no longer Генератор11111181.
- net at Генератор11111171.: now also Приемник1111171.; no longer Приемник1111181.
- net at Генератор11111111.: now also Приемник1111121.; no longer Приемник11111111.
- net at Приемник1111121.: now also Генератор111111121.; no longer Генератор11111111.
- net at Генератор111111101.: now also Приемник11111101.; no longer И1111. (привязка)
- net at Приемник11111101.: now also Генератор11111191.; no longer Генератор111111101.
- net at Приемник1111141.: now also Генератор11111141.; no longer Генератор11111131.
- net at Генератор11111141.: now also Приемник1111151.; no longer Приемник1111141.
- net at Приемник11111121.: now also Генератор111111121.; no longer Генератор11111121.
- net at Генератор11111151.: now also Приемник1111151.; no longer Приемник1111161.
- net at Генератор1111121.: now also Приемник11121.; no longer Приемник1111111.
- net at Приемник11121.: now also Генератор1111111.; no longer Генератор1111121.
- net at Приемник1111191.: now also Генератор11111181.; no longer Генератор11111191.
- net at И111.: now also Генератор11111.
- net at Генератор11111.: now also Приемник11111.; no longer И111. (привязка)
- net at Приемник11111.: now also Генератор1111111.; no longer Генератор11111.
- new net: Генератор11111181., Приемник1111181.
- new net: Генератор11111111., Приемник11111111.
- new net: Генератор111111101., И1111.
- new net: Генератор11111131., Приемник1111141.
- new net: Генератор11111121., Приемник11111121.
- new net: Генератор11111151., Приемник1111161.
- new net: Генератор1111121., Приемник1111111.
- new net: Генератор11111191., Приемник1111191.
