File: example/АБТЦ-2003/Схемы/Т4-5.kicad_sch (KiCad schematic)
At the start: 71 parts

Commit message: Шаблон АБТЦ обновлен
Parts:
- removed Генератор111111101111, Генератор11111111, Генератор1111111111, Генератор11111111111, Генератор111111111111, Генератор111111121111, Генератор11111121111, Генератор11111131111, Генератор11111141111, Генератор11111151111, Генератор11111161111, Генератор11111171111, Генератор11111181111, Генератор11111191111, Генератор1111121111: ~, symbol SCB:Генератор_Нитки
- removed И111111, И1111111: ~, symbol SCB:Изостык
- removed Приемник11111101111, Приемник11111111, Приемник1111111111, Приемник11111111111, Приемник11111121111, Приемник1111121111, Приемник1111131111, Приемник1111141111, Приемник1111151111, Приемник1111161111, Приемник1111171111, Приемник1111181111, Приемник1111191111, Приемник11121111: ~, symbol SCB:Приемник_Нитки
- removed Светофор111111, Светофор1111111, Светофор11111111, Светофор11121111, Светофор11131111, Светофор1121111, Светофор11211111, Светофор1131111, Светофор121111, Светофор1211111, Светофор131111, Светофор1311111: ~, symbol SCB:Светофор
- removed УКСПС111111, УКСПС112111, УКСПС121111, УКСПС131111: ~, symbol SCB:УКСПС
- added Генератор11111, Генератор1111111, Генератор111111101, Генератор11111111, Генератор111111111, Генератор111111121, Генератор11111121, Генератор11111131, Генератор11111141, Генератор11111151, Генератор11111161, Генератор11111171, Генератор11111181, Генератор11111191, Генератор1111121: ~, symbol SCB_АБТЦ:Генератор_Нитки
- added И111, И1111: ~, symbol SCB:Изостык
- added Приемник11111, Приемник11111101, Приемник1111111, Приемник11111111, Приемник11111121, Приемник1111121, Приемник1111131, Приемник1111141, Приемник1111151, Приемник1111161, Приемник1111171, Приемник1111181, Приемник1111191, Приемник11121: ~, symbol SCB_АБТЦ:Приемник_Нитки
- added Светофор111, Светофор1111, Светофор11111, Светофор11121, Светофор11131, Светофор1121, Светофор11211, Светофор1131, Светофор121, Светофор1211, Светофор131, Светофор1311: ~, symbol SCB:Светофор
- added УКСПС111 (x2), УКСПС121, УКСПС131: ~, symbol SCB:УКСПС
Connections:
- new net: Генератор11111131., Приемник1111131.
- new net: Генератор11111131., Приемник1111141.
- new net: Генератор11111191., Приемник11111101.
- new net: Генератор111111101., Приемник11111101.
- new net: Генератор11111121., Приемник11111121.
- new net: Генератор111111121., Приемник11111121.
- new net: Генератор11111141., Приемник1111151.
- new net: Генератор11111141., Приемник1111141.
- new net: Генератор1111121., Приемник11121.
- new net: Генератор1111111., Приемник11121.
- new net: Генератор1111121., Приемник1111111.
- new net: Генератор1111111., Приемник11111.
- new net: Генератор11111., Приемник11111.
- new net: Генератор11111191., Приемник1111191.
- new net: Генератор11111181., Приемник1111191.
- new net: Генератор111111121., Приемник1111121.
- new net: Генератор11111111., Приемник1111121.
- new net: Генератор11111121., Приемник1111131.
- new net: Генератор111111111., Приемник11111111.
- new net: Генератор111111111., Приемник1111111.
- new net: Генератор11111171., Приемник1111171.
- new net: Генератор11111171., Приемник1111181.
- new net: Генератор111111101., И1111. (привязка)
- new net: Генератор11111151., Приемник1111151.
- new net: Генератор11111111., Приемник11111111.
- new net: Генератор11111161., Приемник1111171.
- new net: Генератор11111151., Приемник1111161.
- new net: Генератор11111181., Приемник1111181.
- new net: Генератор11111., И111. (привязка)
- new net: Генератор11111161., Приемник1111161.

Commit message: Обновление примера
Parts:
- Н11, Н111, Н11113, Н1112211, Н11122111, Н111221112, Н11122112, Н1112211212, Н11122113, Н1113, Н11131, Н113, Н1131: symbol SCB_Relay:Контакт_нейтрального_якоря_НЗ -> SCB_Legacy:Контакт_нейтрального_якоря_НЗ_бн
- Н12, Н121, Н1211: symbol SCB_Relay:Контакт_нейтрального_якоря -> SCB_Legacy:Контакт_нейтрального_якоря_бн
Connections:
- net at Генератор11111131.: now also Приемник1111141.; no longer Приемник1111131.
- net at Приемник1111141.: now also Генератор11111141.; no longer Генератор11111131.
- net at Приемник11111101.: now also Генератор111111101.; no longer Генератор11111191.
- net at Генератор111111101.: now also И1111.; no longer Приемник11111101.
- net at Приемник11111121.: now also Генератор111111121.; no longer Генератор11111121.
- net at Генератор111111121.: now also Приемник1111121.; no longer Приемник11111121.
- net at Приемник1111151.: now also Генератор11111151.; no longer Генератор11111141.
- net at Приемник11121.: now also Генератор1111111.; no longer Генератор1111121.
- net at Генератор1111111.: now also Приемник11111.; no longer Приемник11121.
- net at Приемник11111.: now also Генератор11111.; no longer Генератор1111111.
- net at Генератор11111.: now also И111.; no longer Приемник11111.
- net at Приемник1111121.: now also Генератор11111111.; no longer Генератор111111121.
- net at Генератор11111111.: now also Приемник11111111.; no longer Приемник1111121.
- net at Генератор111111111.: now also Приемник1111111.; no longer Приемник11111111.
- net at Генератор11111171.: now also Приемник1111181.; no longer Приемник1111171.
- net at Приемник1111181.: now also Генератор11111181.; no longer Генератор11111171.
- net at Генератор11111151.: now also Приемник1111161.; no longer Приемник1111151.
- net at Приемник1111161.: now also Генератор11111161.; no longer Генератор11111151.
- new net: Генератор11111131., Приемник1111131.
- new net: Генератор11111191., Приемник11111101.
- new net: Генератор11111121., Приемник11111121.
- new net: Генератор11111141., Приемник1111151.
- new net: Генератор1111121., Приемник11121.
- new net: Генератор111111111., Приемник11111111.
- new net: Генератор11111171., Приемник1111171.
Changed lines of the file:
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@@
 (kicad_sch
-	(version 20231120)
+	(version 20250114)
 	(generator "eeschema")
-	(generator_version "8.0")
+	(generator_version "9.0")
 	(paper "A3")
 	(title_block
@@
 		(comment 3 "Бузунова")
 	)
+	(text "НА ЛИСТ 15"
+		(exclude_from_sim no)
+		(at 191.77 219.71 90)
+		(effects
+			(font
+				(size 2 2)
+			)
+		)
+	)
+	(text "НА ЛИСТ 15\nИ НА ЭТОМ ЛИСТЕ"
+		(exclude_from_sim no)
+		(at 344.17 220.98 90)
+		(effects
+			(font
+				(size 2 2)
+			)
+			(justify top)
+		)
+	)
+	(text "НА ЭТОМ ЛИСТЕ"
+		(exclude_from_sim no)
+		(at 30.48 114.3 90)
+		(effects
+			(font
+				(size 2 2)
+			)
+		)
+	)
+	(text "Станция Б"
+		(exclude_from_sim no)
+		(at 396 11 0)
+		(effects
+			(font
+				(size 2 2)
+			)
+		)
+	)
+	(text "Станция А"
+		(exclude_from_sim no)
+		(at 35 11 0)
+		(effects
+			(font
+				(size 2 2)
+			)
+		)
+	)
 	(junction
 		(at 285.75 95.25)
@@
 		)
 	)
-	(text "НА ЛИСТ 15"
-		(exclude_from_sim no)
-		(at 191.77 219.71 90)
-		(effects
-			(font
-				(size 2 2)
-			)
-		)
-	)
-	(text "НА ЛИСТ 15\nИ НА ЭТОМ ЛИСТЕ"
-		(exclude_from_sim no)
-		(at 344.17 220.98 90)
-		(effects
-			(font
-				(size 2 2)
-			)
-			(justify top)
-		)
-	)
-	(text "НА ЭТОМ ЛИСТЕ"
-		(exclude_from_sim no)
-		(at 30.48 114.3 90)
-		(effects
-			(font
-				(size 2 2)
-			)
-		)
-	)
-	(text "Станция Б"
-		(exclude_from_sim no)
-		(at 396 11 0)
-		(effects
-			(font
-				(size 2 2)
-			)
-		)
-	)
-	(text "Станция А"
-		(exclude_from_sim no)
-		(at 35 11 0)
-		(effects
-			(font
-				(size 2 2)
-			)
-		)
-	)
 	(label "ЦП"
 		(at 38.1 165.1 0)
@@
 	)
 	(symbol
-		(lib_id "SCB_Relay:Контакт_нейтрального_якоря_НЗ")
+		(lib_name "Контакт_нейтрального_якоря_НЗ_бн_9")
+		(lib_id "SCB_Legacy:Контакт_нейтрального_якоря_НЗ_бн")
 		(at 69.85 165.1 0)
 		(mirror y)
@@
 	)
 	(symbol
-		(lib_name "SCB_АБТЦ:Генератор_Нитки")
 		(lib_id "SCB_АБТЦ:Генератор_Нитки")
 		(at 225 25 180)
@@
 	)
 	(symbol
-		(lib_name "SCB_Relay:Контакт_нейтрального_якоря_НЗ")
-		(lib_id "SCB_Relay:Контакт_нейтрального_якоря_НЗ")
+		(lib_name "Контакт_нейтрального_якоря_НЗ_бн_7")
+		(lib_id "SCB_Legacy:Контакт_нейтрального_якоря_НЗ_бн")
 		(at 196.85 120.65 0)
 		(mirror y)
@@
 	)
 	(symbol
-		(lib_name "SCB_АБТЦ:Приемник_Нитки")
 		(lib_id "SCB_АБТЦ:Приемник_Нитки")
 		(at 365 25 180)
@@
 	)
 	(symbol
-		(lib_name "SCB_АБТЦ:Приемник_Нитки")
 		(lib_id "SCB_АБТЦ:Приемник_Нитки")
 		(at 190 25 180)
@@
 	)
 	(symbol
-		(lib_name "SCB_АБТЦ:Генератор_Нитки")
 		(lib_id "SCB_АБТЦ:Генератор_Нитки")
 		(at 245 25 180)
@@
 	)
 	(symbol
-		(lib_name "SCB_Relay:Контакт_нейтрального_якоря_НЗ")
-		(lib_id "SCB_Relay:Контакт_нейтрального_якоря_НЗ")
+		(lib_name "Контакт_нейтрального_якоря_НЗ_бн_4")
+		(lib_id "SCB_Legacy:Контакт_нейтрального_якоря_НЗ_бн")
 		(at 146.05 120.65 0)
 		(mirror y)
@@
 	)
 	(symbol
-		(lib_name "SCB_Relay:Контакт_нейтрального_якоря_НЗ")
-		(lib_id "SCB_Relay:Контакт_нейтрального_якоря_НЗ")
+		(lib_name "Контакт_нейтрального_якоря_НЗ_бн_8")
+		(lib_id "SCB_Legacy:Контакт_нейтрального_якоря_НЗ_бн")
 		(at 196.85 69.85 0)
 		(mirror y)
@@
 	)
 	(symbol
-		(lib_name "SCB_Relay:Контакт_нейтрального_якоря_НЗ")
-		(lib_id "SCB_Relay:Контакт_нейтрального_якоря_НЗ")
+		(lib_name "Контакт_нейтрального_якоря_НЗ_бн_3")
+		(lib_id "SCB_Legacy:Контакт_нейтрального_якоря_НЗ_бн")
 		(at 95.25 120.65 0)
 		(mirror y)
@@
 	)
 	(symbol
-		(lib_name "SCB_АБТЦ:Приемник_Нитки")
 		(lib_id "SCB_АБТЦ:Приемник_Нитки")
 		(at 95 25 180)
@@
 	)
 	(symbol
-		(lib_name "SCB_АБТЦ:Генератор_Нитки")
 		(lib_id "SCB_АБТЦ:Генератор_Нитки")
 		(at 105 25 180)
@@
 	)
 	(symbol
-		(lib_name "SCB_Relay:Контакт_нейтрального_якоря_НЗ")
-		(lib_id "SCB_Relay:Контакт_нейтрального_якоря_НЗ")
+		(lib_name "Контакт_нейтрального_якоря_НЗ_бн_10")
+		(lib_id "SCB_Legacy:Контакт_нейтрального_якоря_НЗ_бн")
 		(at 95.25 69.85 0)
 		(mirror y)
@@
 	)
 	(symbol
-		(lib_id "SCB_Relay:Контакт_нейтрального_якоря")
+		(lib_id "SCB_Legacy:Контакт_нейтрального_якоря_бн")
 		(at 222.25 120.65 0)
 		(mirror y)
@@
 	)
 	(symbol
-		(lib_name "SCB_АБТЦ:Приемник_Нитки")
 		(lib_id "SCB_АБТЦ:Приемник_Нитки")
 		(at 75 25 180)
@@
 	)
 	(symbol
-		(lib_name "SCB_АБТЦ:Приемник_Нитки")
 		(lib_id "SCB_АБТЦ:Приемник_Нитки")
 		(at 345 25 180)
@@
 	)
 	(symbol
-		(lib_name "SCB_АБТЦ:Приемник_Нитки")
 		(lib_id "SCB_АБТЦ:Приемник_Нитки")
 		(at 170 25 180)
@@
 	)
 	(symbol
-		(lib_name "SCB_АБТЦ:Генератор_Нитки")
 		(lib_id "SCB_АБТЦ:Генератор_Нитки")
 		(at 200 25 180)
@@
 	)
 	(symbol
-		(lib_name "SCB_АБТЦ:Генератор_Нитки")
 		(lib_id "SCB_АБТЦ:Генератор_Нитки")
 		(at 130 25 180)
@@
 	)
 	(symbol
-		(lib_name "SCB_Relay:Контакт_нейтрального_якоря_НЗ")
-		(lib_id "SCB_Relay:Контакт_нейтрального_якоря_НЗ")
+		(lib_name "Контакт_нейтрального_якоря_НЗ_бн_12")
+		(lib_id "SCB_Legacy:Контакт_нейтрального_якоря_НЗ_бн")
 		(at 146.05 165.1 0)
 		(mirror y)
@@
 	)
 	(symbol
-		(lib_name "SCB_АБТЦ:Генератор_Нитки")
 		(lib_id "SCB_АБТЦ:Генератор_Нитки")
 		(at 310 25 180)
@@
 	)
 	(symbol
-		(lib_name "SCB:Изостык")
 		(lib_id "SCB:Изостык")
 		(at 385 25 180)
@@
 	)
 	(symbol
-		(lib_name "SCB_АБТЦ:Приемник_Нитки")
 		(lib_id "SCB_АБТЦ:Приемник_Нитки")
 		(at 255 25 180)
@@
 	)
 	(symbol
-		(lib_name "SCB_АБТЦ:Приемник_Нитки")
 		(lib_id "SCB_АБТЦ:Приемник_Нитки")
 		(at 140 25 180)
@@
 	)
 	(symbol
-		(lib_name "SCB_АБТЦ:Генератор_Нитки")
 		(lib_id "SCB_АБТЦ:Генератор_Нитки")
 		(at 180 25 180)
@@
 	)
 	(symbol
-		(lib_name "SCB_Relay:Контакт_нейтрального_якоря_НЗ")
-		(lib_id "SCB_Relay:Контакт_нейтрального_якоря_НЗ")
+		(lib_name "Контакт_нейтрального_якоря_НЗ_бн_5")
+		(lib_id "SCB_Legacy:Контакт_нейтрального_якоря_НЗ_бн")
 		(at 247.65 69.85 0)
 		(unit 2)
@@
 	)
 	(symbol
-		(lib_name "SCB_АБТЦ:Генератор_Нитки")
 		(lib_id "SCB_АБТЦ:Генератор_Нитки")
 		(at 85 25 180)
@@
 	)
 	(symbol
-		(lib_name "SCB_Relay:Контакт_нейтрального_якоря_НЗ")
-		(lib_id "SCB_Relay:Контакт_нейтрального_якоря_НЗ")
+		(lib_name "Контакт_нейтрального_якоря_НЗ_бн_2")
+		(lib_id "SCB_Legacy:Контакт_нейтрального_якоря_НЗ_бн")
 		(at 146.05 69.85 0)
 		(mirror y)
@@
 	)
 	(symbol
-		(lib_name "SCB_АБТЦ:Генератор_Нитки")
 		(lib_id "SCB_АБТЦ:Генератор_Нитки")
 		(at 355 25 180)
@@
 	)
 	(symbol
-		(lib_name "SCB_АБТЦ:Генератор_Нитки")
 		(lib_id "SCB_АБТЦ:Генератор_Нитки")
 		(at 150 25 180)
@@
 	)
 	(symbol
-		(lib_name "SCB_АБТЦ:Приемник_Нитки")
 		(lib_id "SCB_АБТЦ:Приемник_Нитки")
 		(at 300 25 180)
@@
 	)
 	(symbol
-		(lib_name "SCB_Relay:Контакт_нейтрального_якоря_НЗ")
-		(lib_id "SCB_Relay:Контакт_нейтрального_якоря_НЗ")
+		(lib_name "Контакт_нейтрального_якоря_НЗ_бн_6")
+		(lib_id "SCB_Legacy:Контакт_нейтрального_якоря_НЗ_бн")
 		(at 95.25 165.1 0)
 		(mirror y)
@@
 	)
 	(symbol
-		(lib_name "SCB_Relay:Контакт_нейтрального_якоря")
-		(lib_id "SCB_Relay:Контакт_нейтрального_якоря")
+		(lib_name "Контакт_нейтрального_якоря_бн_2")
+		(lib_id "SCB_Legacy:Контакт_нейтрального_якоря_бн")
 		(at 120.65 69.85 0)
 		(mirror y)
@@
 	)
 	(symbol
-		(lib_name "SCB_АБТЦ:Генератор_Нитки")
 		(lib_id "SCB_АБТЦ:Генератор_Нитки")
 		(at 375 25 180)
@@
 	)
 	(symbol
-		(lib_name "SCB_АБТЦ:Генератор_Нитки")
 		(lib_id "SCB_АБТЦ:Генератор_Нитки")
 		(at 265 25 180)
@@
 	)
 	(symbol
-		(lib_name "SCB_Relay:Контакт_нейтрального_якоря_НЗ")
-		(lib_id "SCB_Relay:Контакт_нейтрального_якоря_НЗ")
+		(lib_name "Контакт_нейтрального_якоря_НЗ_бн_13")
+		(lib_id "SCB_Legacy:Контакт_нейтрального_якоря_НЗ_бн")
 		(at 323.85 165.1 0)
 		(mirror y)
@@
 	)
 	(symbol
-		(lib_name "SCB_АБТЦ:Генератор_Нитки")
 		(lib_id "SCB_АБТЦ:Генератор_Нитки")
 		(at 335 25 180)
@@
 	)
 	(symbol
-		(lib_name "SCB_Relay:Контакт_нейтрального_якоря_НЗ")
-		(lib_id "SCB_Relay:Контакт_нейтрального_якоря_НЗ")
+		(lib_id "SCB_Legacy:Контакт_нейтрального_якоря_НЗ_бн")
 		(at 120.65 165.1 0)
 		(mirror y)
@@
 	)
 	(symbol
-		(lib_name "SCB:Изостык")
 		(lib_id "SCB:Изостык")
 		(at 55 25 0)
@@
 	)
 	(symbol
-		(lib_name "SCB_АБТЦ:Приемник_Нитки")
 		(lib_id "SCB_АБТЦ:Приемник_Нитки")
 		(at 120 25 180)
@@
 	)
 	(symbol
-		(lib_name "SCB_АБТЦ:Приемник_Нитки")
 		(lib_id "SCB_АБТЦ:Приемник_Нитки")
 		(at 320 25 180)
@@
 	)
 	(symbol
-		(lib_name "SCB_Relay:Контакт_нейтрального_якоря")
-		(lib_id "SCB_Relay:Контакт_нейтрального_якоря")
+		(lib_name "Контакт_нейтрального_якоря_бн_1")
+		(lib_id "SCB_Legacy:Контакт_нейтрального_якоря_бн")
 		(at 120.65 120.65 0)
 		(mirror y)
@@
 	)
 	(symbol
-		(lib_name "SCB_АБТЦ:Приемник_Нитки")
 		(lib_id "SCB_АБТЦ:Приемник_Нитки")
 		(at 215 25 180)
@@
 	)
 	(symbol
-		(lib_name "SCB_АБТЦ:Приемник_Нитки")
 		(lib_id "SCB_АБТЦ:Приемник_Нитки")
 		(at 275 25 180)
@@
 	)
 	(symbol
-		(lib_name "SCB_АБТЦ:Генератор_Нитки")
 		(lib_id "SCB_АБТЦ:Генератор_Нитки")
 		(at 65 25 180)
@@
 	)
 	(symbol
-		(lib_name "SCB_АБТЦ:Приемник_Нитки")
 		(lib_id "SCB_АБТЦ:Приемник_Нитки")
 		(at 235 25 180)
@@
 	)
 	(symbol
-		(lib_name "SCB_АБТЦ:Генератор_Нитки")
 		(lib_id "SCB_АБТЦ:Генератор_Нитки")
 		(at 290 25 180)
@@
 	)
 	(symbol
-		(lib_name "SCB_Relay:Контакт_нейтрального_якоря_НЗ")
-		(lib_id "SCB_Relay:Контакт_нейтрального_якоря_НЗ")
+		(lib_name "Контакт_нейтрального_якоря_НЗ_бн_1")
+		(lib_id "SCB_Legacy:Контакт_нейтрального_якоря_НЗ_бн")
 		(at 222.25 69.85 0)
 		(mirror y)
@@
 	)
 	(symbol
-		(lib_name "SCB_Relay:Контакт_нейтрального_якоря_НЗ")
-		(lib_id "SCB_Relay:Контакт_нейтрального_якоря_НЗ")
+		(lib_name "Контакт_нейтрального_якоря_НЗ_бн_11")
+		(lib_id "SCB_Legacy:Контакт_нейтрального_якоря_НЗ_бн")
 		(at 349.25 165.1 0)
 		(mirror y)
