File: example/АБТЦ-2003/Схемы/предвходной.kicad_sch (KiCad schematic)
At the start: 34 parts

Commit message: Шаблон АБТЦ обновлен
Parts:
- R15: Тип C5-35В -> (none)

Commit message: Обновление примера
Parts:
- Н1, Н11, Н111, Н1111, Н11111, Н111111, Н1111111, Н11111111, Н111111111: symbol SCB_Relay:Контакт_нейтрального_якоря_НЗ -> SCB_Legacy:Контакт_нейтрального_якоря_НЗ_бн
- Н1, Н11, Н111, Н1111, Н11111, Н111111, Н1111111, Н11111111, Н111111111, Н1111111111: symbol SCB_Relay:Контакт_нейтрального_якоря -> SCB_Legacy:Контакт_нейтрального_якоря_бн
