File: example/АБТЦ-2003/Схемы/Л1-2.kicad_sch (KiCad schematic)
At the start: 107 parts

Commit message: Шаблон АБТЦ обновлен
Parts:
- removed Генератор11111, Генератор1111111, Генератор111111101, Генератор11111111, Генератор111111111, Генератор111111121, Генератор11111121, Генератор11111131, Генератор11111141, Генератор11111151, Генератор11111161, Генератор11111171, Генератор11111181, Генератор11111191, Генератор1111121: ~, symbol SCB:Генератор_Нитки
- removed Приемник11111, Приемник11111101, Приемник1111111, Приемник11111111, Приемник11111121, Приемник1111121, Приемник1111131, Приемник1111141, Приемник1111151, Приемник1111161, Приемник1111171, Приемник1111181, Приемник1111191, Приемник11121: ~, symbol SCB:Приемник_Нитки
- removed УКСПС111, УКСПС112: ~, symbol SCB:УКСПС
- added Генератор11111, Генератор1111111, Генератор111111101, Генератор11111111, Генератор111111111, Генератор111111121, Генератор11111121, Генератор11111131, Генератор11111141, Генератор11111151, Генератор11111161, Генератор11111171, Генератор11111181, Генератор11111191, Генератор1111121: ~, symbol SCB_АБТЦ:Генератор_Нитки
- added Приемник11111, Приемник11111101, Приемник1111111, Приемник11111111, Приемник11111121, Приемник1111121, Приемник1111131, Приемник1111141, Приемник1111151, Приемник1111161, Приемник1111171, Приемник1111181, Приемник1111191, Приемник11121: ~, symbol SCB_АБТЦ:Приемник_Нитки
- added УКСПС111 (x2): ~, symbol SCB:УКСПС
Connections:
- net at И111. (привязка): now also Генератор11111.; no longer Светофор111. (привязка)
- net at УКСПС131. (привязка): no longer Светофор1211. (привязка)
- net at УКСПС121. (привязка): no longer Светофор11131. (привязка)
- new net: Генератор1111121., Приемник1111111.
- new net: Генератор1111121., Приемник11121.
- new net: Генератор11111121., Приемник1111131.
- new net: Генератор11111131., Приемник1111131.
- new net: Генератор111111111., Приемник1111111.
- new net: Генератор111111111., Приемник11111111.
- new net: Генератор11111121., Приемник11111121.
- new net: Генератор111111121., Приемник11111121.
- new net: Генератор11111111., Приемник11111111.
- new net: Генератор11111111., Приемник1111121.
- new net: Генератор11111171., Приемник1111171.
- new net: Генератор11111171., Приемник1111181.
- new net: Генератор11111191., Приемник11111101.
- new net: Генератор11111191., Приемник1111191.
- new net: Генератор111111101., Приемник11111101.
- new net: Генератор111111101., И1111. (привязка)
- new net: Генератор11111161., Приемник1111171.
- new net: Генератор11111181., Приемник1111181.
- new net: Генератор11111181., Приемник1111191.
- new net: Генератор111111121., Приемник1111121.
- new net: Генератор11111161., Приемник1111161.
- new net: Генератор1111111., Приемник11111.
- new net: Генератор1111111., Приемник11121.
- new net: Генератор11111141., Приемник1111141.
- new net: Генератор11111141., Приемник1111151.
- new net: Генератор11111., Приемник11111.
- new net: Генератор11111151., Приемник1111161.
- new net: Генератор11111151., Приемник1111151.
- new net: Генератор11111131., Приемник1111141.
- now unconnected: И1111. (привязка)

Commit message: Обновление примера
Parts:
- Н1, Н11, Н111, Н1111, Н11111, Н111111, Н112, Н1121, Н12, Н121, Н1221, Н13, Н141: symbol SCB_Relay:Контакт_нейтрального_якоря_НЗ -> SCB_Legacy:Контакт_нейтрального_якоря_НЗ_бн
- Н1, Н111, Н1111, Н1121, Н11211, Н12, Н122, Н14: symbol SCB_Relay:Контакт_нейтрального_якоря -> SCB_Legacy:Контакт_нейтрального_якоря_бн
Connections:
- net at Генератор1111121.: now also Приемник11121.; no longer Приемник1111111.
- net at Приемник11121.: now also Генератор1111111.; no longer Генератор1111121.
- net at Приемник1111131.: now also Генератор11111131.; no longer Генератор11111121.
- net at Генератор11111131.: now also Приемник1111141.; no longer Приемник1111131.
- net at Генератор11111171.: now also Приемник1111181.; no longer Приемник1111171.
- net at Приемник1111181.: now also Генератор11111181.; no longer Генератор11111171.
- net at Генератор11111191.: now also Приемник1111191.; no longer Приемник11111101.
- net at Приемник1111191.: now also Генератор11111181.; no longer Генератор11111191.
- net at И111.: now also Генератор11111.
- net at Генератор11111.: now also Приемник11111.; no longer И111. (привязка)
- net at Генератор11111141.: now also Приемник1111151.; no longer Приемник1111141.
- net at Приемник1111151.: now also Генератор11111151.; no longer Генератор11111141.
- new net: Генератор1111121., Приемник1111111.
- new net: Генератор11111121., Приемник1111131.
- new net: Генератор11111171., Приемник1111171.
- new net: Генератор11111191., Приемник11111101.
- new net: Генератор1111111., Приемник11111.
- new net: Генератор11111141., Приемник1111141.

Commit message: Поправлены ссылки
Parts:
- П1, П11, П111: symbol SCB_Relay:Контакт_поляризованного_якоря -> SCB_Legacy:Контакт_поляризованного_якоря
Connections:
- net at Генератор1111121.: now also Приемник11121.; no longer Приемник1111111.
- net at Приемник11121.: now also Генератор1111111.; no longer Генератор1111121.
- net at Приемник1111131.: now also Генератор11111131.; no longer Генератор11111121.
- net at Генератор11111131.: now also Приемник1111141.; no longer Приемник1111131.
- net at Генератор11111171.: now also Приемник1111181.; no longer Приемник1111171.
- net at Приемник1111181.: now also Генератор11111181.; no longer Генератор11111171.
- net at Генератор11111191.: now also Приемник1111191.; no longer Приемник11111101.
- net at Приемник1111191.: now also Генератор11111181.; no longer Генератор11111191.
- net at И111.: now also Генератор11111.
- net at Генератор11111.: now also Приемник11111.; no longer И111.
- net at Генератор11111141.: now also Приемник1111151.; no longer Приемник1111141.
- net at Приемник1111151.: now also Генератор11111151.; no longer Генератор11111141.
- new net: Генератор1111121., Приемник1111111.
- new net: Генератор11111121., Приемник1111131.
- new net: Генератор11111171., Приемник1111171.
- new net: Генератор11111191., Приемник11111101.
- new net: Генератор1111111., Приемник11111.
- new net: Генератор11111141., Приемник1111141.
Changed lines of the file:
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@@
 	)
 	(symbol
-		(lib_id "SCB_Relay:Контакт_поляризованного_якоря")
+		(lib_id "SCB_Legacy:Контакт_поляризованного_якоря")
 		(at 306.705 254 0)
 		(unit 1)
@@
 	)
 	(symbol
-		(lib_id "SCB_Relay:Контакт_поляризованного_якоря")
+		(lib_id "SCB_Legacy:Контакт_поляризованного_якоря")
 		(at 141.605 254 0)
 		(unit 1)
@@
 	)
 	(symbol
-		(lib_id "SCB_Relay:Контакт_поляризованного_якоря")
+		(lib_id "SCB_Legacy:Контакт_поляризованного_якоря")
 		(at 332.105 254 0)
 		(unit 1)
@@
 	)
 	(symbol
-		(lib_id "SCB_Relay:Контакт_поляризованного_якоря")
+		(lib_id "SCB_Legacy:Контакт_поляризованного_якоря")
 		(at 167.005 254 0)
 		(unit 1)
