File: example/АБТЦ-2003/Схемы/Л3-4.kicad_sch (KiCad schematic)
At the start: 116 parts

Commit message: Шаблон АБТЦ обновлен
Parts:
- removed Генератор111111, Генератор1111111011, Генератор11111111, Генератор111111111, Генератор1111111111, Генератор1111111211, Генератор111111211, Генератор111111311, Генератор111111411, Генератор111111511, Генератор111111611, Генератор111111711, Генератор111111811, Генератор111111911, Генератор11111211: ~, symbol SCB:Генератор_Нитки
- removed И11111: ~, symbol SCB:Изостык
- removed Приемник111111, Приемник111111011, Приемник11111111, Приемник111111111, Приемник111111211, Приемник11111211, Приемник11111311, Приемник11111411, Приемник11111511, Приемник11111611, Приемник11111711, Приемник11111811, Приемник11111911, Приемник111211: ~, symbol SCB:Приемник_Нитки
- removed Светофор111111, Светофор111211, Светофор111311, Светофор112111, Светофор11311, Светофор12111, Светофор13111: ~, symbol SCB:Светофор
- removed УКСПС1111, УКСПС1121, УКСПС1211, УКСПС1311: ~, symbol SCB:УКСПС
- added Генератор11111, Генератор1111111, Генератор111111101, Генератор11111111, Генератор111111111, Генератор111111121, Генератор11111121, Генератор11111131, Генератор11111141, Генератор11111151, Генератор11111161, Генератор11111171, Генератор11111181, Генератор11111191, Генератор1111121: ~, symbol SCB_АБТЦ:Генератор_Нитки
- added И111: ~, symbol SCB:Изостык
- added Приемник11111, Приемник11111101, Приемник1111111, Приемник11111111, Приемник11111121, Приемник1111121, Приемник1111131, Приемник1111141, Приемник1111151, Приемник1111161, Приемник1111171, Приемник1111181, Приемник1111191, Приемник11121: ~, symbol SCB_АБТЦ:Приемник_Нитки
- added Светофор111, Светофор11121, Светофор11131, Светофор1121, Светофор1131, Светофор121, Светофор131: ~, symbol SCB:Светофор
- added УКСПС111, УКСПС112, УКСПС121, УКСПС131: ~, symbol SCB:УКСПС
- Светофор1111: Литера Ч -> 7
- Светофор11111: Литера 7 -> 5
- Светофор11211: Литера 4 -> 8
- Светофор1211: Литера 9 -> 1
- Светофор1311: Литера 2 -> 10
Connections:
- new net: Генератор1111111., Приемник11121.
- new net: Генератор1111121., Приемник11121.
- new net: Генератор111111111., Приемник11111111.
- new net: Генератор111111111., Приемник1111111.
- new net: Генератор11111121., Приемник1111131.
- new net: Генератор11111131., Приемник1111131.
- new net: Генератор11111171., Приемник1111181.
- new net: Генератор11111171., Приемник1111171.
- new net: Генератор11111141., Приемник1111151.
- new net: Генератор11111151., Приемник1111151.
- new net: Генератор11111121., Приемник11111121.
- new net: Генератор11111161., Приемник1111161.
- new net: Генератор11111151., Приемник1111161.
- new net: Генератор111111121., Приемник11111121.
- new net: Генератор11111., Приемник11111.
- new net: Генератор11111., И111. (привязка)
- new net: Генератор11111111., Приемник11111111.
- new net: Генератор11111141., Приемник1111141.
- new net: Генератор11111131., Приемник1111141.
- new net: Генератор11111111., Приемник1111121.
- new net: Генератор11111181., Приемник1111191.
- new net: Генератор11111181., Приемник1111181.
- new net: Генератор11111161., Приемник1111171.
- new net: Генератор11111191., Приемник1111191.
- new net: Генератор111111101., Приемник11111101.
- new net: Генератор111111101., И1111. (привязка)
- new net: Генератор1111121., Приемник1111111.
- new net: Генератор1111111., Приемник11111.
- new net: Генератор11111191., Приемник11111101.
- new net: Генератор111111121., Приемник1111121.
- now unconnected: И1111. (привязка)

Commit message: Обновление примера
Parts:
- Н1, Н11, Н1113, Н11211, Н121, Н12211, Н14, Н1411, Н14111, Н141111: symbol SCB_Relay:Контакт_нейтрального_якоря -> SCB_Legacy:Контакт_нейтрального_якоря_бн
- Н11, Н11111, Н111111, Н11113, Н11115, Н111151, Н1112, Н11121, Н111211, Н1112111, Н1116, Н1117, Н1121, Н112111, Н1121111, Н11212, Н114, Н1212, Н123, Н1231: symbol SCB_Relay:Контакт_нейтрального_якоря_НЗ -> SCB_Legacy:Контакт_нейтрального_якоря_НЗ_бн
Connections:
- net at Приемник11121.: now also Генератор1111121.; no longer Генератор1111111.
- net at Генератор1111121.: now also Приемник1111111.; no longer Приемник11121.
- net at Генератор111111111.: now also Приемник1111111.; no longer Приемник11111111.
- net at Приемник1111131.: now also Генератор11111131.; no longer Генератор11111121.
- net at Генератор11111131.: now also Приемник1111141.; no longer Приемник1111131.
- net at Генератор11111171.: now also Приемник1111171.; no longer Приемник1111181.
- net at Приемник1111171.: now also Генератор11111161.; no longer Генератор11111171.
- net at Приемник1111151.: now also Генератор11111151.; no longer Генератор11111141.
- net at Генератор11111151.: now also Приемник1111161.; no longer Приемник1111151.
- net at Генератор11111.: now also И111.; no longer Приемник11111.
- net at И111.: no longer Генератор11111.
- net at Генератор11111181.: now also Приемник1111181.; no longer Приемник1111191.
- net at Генератор111111101.: now also И1111.; no longer Приемник11111101.
- net at И1111.: no longer Генератор111111101.
- new net: Генератор1111111., Приемник11121.
- new net: Генератор111111111., Приемник11111111.
- new net: Генератор11111121., Приемник1111131.
- new net: Генератор11111171., Приемник1111181.
- new net: Генератор11111141., Приемник1111151.
- new net: Генератор11111161., Приемник1111161.
- new net: Генератор11111., Приемник11111.
- new net: Генератор11111181., Приемник1111191.
- new net: Генератор111111101., Приемник11111101.

Commit message: Поправлены ссылки
Parts:
- П11, П111, П1111, П11111: symbol SCB_Relay:Контакт_поляризованного_якоря_П -> SCB_Legacy:Контакт_поляризованного_якоря_П
Connections:
- net at Приемник11121.: now also Генератор1111121.; no longer Генератор1111111.
- net at Генератор1111121.: now also Приемник1111111.; no longer Приемник11121.
- net at Генератор111111111.: now also Приемник1111111.; no longer Приемник11111111.
- net at Приемник1111131.: now also Генератор11111131.; no longer Генератор11111121.
- net at Генератор11111131.: now also Приемник1111141.; no longer Приемник1111131.
- net at Генератор11111171.: now also Приемник1111171.; no longer Приемник1111181.
- net at Приемник1111171.: now also Генератор11111161.; no longer Генератор11111171.
- net at Приемник1111151.: now also Генератор11111151.; no longer Генератор11111141.
- net at Генератор11111151.: now also Приемник1111161.; no longer Приемник1111151.
- net at Генератор11111.: now also И111.; no longer Приемник11111.
- net at И111.: no longer Генератор11111.
- net at Генератор11111181.: now also Приемник1111181.; no longer Приемник1111191.
- net at Генератор111111101.: now also И1111.; no longer Приемник11111101.
- net at И1111.: no longer Генератор111111101.
- new net: Генератор1111111., Приемник11121.
- new net: Генератор111111111., Приемник11111111.
- new net: Генератор11111121., Приемник1111131.
- new net: Генератор11111171., Приемник1111181.
- new net: Генератор11111141., Приемник1111151.
- new net: Генератор11111161., Приемник1111161.
- new net: Генератор11111., Приемник11111.
- new net: Генератор11111181., Приемник1111191.
- new net: Генератор111111101., Приемник11111101.
Changed lines of the file:
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@@
 	)
 	(symbol
-		(lib_id "SCB_Relay:Контакт_поляризованного_якоря_П")
+		(lib_id "SCB_Legacy:Контакт_поляризованного_якоря_П")
 		(at 71.755 139.7 0)
 		(unit 1)
@@
 	)
 	(symbol
-		(lib_id "SCB_Relay:Контакт_поляризованного_якоря_П")
+		(lib_id "SCB_Legacy:Контакт_поляризованного_якоря_П")
 		(at 306.705 254 0)
 		(unit 1)
@@
 	)
 	(symbol
-		(lib_id "SCB_Relay:Контакт_поляризованного_якоря_П")
+		(lib_id "SCB_Legacy:Контакт_поляризованного_якоря_П")
 		(at 97.155 139.7 0)
 		(unit 1)
@@
 	)
 	(symbol
-		(lib_id "SCB_Relay:Контакт_поляризованного_якоря_П")
+		(lib_id "SCB_Legacy:Контакт_поляризованного_якоря_П")
 		(at 167.005 254 0)
 		(unit 1)
@@
 	)
 	(symbol
-		(lib_id "SCB_Relay:Контакт_поляризованного_якоря_П")
+		(lib_id "SCB_Legacy:Контакт_поляризованного_якоря_П")
 		(at 141.605 254 0)
 		(unit 1)
@@
 	)
 	(symbol
-		(lib_id "SCB_Relay:Контакт_поляризованного_якоря_П")
+		(lib_id "SCB_Legacy:Контакт_поляризованного_якоря_П")
 		(at 332.105 254 0)
 		(unit 1)
