File: example/АБТЦ-2003/Схемы/Л7-8.kicad_sch (KiCad schematic)
At the start: 105 parts

Commit message: Шаблон АБТЦ обновлен
Parts:
- removed Генератор1111111, Генератор11111110111, Генератор111111111, Генератор1111111111, Генератор11111111111, Генератор11111112111, Генератор1111112111, Генератор1111113111, Генератор1111114111, Генератор1111115111, Генератор1111116111, Генератор1111117111, Генератор1111118111, Генератор1111119111, Генератор111112111: ~, symbol SCB:Генератор_Нитки
- removed И11111, И111111: ~, symbol SCB:Изостык
- removed Приемник1111110111, Приемник1111111, Приемник111111111, Приемник1111111111, Приемник1111112111, Приемник111112111, Приемник111113111, Приемник111114111, Приемник111115111, Приемник111116111, Приемник111117111, Приемник111118111, Приемник111119111, Приемник1112111: ~, symbol SCB:Приемник_Нитки
- removed Светофор111111, Светофор1111111, Светофор1112111, Светофор1113111, Светофор112111, Светофор1121111, Светофор113111, Светофор12111, Светофор121111, Светофор13111, Светофор131111: ~, symbol SCB:Светофор
- removed УКСПС11111, УКСПС11211, УКСПС12111, УКСПС13111: ~, symbol SCB:УКСПС
- added Генератор11111, Генератор1111111, Генератор111111101, Генератор11111111, Генератор111111111, Генератор111111121, Генератор11111121, Генератор11111131, Генератор11111141, Генератор11111151, Генератор11111161, Генератор11111171, Генератор11111181, Генератор11111191, Генератор1111121: ~, symbol SCB_АБТЦ:Генератор_Нитки
- added И111, И1111: ~, symbol SCB:Изостык
- added Приемник11111, Приемник11111101, Приемник1111111, Приемник11111111, Приемник11111121, Приемник1111121, Приемник1111131, Приемник1111141, Приемник1111151, Приемник1111161, Приемник1111171, Приемник1111181, Приемник1111191, Приемник11121: ~, symbol SCB_АБТЦ:Приемник_Нитки
- added Светофор111, Светофор1111, Светофор11121, Светофор11131, Светофор1121, Светофор11211, Светофор1131, Светофор121, Светофор1211, Светофор131, Светофор1311: ~, symbol SCB:Светофор
- added УКСПС111 (x2), УКСПС121, УКСПС131: ~, symbol SCB:УКСПС
- Светофор11111: Литера Ч -> 5
Connections:
- new net: Генератор11111131., Приемник1111131.
- new net: Генератор11111131., Приемник1111141.
- new net: Генератор11111181., Приемник1111191.
- new net: Генератор11111181., Приемник1111181.
- new net: Генератор1111111., Приемник11121.
- new net: Генератор1111121., Приемник11121.
- new net: Генератор111111101., Приемник11111101.
- new net: Генератор111111101., И1111. (привязка)
- new net: Генератор11111171., Приемник1111171.
- new net: Генератор11111171., Приемник1111181.
- new net: Генератор11111121., Приемник1111131.
- new net: Генератор11111111., Приемник11111111.
- new net: Генератор111111111., Приемник11111111.
- new net: Генератор111111121., Приемник11111121.
- new net: Генератор111111121., Приемник1111121.
- new net: Генератор1111121., Приемник1111111.
- new net: Генератор111111111., Приемник1111111.
- new net: Генератор11111161., Приемник1111161.
- new net: Генератор11111151., Приемник1111161.
- new net: Генератор11111141., Приемник1111151.
- new net: Генератор11111151., Приемник1111151.
- new net: Генератор11111111., Приемник1111121.
- new net: Генератор11111191., Приемник11111101.
- new net: Генератор1111111., Приемник11111.
- new net: Генератор11111., Приемник11111.
- new net: Генератор11111161., Приемник1111171.
- new net: Генератор11111121., Приемник11111121.
- new net: Генератор11111141., Приемник1111141.
- new net: Генератор11111191., Приемник1111191.
- new net: Генератор11111., И111. (привязка)

Commit message: Обновление примера
Parts:
- Н111, Н1111, Н11111, Н111111, Н11131, Н12, Н121: symbol SCB_Relay:Контакт_нейтрального_якоря_НЗ -> SCB_Legacy:Контакт_нейтрального_якоря_НЗ_бн
- Н1111411, Н11114111, Н111311, Н11151, Н112111, Н1121111, Н11211111, Н112111111, Н1121111111, Н1211, Н141: symbol SCB_Relay:Контакт_нейтрального_якоря -> SCB_Legacy:Контакт_нейтрального_якоря_бн
Connections:
- net at Генератор11111131.: now also Приемник1111141.; no longer Приемник1111131.
- net at Приемник1111141.: now also Генератор11111141.; no longer Генератор11111131.
- net at Генератор11111181.: now also Приемник1111181.; no longer Приемник1111191.
- net at Приемник1111181.: now also Генератор11111171.; no longer Генератор11111181.
- net at Приемник11121.: now also Генератор1111121.; no longer Генератор1111111.
- net at Генератор1111121.: now also Приемник1111111.; no longer Приемник11121.
- net at Генератор111111101.: now also И1111.; no longer Приемник11111101.
- net at И1111.: no longer Генератор111111101.
- net at Приемник1111171.: now also Генератор11111161.; no longer Генератор11111171.
- net at Приемник11111111.: now also Генератор111111111.; no longer Генератор11111111.
- net at Генератор111111111.: now also Приемник1111111.; no longer Приемник11111111.
- net at Генератор111111121.: now also Приемник1111121.; no longer Приемник11111121.
- net at Приемник1111121.: now also Генератор11111111.; no longer Генератор111111121.
- net at Приемник1111161.: now also Генератор11111151.; no longer Генератор11111161.
- net at Генератор11111151.: now also Приемник1111151.; no longer Приемник1111161.
- net at И111.: now also Генератор11111.
- new net: Генератор11111131., Приемник1111131.
- new net: Генератор11111181., Приемник1111191.
- new net: Генератор1111111., Приемник11121.
- new net: Генератор111111101., Приемник11111101.
- new net: Генератор11111171., Приемник1111171.
- new net: Генератор11111111., Приемник11111111.
- new net: Генератор111111121., Приемник11111121.
- new net: Генератор11111161., Приемник1111161.
- new net: Генератор11111141., Приемник1111151.

Commit message: Поправлены ссылки
Parts:
- П111, П1111, П11111, П111111, П1111111, П1112, П11211, П112111: symbol SCB_Relay:Контакт_поляризованного_якоря -> SCB_Legacy:Контакт_поляризованного_якоря
Connections:
- net at Генератор11111131.: now also Приемник1111141.; no longer Приемник1111131.
- net at Приемник1111141.: now also Генератор11111141.; no longer Генератор11111131.
- net at Генератор11111181.: now also Приемник1111181.; no longer Приемник1111191.
- net at Приемник1111181.: now also Генератор11111171.; no longer Генератор11111181.
- net at Приемник11121.: now also Генератор1111121.; no longer Генератор1111111.
- net at Генератор1111121.: now also Приемник1111111.; no longer Приемник11121.
- net at Генератор111111101.: now also И1111.; no longer Приемник11111101.
- net at И1111.: no longer Генератор111111101.
- net at Приемник1111171.: now also Генератор11111161.; no longer Генератор11111171.
- net at Приемник11111111.: now also Генератор111111111.; no longer Генератор11111111.
- net at Генератор111111111.: now also Приемник1111111.; no longer Приемник11111111.
- net at Генератор111111121.: now also Приемник1111121.; no longer Приемник11111121.
- net at Приемник1111121.: now also Генератор11111111.; no longer Генератор111111121.
- net at Приемник1111161.: now also Генератор11111151.; no longer Генератор11111161.
- net at Генератор11111151.: now also Приемник1111151.; no longer Приемник1111161.
- net at И111.: now also Генератор11111.
- new net: Генератор11111131., Приемник1111131.
- new net: Генератор11111181., Приемник1111191.
- new net: Генератор1111111., Приемник11121.
- new net: Генератор111111101., Приемник11111101.
- new net: Генератор11111171., Приемник1111171.
- new net: Генератор11111111., Приемник11111111.
- new net: Генератор111111121., Приемник11111121.
- new net: Генератор11111161., Приемник1111161.
- new net: Генератор11111141., Приемник1111151.
Changed lines of the file:
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@@
 	)
 	(symbol
-		(lib_id "SCB_Relay:Контакт_поляризованного_якоря")
+		(lib_id "SCB_Legacy:Контакт_поляризованного_якоря")
 		(at 306.705 158.75 0)
 		(mirror x)
@@
 	)
 	(symbol
-		(lib_id "SCB_Relay:Контакт_поляризованного_якоря")
+		(lib_id "SCB_Legacy:Контакт_поляризованного_якоря")
 		(at 332.105 158.75 0)
 		(mirror x)
@@
 	)
 	(symbol
-		(lib_id "SCB_Relay:Контакт_поляризованного_якоря")
+		(lib_id "SCB_Legacy:Контакт_поляризованного_якоря")
 		(at 306.705 133.35 0)
 		(unit 1)
@@
 	)
 	(symbol
-		(lib_id "SCB_Relay:Контакт_поляризованного_якоря")
+		(lib_id "SCB_Legacy:Контакт_поляризованного_якоря")
 		(at 141.605 133.35 0)
 		(mirror x)
@@
 	)
 	(symbol
-		(lib_id "SCB_Relay:Контакт_поляризованного_якоря")
+		(lib_id "SCB_Legacy:Контакт_поляризованного_якоря")
 		(at 167.005 133.35 0)
 		(mirror x)
@@
 	)
 	(symbol
-		(lib_id "SCB_Relay:Контакт_поляризованного_якоря")
+		(lib_id "SCB_Legacy:Контакт_поляризованного_якоря")
 		(at 332.105 133.35 0)
 		(unit 1)
@@
 	)
 	(symbol
-		(lib_id "SCB_Relay:Контакт_поляризованного_якоря")
+		(lib_id "SCB_Legacy:Контакт_поляризованного_якоря")
 		(at 97.155 171.45 0)
 		(unit 1)
@@
 	)
 	(symbol
-		(lib_id "SCB_Relay:Контакт_поляризованного_якоря")
+		(lib_id "SCB_Legacy:Контакт_поляризованного_якоря")
 		(at 71.755 171.45 0)
 		(unit 1)
