File: example/АБТЦ-2003/Схемы/Схемы.kicad_sch (KiCad schematic)
At the start: 81 parts

Commit message: Шаблон АБТЦ обновлен
Parts:
- Генератор1111, Генератор111111, Генератор1111111, Генератор11111110, Генератор11111111, Генератор11111112, Генератор1111112, Генератор1111113, Генератор1111114, Генератор1111115, Генератор1111116, Генератор1111117, Генератор1111118, Генератор1111119, Генератор111112: symbol SCB:Генератор_Нитки -> SCB_АБТЦ:Генератор_Нитки
- Приемник1111, Приемник111111, Приемник1111110, Приемник1111111, Приемник1111112, Приемник111112, Приемник111113, Приемник111114, Приемник111115, Приемник111116, Приемник111117, Приемник111118, Приемник111119, Приемник1112: symbol SCB:Приемник_Нитки -> SCB_АБТЦ:Приемник_Нитки
Connections:
- net at Приемник111111.: now also Генератор11111111.; no longer Генератор111112.
- net at Генератор11111111.: now also Приемник1111111.; no longer Приемник111111.
- net at Генератор1111118.: now also Приемник111118.; no longer Приемник111119.
- net at Приемник111118.: now also Генератор1111117.; no longer Генератор1111118.
- net at Генератор11111112.: now also Приемник111112.; no longer Приемник1111112.
- net at Приемник111112.: now also Генератор1111111.; no longer Генератор11111112.
- net at И11. (привязка): no longer Светофор11. (привязка)
- net at Генератор1111111.: now also Приемник1111111.; no longer Приемник111112.
- net at УКСПС11. (привязка): no longer Светофор112. (привязка)
- net at УКСПС11. (привязка): no longer Светофор13. (привязка)
- net at Генератор1111.: now also И11. (привязка); no longer Приемник1111.
- net at Генератор1111114.: now also Приемник111115.; no longer Приемник111114.
- net at Приемник111115.: now also Генератор1111115.; no longer Генератор1111114.
- net at Приемник111117.: now also Генератор1111116.; no longer Генератор1111117.
- net at Генератор1111116.: now also Приемник111116.; no longer Приемник111117.
- net at И111. (привязка): now also Генератор11111110.
- net at УКСПС12. (привязка): no longer Светофор1113. (привязка)
- net at УКСПС13. (привязка): no longer Светофор121. (привязка)
- new net: Генератор111112., Приемник111111.
- new net: Генератор1111118., Приемник111119.
- new net: Генератор11111112., Приемник1111112.
- new net: Генератор1111., Приемник1111.
- new net: Генератор1111114., Приемник111114.
- new net: Генератор1111117., Приемник111117.
- new net: Генератор1111115., Приемник111116.
- now unconnected: И11. (привязка)

Commit message: Обновление примера
Parts:
- Н1: symbol SCB_Relay:Контакт_нейтрального_якоря -> SCB_Legacy:Контакт_нейтрального_якоря_бн
- Н1, Н11, Н111, Н1111, Н11111, Н111111, Н1111111, Н1111112, Н111112, Н11112: symbol SCB_Relay:Контакт_нейтрального_якоря_НЗ -> SCB_Legacy:Контакт_нейтрального_якоря_НЗ_бн
Connections:
- net at Приемник111111.: now also Генератор11111111.; no longer Генератор111112.
- net at Генератор11111111.: now also Приемник1111111.; no longer Приемник111111.
- net at Генератор1111118.: now also Приемник111118.; no longer Приемник111119.
- net at Приемник111118.: now also Генератор1111117.; no longer Генератор1111118.
- net at Генератор11111112.: now also Приемник111112.; no longer Приемник1111112.
- net at Приемник111112.: now also Генератор1111111.; no longer Генератор11111112.
- net at Генератор1111111.: now also Приемник1111111.; no longer Приемник111112.
- net at Генератор1111.: now also И11.; no longer Приемник1111.
- net at И11.: no longer Генератор1111.
- net at Генератор1111114.: now also Приемник111115.; no longer Приемник111114.
- net at Приемник111115.: now also Генератор1111115.; no longer Генератор1111114.
- net at Приемник111117.: now also Генератор1111116.; no longer Генератор1111117.
- net at Генератор1111116.: now also Приемник111116.; no longer Приемник111117.
- net at И111.: now also Генератор11111110.
- new net: Генератор111112., Приемник111111.
- new net: Генератор1111118., Приемник111119.
- new net: Генератор11111112., Приемник1111112.
- new net: Генератор1111., Приемник1111.
- new net: Генератор1111114., Приемник111114.
- new net: Генератор1111117., Приемник111117.
- new net: Генератор1111115., Приемник111116.

Commit message: Embed рамки
Connections:
- net at Приемник111111.: now also Генератор11111111.; no longer Генератор111112.
- net at Генератор11111111.: now also Приемник1111111.; no longer Приемник111111.
- net at Генератор1111118.: now also Приемник111118.; no longer Приемник111119.
- net at Приемник111118.: now also Генератор1111117.; no longer Генератор1111118.
- net at Генератор11111112.: now also Приемник111112.; no longer Приемник1111112.
- net at Приемник111112.: now also Генератор1111111.; no longer Генератор11111112.
- net at Генератор1111111.: now also Приемник1111111.; no longer Приемник111112.
- net at Генератор1111.: now also И11.; no longer Приемник1111.
- net at И11.: no longer Генератор1111.
- net at Генератор1111114.: now also Приемник111115.; no longer Приемник111114.
- net at Приемник111115.: now also Генератор1111115.; no longer Генератор1111114.
- net at Приемник111117.: now also Генератор1111116.; no longer Генератор1111117.
- net at Генератор1111116.: now also Приемник111116.; no longer Приемник111117.
- net at И111.: now also Генератор11111110.
- new net: Генератор111112., Приемник111111.
- new net: Генератор1111118., Приемник111119.
- new net: Генератор11111112., Приемник1111112.
- new net: Генератор1111., Приемник1111.
- new net: Генератор1111114., Приемник111114.
- new net: Генератор1111117., Приемник111117.
- new net: Генератор1111115., Приемник111116.
Changed lines of the file:
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@@
 	)
 	(embedded_fonts no)
+	(embedded_files
+		(file
+			(name "КП_МКТ.kicad_wks")
+			(type worksheet)
+			(data |KLUv/WBoIM0nAIZtizBAdTpUIcw/MEEl5UD9vvRxVUaTt7Tdim1NsQHCcIaa6NdKKWWSMk3Fl5PY
+				Ge6GSwSJAG0AhwD9ludlJRB0aTRPj2bLyztxzWxeGSaSIC2v99IsRE8fKpoOBP3ZWQpdVDSzEkYp
+				JmHCaMXIyuJe1igLlSIoxXRQq3gr6ISlMS+LBPrKd3JYJ4qaVKDT8Zgw6DxxFT8Rnwyj1sSMIJk+
+				m2E0lM1rjgQ6HlDs7ubse2HWKZsZAh3P6UIjYiIksi4EArDjY/dOthYZ9rOLcbmxtwuj2PXd7fUy
+				N34NRl+WkSG7993L/v7O9cC35W+wBxblzR3F7LLZmbmS//9a+3bs9qNrGyFs8cHn75zr5rxBurCe
+				o5CJmjBedubqf2WUleyWHt81fN+NTHRZbWlomjwrU7fCSXlnmwpTa6oMTt2PFExNkbGljjzYICwV
+				BTb3qhB33futwQ5JgaRk6om3fMGBMtLUlpf61dtrklChUsdn8t6uhqRYagnLnTREsaxyuK1yqTZV
+				prLUmEpSPZv0mqLdoLDoCcOi8rZfve89YSaKmg8E/alqqkhqpt7Ul8qSs/BZippUgsIekAfU8YDe
+				vXNf5ph5fJWvdLF6sSU/99gebP92zq5V7b4OX0t3/Ptw/8FvZ/4Kuv3XDwsHCq6jc+se7vtDLBQ0
+				KDAYcNtZIbvbto6HXhhF9G3RHSQ8IDw46dyEUdmxmwcAQEfAyobOsgJfjIqL7/KRSnGwdYPu2l9q
+				gUuoIUmqZkaSgqSSNgNRESGMWKeuDnJwGINQCMJwDENSKAcZZwhhxAgKMkRkZEi0A8hZg3bWYlb2
+				h4YoYKGFmekygghKPx7M15IDD7IYd0WZcR9+6xUxAWj38yoXAmC92oZMMfSB1X7rMp20tBrmEBIe
+				hJakM3LW1t3YaQqxwLlbgpwXnM4OLhkcj+VMBQPN2YfN4GDyKLQvgbLaFMHD7rsVHUKT0f1CBDFP
+				XSbe2VB8O79sP6vXCAAfQsfS9FmMsucETSZlwUkkPcQNppQ7TSRxPLsSCN3qj6BnCn09e0/ycEVX
+				3g7wv0CN+KgnLnaDw8y9wQhha3BdLY2v2im89zFrK+VXxtKex5HrauhBrs/tfKi6CNhwPzqzFi3z
+				9U9Sfevn18nGhVF6A8vogOXyMhBb5VwDaXeWAKXYKMLnvwFgs6HSKajyFcrFafcXwJdaG1hIPkiI
+				V/sxYh7nQd22wwlq3PVReFUKBL6a2LzD6KYLdqFI5QQgIR7waZWh9JSLVhZEctJdcwR7A21bB4Hz
+				YfEHf73jPKpiFEOcdpvT9+AQ+tz+oKOKfBl8eLO27y8VJRblwQT7135UnaHRYO7Y2aumWmyLln0M
+				EkEDoZrYI3+aWzQDyapNeKGVQYAECUSWgbsKzB1f7vHwQoUlWbzELbjETzjux+sduNZypQe0pMC3
+				27OXquavENrbkZwas/aMKEFFfiCsrJGJaiGom2yCQx+xet8JSY59VXzJJZZqANQJJJLQ10mk4+Zo
+				KFq0lCRIAwvRiSaVy+NmH7CuRcJ8H5tzH5nMFpPSW2OVDZxoTeXn3khhg88GFYDHgwvheKwMphGy
+				pUNF15jqOumO8hmv3H0Kp2Kv648A3/nhJFgFVZKCoNKJ80sYuikSwx16AEgHvf+okhOf8aBlIYg9
+				C5pjkJDYaAirz+RKmgVKCmny3vo9qWmdnfGSrgI=|
+			)
+			(checksum "3FBF103777E8EE01081CA18737155A0D")
+		)
+	)
 )

Commit message: Поправлены ссылки
Connections:
- net at Приемник111111.: now also Генератор11111111.; no longer Генератор111112.
- net at Генератор11111111.: now also Приемник1111111.; no longer Приемник111111.
- net at Генератор1111118.: now also Приемник111118.; no longer Приемник111119.
- net at Приемник111118.: now also Генератор1111117.; no longer Генератор1111118.
- net at Генератор11111112.: now also Приемник111112.; no longer Приемник1111112.
- net at Приемник111112.: now also Генератор1111111.; no longer Генератор11111112.
- net at Генератор1111111.: now also Приемник1111111.; no longer Приемник111112.
- net at Генератор1111.: now also И11.; no longer Приемник1111.
- net at И11.: no longer Генератор1111.
- net at Генератор1111114.: now also Приемник111115.; no longer Приемник111114.
- net at Приемник111115.: now also Генератор1111115.; no longer Генератор1111114.
- net at Приемник111117.: now also Генератор1111116.; no longer Генератор1111117.
- net at Генератор1111116.: now also Приемник111116.; no longer Приемник111117.
- net at И111.: now also Генератор11111110.
- new net: Генератор111112., Приемник111111.
- new net: Генератор1111118., Приемник111119.
- new net: Генератор11111112., Приемник1111112.
- new net: Генератор1111., Приемник1111.
- new net: Генератор1111114., Приемник111114.
- new net: Генератор1111117., Приемник111117.
- new net: Генератор1111115., Приемник111116.
Changed lines of the file:
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@@
 	)
 	(symbol
+		(lib_name "Приемник_Нитки_1")
 		(lib_id "SCB_АБТЦ:Приемник_Нитки")
 		(at 120 25 180)
@@
 	)
 	(symbol
+		(lib_name "Генератор_Нитки_1")
 		(lib_id "SCB_АБТЦ:Генератор_Нитки")
 		(at 335 25 180)
@@
 	)
 	(symbol
+		(lib_name "Приемник_Нитки_2")
 		(lib_id "SCB_АБТЦ:Приемник_Нитки")
 		(at 345 25 180)
@@
 	)
 	(symbol
+		(lib_name "Приемник_Нитки_3")
 		(lib_id "SCB_АБТЦ:Приемник_Нитки")
 		(at 190 25 180)
@@
 	)
 	(symbol
+		(lib_name "Лампа_1")
 		(lib_id "SCB_Relay:Лампа")
 		(at 355.6 88.9 0)
@@
 	)
 	(symbol
+		(lib_name "Генератор_Нитки_2")
 		(lib_id "SCB_АБТЦ:Генератор_Нитки")
 		(at 355 25 180)
@@
 	)
 	(symbol
+		(lib_name "Приемник_Нитки_4")
 		(lib_id "SCB_АБТЦ:Приемник_Нитки")
 		(at 365 25 180)
@@
 	)
 	(symbol
+		(lib_name "Лампа_2")
 		(lib_id "SCB_Relay:Лампа")
 		(at 355.6 99.06 0)
@@
 	)
 	(symbol
+		(lib_name "Нейтральное_1")
 		(lib_id "SCB_Relay:Нейтральное")
 		(at 63.5 88.9 0)
@@
 	)
 	(symbol
+		(lib_name "Генератор_Нитки_3")
 		(lib_id "SCB_АБТЦ:Генератор_Нитки")
 		(at 200 25 180)
@@
 	)
 	(symbol
+		(lib_name "Светофор_1")
 		(lib_id "SCB:Светофор")
 		(at 55 15 0)
@@
 	)
 	(symbol
+		(lib_name "Генератор_Нитки_4")
 		(lib_id "SCB_АБТЦ:Генератор_Нитки")
 		(at 150 25 180)
@@
 	)
 	(symbol
+		(lib_name "УКСПС_1")
 		(lib_id "SCB:УКСПС")
 		(at 204 25 0)
@@
 	)
 	(symbol
+		(lib_name "УКСПС_2")
 		(lib_id "SCB:УКСПС")
 		(at 109 25 0)
@@
 	)
 	(symbol
+		(lib_name "Нейтральное_2")
 		(lib_id "SCB_Relay:Нейтральное")
 		(at 63.5 165.1 0)
@@
 	)
 	(symbol
+		(lib_name "Светофор_2")
 		(lib_id "SCB:Светофор")
 		(at 249 15 0)
@@
 	)
 	(symbol
+		(lib_name "Светофор_3")
 		(lib_id "SCB:Светофор")
 		(at 101 32 180)
@@
 	)
 	(symbol
+		(lib_name "Генератор_Нитки_6")
 		(lib_id "SCB_АБТЦ:Генератор_Нитки")
 		(at 65 25 180)
@@
 	)
 	(symbol
+		(lib_name "Приемник_Нитки_5")
 		(lib_id "SCB_АБТЦ:Приемник_Нитки")
 		(at 75 25 180)
@@
 	)
 	(symbol
+		(lib_name "Генератор_Нитки_5")
 		(lib_id "SCB_АБТЦ:Генератор_Нитки")
 		(at 245 25 180)
@@
 	)
 	(symbol
+		(lib_name "Приемник_Нитки_6")
 		(lib_id "SCB_АБТЦ:Приемник_Нитки")
 		(at 300 25 180)
@@
 	)
 	(symbol
+		(lib_name "Генератор_Нитки_7")
 		(lib_id "SCB_АБТЦ:Генератор_Нитки")
 		(at 105 25 180)
@@
 	)
 	(symbol
+		(lib_name "Изостык_1")
 		(lib_id "SCB:Изостык")
 		(at 385 25 180)
@@
 	)
 	(symbol
+		(lib_name "Лампа_3")
 		(lib_id "SCB_Relay:Лампа")
 		(at 63.5 50.8 0)
@@
 	)
 	(symbol
+		(lib_name "Светофор_4")
 		(lib_id "SCB:Светофор")
 		(at 241 32 180)
@@
 	)
 	(symbol
+		(lib_name "Генератор_Нитки_8")
 		(lib_id "SCB_АБТЦ:Генератор_Нитки")
 		(at 375 25 180)
@@
 	)
 	(symbol
+		(lib_name "Генератор_Нитки_9")
 		(lib_id "SCB_АБТЦ:Генератор_Нитки")
 		(at 85 25 180)
@@
 	)
 	(symbol
+		(lib_name "Нейтральное_3")
 		(lib_id "SCB_Relay:Нейтральное")
 		(at 279.4 190.5 0)
@@
 	)
 	(symbol
+		(lib_name "Приемник_Нитки_7")
 		(lib_id "SCB_АБТЦ:Приемник_Нитки")
 		(at 320 25 180)
@@
 	)
 	(symbol
+		(lib_name "Светофор_5")
 		(lib_id "SCB:Светофор")
 		(at 286 32 180)
@@
 	)
 	(symbol
+		(lib_name "Генератор_Нитки_10")
 		(lib_id "SCB_АБТЦ:Генератор_Нитки")
 		(at 265 25 180)
@@
 	)
 	(symbol
+		(lib_name "Светофор_6")
 		(lib_id "SCB:Светофор")
 		(at 385 32 180)
@@
 	)
 	(symbol
+		(lib_name "Приемник_Нитки_8")
 		(lib_id "SCB_АБТЦ:Приемник_Нитки")
 		(at 170 25 180)
@@
 	)
 	(symbol
+		(lib_name "Светофор_7")
 		(lib_id "SCB:Светофор")
 		(at 339 15 0)
@@
 	)
 	(symbol
+		(lib_name "Светофор_8")
 		(lib_id "SCB:Светофор")
 		(at 294 15 0)
@@
 	)
 	(symbol
+		(lib_name "Генератор_Нитки_11")
 		(lib_id "SCB_АБТЦ:Генератор_Нитки")
 		(at 130 25 180)
@@
 	)
 	(symbol
+		(lib_name "Светофор_9")
 		(lib_id "SCB:Светофор")
 		(at 109 15 0)
@@
 	)
 	(symbol
+		(lib_name "Светофор_10")
 		(lib_id "SCB:Светофор")
 		(at 196 32 180)
@@
 	)
 	(symbol
+		(lib_name "Генератор_Нитки_12")
 		(lib_id "SCB_АБТЦ:Генератор_Нитки")
 		(at 225 25 180)
@@
 	)
 	(symbol
+		(lib_name "Приемник_Нитки_10")
 		(lib_id "SCB_АБТЦ:Приемник_Нитки")
 		(at 95 25 180)
@@
 	)
 	(symbol
+		(lib_name "УКСПС_3")
 		(lib_id "SCB:УКСПС")
 		(at 286 25 0)
@@
 	)
 	(symbol
+		(lib_name "Светофор_11")
 		(lib_id "SCB:Светофор")
 		(at 331 32 180)
@@
 	)
 	(symbol
+		(lib_name "Генератор_Нитки_13")
 		(lib_id "SCB_АБТЦ:Генератор_Нитки")
 		(at 310 25 180)
@@
 	)
 	(symbol
+		(lib_name "Приемник_Нитки_11")
 		(lib_id "SCB_АБТЦ:Приемник_Нитки")
 		(at 275 25 180)
@@
 	)
 	(symbol
+		(lib_name "Приемник_Нитки_9")
 		(lib_id "SCB_АБТЦ:Приемник_Нитки")
 		(at 235 25 180)
@@
 	)
 	(symbol
+		(lib_name "Приемник_Нитки_12")
 		(lib_id "SCB_АБТЦ:Приемник_Нитки")
 		(at 215 25 180)
@@
 	)
 	(symbol
+		(lib_name "Генератор_Нитки_14")
 		(lib_id "SCB_АБТЦ:Генератор_Нитки")
 		(at 290 25 180)
@@
 	)
 	(symbol
+		(lib_name "Приемник_Нитки_13")
 		(lib_id "SCB_АБТЦ:Приемник_Нитки")
 		(at 255 25 180)
@@
 	)
 	(embedded_fonts no)
-	(embedded_files
-		(file
-			(name "КП_МКТ.kicad_wks")
-			(type worksheet)
-			(data |KLUv/WBoIM0nAIZtizBAdTpUIcw/MEEl5UD9vvRxVUaTt7Tdim1NsQHCcIaa6NdKKWWSMk3Fl5PY
-				Ge6GSwSJAG0AhwD9ludlJRB0aTRPj2bLyztxzWxeGSaSIC2v99IsRE8fKpoOBP3ZWQpdVDSzEkYp
-				JmHCaMXIyuJe1igLlSIoxXRQq3gr6ISlMS+LBPrKd3JYJ4qaVKDT8Zgw6DxxFT8Rnwyj1sSMIJk+
-				m2E0lM1rjgQ6HlDs7ubse2HWKZsZAh3P6UIjYiIksi4EArDjY/dOthYZ9rOLcbmxtwuj2PXd7fUy
-				N34NRl+WkSG7993L/v7O9cC35W+wBxblzR3F7LLZmbmS//9a+3bs9qNrGyFs8cHn75zr5rxBurCe
-				o5CJmjBedubqf2WUleyWHt81fN+NTHRZbWlomjwrU7fCSXlnmwpTa6oMTt2PFExNkbGljjzYICwV
-				BTb3qhB33futwQ5JgaRk6om3fMGBMtLUlpf61dtrklChUsdn8t6uhqRYagnLnTREsaxyuK1yqTZV
-				prLUmEpSPZv0mqLdoLDoCcOi8rZfve89YSaKmg8E/alqqkhqpt7Ul8qSs/BZippUgsIekAfU8YDe
-				vXNf5ph5fJWvdLF6sSU/99gebP92zq5V7b4OX0t3/Ptw/8FvZ/4Kuv3XDwsHCq6jc+se7vtDLBQ0
-				KDAYcNtZIbvbto6HXhhF9G3RHSQ8IDw46dyEUdmxmwcAQEfAyobOsgJfjIqL7/KRSnGwdYPu2l9q
-				gUuoIUmqZkaSgqSSNgNRESGMWKeuDnJwGINQCMJwDENSKAcZZwhhxAgKMkRkZEi0A8hZg3bWYlb2
-				h4YoYKGFmekygghKPx7M15IDD7IYd0WZcR9+6xUxAWj38yoXAmC92oZMMfSB1X7rMp20tBrmEBIe
-				hJakM3LW1t3YaQqxwLlbgpwXnM4OLhkcj+VMBQPN2YfN4GDyKLQvgbLaFMHD7rsVHUKT0f1CBDFP
-				XSbe2VB8O79sP6vXCAAfQsfS9FmMsucETSZlwUkkPcQNppQ7TSRxPLsSCN3qj6BnCn09e0/ycEVX
-				3g7wv0CN+KgnLnaDw8y9wQhha3BdLY2v2im89zFrK+VXxtKex5HrauhBrs/tfKi6CNhwPzqzFi3z
-				9U9Sfevn18nGhVF6A8vogOXyMhBb5VwDaXeWAKXYKMLnvwFgs6HSKajyFcrFafcXwJdaG1hIPkiI
-				V/sxYh7nQd22wwlq3PVReFUKBL6a2LzD6KYLdqFI5QQgIR7waZWh9JSLVhZEctJdcwR7A21bB4Hz
-				YfEHf73jPKpiFEOcdpvT9+AQ+tz+oKOKfBl8eLO27y8VJRblwQT7135UnaHRYO7Y2aumWmyLln0M
-				EkEDoZrYI3+aWzQDyapNeKGVQYAECUSWgbsKzB1f7vHwQoUlWbzELbjETzjux+sduNZypQe0pMC3
-				27OXquavENrbkZwas/aMKEFFfiCsrJGJaiGom2yCQx+xet8JSY59VXzJJZZqANQJJJLQ10mk4+Zo
-				KFq0lCRIAwvRiSaVy+NmH7CuRcJ8H5tzH5nMFpPSW2OVDZxoTeXn3khhg88GFYDHgwvheKwMphGy
-				pUNF15jqOumO8hmv3H0Kp2Kv648A3/nhJFgFVZKCoNKJ80sYuikSwx16AEgHvf+okhOf8aBlIYg9
-				C5pjkJDYaAirz+RKmgVKCmny3vo9qWmdnfGSrgI=|
-			)
-			(checksum "3FBF103777E8EE01081CA18737155A0D")
-		)
-	)
 )
