File: example/АБТЦ-2003/Схемы/контроль_повторителей.kicad_sch (KiCad schematic)
At the start: 23 parts

Commit message: Шаблон АБТЦ обновлен
Parts:
- R10, R9: Тип C5-35В -> (none)

Commit message: Обновление примера
Parts:
- Н1, Н11: symbol SCB_Relay:Контакт_нейтрального_якоря_НЗ -> SCB_Legacy:Контакт_нейтрального_якоря_НЗ_бн

Commit message: Поправлены ссылки
Parts:
- П1, П11: symbol SCB_Relay:Контакт_поляризованного_якоря -> SCB_Legacy:Контакт_поляризованного_якоря
Changed lines of the file:
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@@
 	)
 	(symbol
-		(lib_id "SCB_Relay:Контакт_поляризованного_якоря")
+		(lib_id "SCB_Legacy:Контакт_поляризованного_якоря")
 		(at 262.255 155.575 0)
 		(mirror y)
@@
 	)
 	(symbol
-		(lib_id "SCB_Relay:Контакт_поляризованного_якоря")
+		(lib_id "SCB_Legacy:Контакт_поляризованного_якоря")
 		(at 86.995 155.575 0)
 		(unit 1)
