File: example/АБТЦ-2003/Кабельная_сеть/КС.kicad_sch (KiCad schematic)
At the start: 111 parts

Commit message: Шаблон АБТЦ обновлен
Parts:
- removed ДТ1, ДТ11: ~, symbol SCB:Дроссель-трансформатор
- removed unit 2 of Я1
- removed unit 2 of Я11 (x5)
- removed unit 2 of Я111 (x3)
- removed unit 2 of Я1111 (x2)
- removed unit 2 of Я11111 (x2)
- removed Я111111: ~, symbol SCB:Ящик_сдвоенный
- added ДТ1 (x2): ~, symbol SCB_Двухнитка:ДТ-1_сдвоенный
- added Я1 (x14): ~, symbol SCB_АБТЦ:Приемник_Кабельная
- added Я1 (x2): ~, symbol SCB_Двухнитка:Трансформатор_путевой
- БШ: Шкаф (none) -> БШ
- П111, П112: symbol SCB:Приближение -> SCB_АБТЦ:Приближение
- ПЕРЕЕЗД?: symbol SCB:Переезд_Кабельная -> SCB_АБТЦ:Переезд_Кабельная
- РШ1: symbol SCB:Шкаф_переезд -> SCB_АБТЦ:Шкаф_переезд
- УКСПС1, УКСПС111, УКСПС1111: symbol SCB:УКСПС_Кабельная -> SCB_АБТЦ:УКСПС_Кабельная
- Я1, Я11, Я111, Я1111, Я11111, Я12: symbol SCB:Ящик_путевой -> SCB_АБТЦ:Генератор_Кабельная
Connections:
- net 200: now also Я1., ДТ1. (П), Я1., Я1.; no longer Проходной1. (привязка), Проходной3. (привязка), Проходной5. (привязка), Проходной7. (привязка), Проходной9. (привязка), УКСПС1. (привязка), УКСПС1. (привязка), УКСПС111. (привязка), УКСПС1111. (привязка)
- net 5-3(1): now also Я1., Я1., Я1., Я1., Я1., Я1., Я1., Я1., Я1., Я1., Я1., Я1., Я1., Я1., Я1., Я1.
- net Н11П: now also Я1.
- net Н13П: now also Я1.
- net Н15П: now also Я1.; no longer Проходной8. (привязка)
- net Н17П: now also Я1.
- net Н19П: now also Я1.
- net Н1П: now also ДТ1. (П), Я1., Я1.
- net Н21П: now also Я1.
- net Н23П: now also Я1.; no longer Проходной6. (привязка)
- net Н3П : now also Я1.
- net Н5П: now also Я1.
- net Н7П: now also Я1.; no longer Проходной10. (привязка)
- net Н9П: now also Я1.
- net Ч10П: now also Я1.; no longer Проходной2. (привязка)
- net Ч12П: now also Я1.
- net Ч14П: no longer Я1.
- net Ч16П: no longer Я1.
- net Ч20П: now also Я1.
- net Ч22П: now also Я1.
- net Ч24П: now also Я1.
- net Ч26П: now also Я1.; no longer Проходной4. (привязка)
- net Ч28П: now also Я1.
- net Ч2П: now also ДТ1. (П), Я1., Я1.
- net Ч30П: now also Я1.
- net Ч32П: now also Я1.
- net Ч4П: now also Я1.
- net Ч6П: now also Я1.
- net Ч8П: now also Я1.
- new net: ПЕРЕЕЗД?. (привязка), Я1. (x2)
- new net 250: Я1., Я1.
- new net 300: ДТ1. (П), УКСПС1. (привязка), УКСПС1. (привязка), УКСПС111. (привязка), УКСПС1111. (привязка), Я1., Я1., Я1., Я1., Я1., Я1., Я1., Я1., Я1., Я1., Я1., Я1., Я1., Я11., Я111., Я1111., Я12.
- new net 325: Я1., Я1., Я1.
- new net 375: Я1., Я1., Я11.
- new net 400: Я1., Я1., Я1.
- new net 525: Я1., Я1., Я11111.
- new net 650: Я1., Я1., Я111.
- new net 680: Я1., Я1., Я11.
- new net 725: Я1., Я1., Я1111.
Other:
- note removed: "580/12"
- note removed: "720/12"

Commit message: Обновление до 9 KiCad
Connections:
- new net: ПЕРЕЕЗД?. (привязка), Я1. (x2)

Commit message: Embed рамки
Connections:
- new net: ПЕРЕЕЗД?. (привязка), Я1. (x2)
Changed lines of the file:
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@@
 	(generator "eeschema")
 	(generator_version "9.0")
-	(paper "User" 2000 297)
+	(paper "User" 1189 297)
 	(title_block
 		(company "МКТ АТ-351")
