File: example/АБТЦ-2003/Путевой_план/Путевой_план.kicad_sch (KiCad schematic)
At the start: 114 parts

Commit message: Шаблон АБТЦ обновлен
Parts:
- Н1: symbol SCB:Деление_перегона -> SCB_АБТЦ:Деление_перегона
- П1: symbol SCB:Приближение -> SCB_АБТЦ:Приближение
- ПЕРЕЕЗД1: symbol SCB:Переезд_1п -> SCB_АБТЦ:Переезд_1п
Connections:
- net at Магистральный_кабель?. (привязка): now also Магистральный_кабель?. (привязка); no longer Магистральный_кабель?. (привязка) (x28)
- net at Магистральный_кабель?. (привязка): now also Магистральный_кабель1. (привязка); no longer Магистральный_кабель?. (привязка)
- net at Магистральный_кабель1. (привязка): now also Магистральный_кабель1. (привязка); no longer Магистральный_кабель?. (привязка)
- net at Магистральный_2. (привязка): now also Магистральный_4. (привязка)
- net at Магистральный_4. (привязка): now also Магистральный_кабель1. (привязка); no longer Магистральный_2. (привязка)
- net at Магистральный_кабель?. (привязка): now also Магистральный_кабель?. (привязка)
- net at Магистральный_3. (привязка): now also Магистральный_1. (привязка); no longer Магистральный_кабель1. (привязка)
- net at Магистральный_кабель1. (привязка): now also Магистральный_кабель1. (привязка); no longer Магистральный_4. (привязка)
- net at Магистральный_кабель1. (привязка): now also Магистральный_кабель?. (привязка); no longer Магистральный_кабель1. (привязка)
- net at Магистральный_кабель?. (привязка): no longer Магистральный_кабель?. (привязка)
- new net: Магистральный_кабель?. (привязка), Магистральный_кабель?. (привязка) (x17)
- new net: И1. (привязка), ПЕРЕЕЗД1. (привязка), УКСПС1. (привязка)
- new net: Магистральный_3. (привязка), Магистральный_кабель1. (привязка)
- new net: И1. (привязка), ПЕРЕЕЗД1. (привязка), УКСПС1. (привязка), УКСПС1. (привязка), УКСПС1. (привязка)
- now unconnected: Проходной1. (привязка), Проходной11. (привязка), Проходной11. (привязка), Проходной11. (привязка), Проходной11. (привязка), Проходной11. (привязка), Проходной111. (привязка), Проходной111. (привязка), Проходной111. (привязка), Проходной111. (привязка)

Commit message: Обновление до 9 KiCad
Connections:
- net at Магистральный_кабель?. (привязка): now also Магистральный_кабель?. (привязка); no longer Магистральный_кабель?. (привязка) (x28)
- net at Магистральный_кабель?. (привязка): now also Магистральный_кабель1. (привязка); no longer Магистральный_кабель?. (привязка)
- net at Магистральный_кабель1. (привязка): now also Магистральный_кабель1. (привязка); no longer Магистральный_кабель?. (привязка)
- net at Магистральный_2. (привязка): now also Магистральный_4. (привязка)
- net at Магистральный_4. (привязка): now also Магистральный_кабель1. (привязка); no longer Магистральный_2. (привязка)
- net at Магистральный_кабель?. (привязка): now also Магистральный_кабель?. (привязка)
- net at Магистральный_3. (привязка): now also Магистральный_1. (привязка); no longer Магистральный_кабель1. (привязка)
- net at Магистральный_кабель1. (привязка): now also Магистральный_кабель1. (привязка); no longer Магистральный_4. (привязка)
- net at Магистральный_кабель1. (привязка): now also Магистральный_кабель?. (привязка); no longer Магистральный_кабель1. (привязка)
- net at Магистральный_кабель?. (привязка): no longer Магистральный_кабель?. (привязка)
- new net: Магистральный_кабель?. (привязка), Магистральный_кабель?. (привязка) (x17)
- new net: Магистральный_3. (привязка), Магистральный_кабель1. (привязка)

Commit message: Embed рамки
Connections:
- net at Магистральный_кабель?. (привязка): now also Магистральный_кабель?. (привязка); no longer Магистральный_кабель?. (привязка) (x28)
- net at Магистральный_кабель?. (привязка): now also Магистральный_кабель1. (привязка); no longer Магистральный_кабель?. (привязка)
- net at Магистральный_кабель1. (привязка): now also Магистральный_кабель1. (привязка); no longer Магистральный_кабель?. (привязка)
- net at Магистральный_2. (привязка): now also Магистральный_4. (привязка)
- net at Магистральный_4. (привязка): now also Магистральный_кабель1. (привязка); no longer Магистральный_2. (привязка)
- net at Магистральный_кабель?. (привязка): now also Магистральный_кабель?. (привязка)
- net at Магистральный_3. (привязка): now also Магистральный_1. (привязка); no longer Магистральный_кабель1. (привязка)
- net at Магистральный_кабель1. (привязка): now also Магистральный_кабель1. (привязка); no longer Магистральный_4. (привязка)
- net at Магистральный_кабель1. (привязка): now also Магистральный_кабель?. (привязка); no longer Магистральный_кабель1. (привязка)
- net at Магистральный_кабель?. (привязка): no longer Магистральный_кабель?. (привязка)
- new net: Магистральный_кабель?. (привязка), Магистральный_кабель?. (привязка) (x17)
- new net: Магистральный_3. (привязка), Магистральный_кабель1. (привязка)
Changed lines of the file:
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@@
 	)
 	(embedded_fonts no)
+	(embedded_files
+		(file
+			(name "КП_МКТ.kicad_wks")
+			(type worksheet)
+			(data |KLUv/WBoIM0nAIZtizBAdTpUIcw/MEEl5UD9vvRxVUaTt7Tdim1NsQHCcIaa6NdKKWWSMk3Fl5PY
+				Ge6GSwSJAG0AhwD9ludlJRB0aTRPj2bLyztxzWxeGSaSIC2v99IsRE8fKpoOBP3ZWQpdVDSzEkYp
+				JmHCaMXIyuJe1igLlSIoxXRQq3gr6ISlMS+LBPrKd3JYJ4qaVKDT8Zgw6DxxFT8Rnwyj1sSMIJk+
+				m2E0lM1rjgQ6HlDs7ubse2HWKZsZAh3P6UIjYiIksi4EArDjY/dOthYZ9rOLcbmxtwuj2PXd7fUy
+				N34NRl+WkSG7993L/v7O9cC35W+wBxblzR3F7LLZmbmS//9a+3bs9qNrGyFs8cHn75zr5rxBurCe
+				o5CJmjBedubqf2WUleyWHt81fN+NTHRZbWlomjwrU7fCSXlnmwpTa6oMTt2PFExNkbGljjzYICwV
+				BTb3qhB33futwQ5JgaRk6om3fMGBMtLUlpf61dtrklChUsdn8t6uhqRYagnLnTREsaxyuK1yqTZV
+				prLUmEpSPZv0mqLdoLDoCcOi8rZfve89YSaKmg8E/alqqkhqpt7Ul8qSs/BZippUgsIekAfU8YDe
+				vXNf5ph5fJWvdLF6sSU/99gebP92zq5V7b4OX0t3/Ptw/8FvZ/4Kuv3XDwsHCq6jc+se7vtDLBQ0
+				KDAYcNtZIbvbto6HXhhF9G3RHSQ8IDw46dyEUdmxmwcAQEfAyobOsgJfjIqL7/KRSnGwdYPu2l9q
+				gUuoIUmqZkaSgqSSNgNRESGMWKeuDnJwGINQCMJwDENSKAcZZwhhxAgKMkRkZEi0A8hZg3bWYlb2
+				h4YoYKGFmekygghKPx7M15IDD7IYd0WZcR9+6xUxAWj38yoXAmC92oZMMfSB1X7rMp20tBrmEBIe
+				hJakM3LW1t3YaQqxwLlbgpwXnM4OLhkcj+VMBQPN2YfN4GDyKLQvgbLaFMHD7rsVHUKT0f1CBDFP
+				XSbe2VB8O79sP6vXCAAfQsfS9FmMsucETSZlwUkkPcQNppQ7TSRxPLsSCN3qj6BnCn09e0/ycEVX
+				3g7wv0CN+KgnLnaDw8y9wQhha3BdLY2v2im89zFrK+VXxtKex5HrauhBrs/tfKi6CNhwPzqzFi3z
+				9U9Sfevn18nGhVF6A8vogOXyMhBb5VwDaXeWAKXYKMLnvwFgs6HSKajyFcrFafcXwJdaG1hIPkiI
+				V/sxYh7nQd22wwlq3PVReFUKBL6a2LzD6KYLdqFI5QQgIR7waZWh9JSLVhZEctJdcwR7A21bB4Hz
+				YfEHf73jPKpiFEOcdpvT9+AQ+tz+oKOKfBl8eLO27y8VJRblwQT7135UnaHRYO7Y2aumWmyLln0M
+				EkEDoZrYI3+aWzQDyapNeKGVQYAECUSWgbsKzB1f7vHwQoUlWbzELbjETzjux+sduNZypQe0pMC3
+				27OXquavENrbkZwas/aMKEFFfiCsrJGJaiGom2yCQx+xet8JSY59VXzJJZZqANQJJJLQ10mk4+Zo
+				KFq0lCRIAwvRiSaVy+NmH7CuRcJ8H5tzH5nMFpPSW2OVDZxoTeXn3khhg88GFYDHgwvheKwMphGy
+				pUNF15jqOumO8hmv3H0Kp2Kv648A3/nhJFgFVZKCoNKJ80sYuikSwx16AEgHvf+okhOf8aBlIYg9
+				C5pjkJDYaAirz+RKmgVKCmny3vo9qWmdnfGSrgI=|
+			)
+			(checksum "3FBF103777E8EE01081CA18737155A0D")
+		)
+	)
 )
