File: example/БМРЦ/Двухниточный/Двухниточный.kicad_sch (KiCad schematic)
At the start: 175 parts

Commit message: Новое дерево для КП 01.01
Connections:
- net at ЯП37.: now also ДТ18. (П), Соединитель18.1, Соединитель19.2, Стрелка19.1, Стрелка20.2
- net at Магистральный_кабель1. (привязка): now also Магистральный_кабель1. (привязка); no longer Магистральный_кабель1. (привязка) (x7)
- net at Магистральный_кабель1. (привязка): now also К111.; no longer Магистральный_кабель1. (привязка)
- net at Путь3.: now also ДТ23. (П)
- net at ДТ23. (П): now also Стрелка15.; no longer Путь3.
- net at Магистральный_кабель1. (привязка): now also Магистральный_кабель1. (привязка); no longer К1.
- net at ДТ22. (П): now also Путь1.; no longer Стрелка15.
- net at ДТ16. (П): now also Стрелка14.; no longer Стрелка15.
- net at ДТ21. (П): now also Путь6.2, Стрелка20.6, Электротяга4.2, ЯР6П.
- net at Магистральный_кабель1. (привязка): now also Магистральный_кабель1. (привязка); no longer Магистральный_9. (привязка)
- net at Стрелка13.: now also ДТ14. (П)
- net at Стрелка14.: now also ДТ10. (П); no longer Стрелка13.
- net at ДТ14. (П): now also Путь2.; no longer Стрелка13.
- net at Стрелка10.: now also ДТ4. (П)
- net at Стрелка10.: now also ДТ8. (П); no longer Стрелка10.
- net at ДТ4. (П): no longer Стрелка10.
- net at ДТ1. (П): now also ДТ3. (П), Путь1.2, Соединитель1.2, Стрелка9.2
- net at ДТ3. (П): now also Стрелка9.; no longer ДТ1. (П)
- net at ДТ8. (П): now also Стрелка11.; no longer Стрелка10.
- net at ДТ10. (П): now also Стрелка12.; no longer Стрелка14.
- net at Магистральный_1. (привязка): now also Магистральный_кабель1. (привязка); no longer Магистральный_3. (привязка)
- net at Магистральный_кабель1. (привязка): now also Магистральный_8. (привязка); no longer Магистральный_1. (привязка)
- net at Стрелка17.: now also ДТ13. (П)
- net at ДТ11. (П): now also Стрелка13.; no longer Стрелка17.
- net at ДТ13. (П): now also Стрелка18.; no longer Стрелка17.
- net at К111.: now also Магистральный_кабель1. (привязка)
- net at Магистральный_кабель1. (привязка): now also Магистральный_кабель1. (привязка); no longer К111.
- net at ДТ17. (П): now also Путь4.; no longer Стрелка18.
- net at Путь4.: no longer ДТ17. (П)
- net at Стрелка9.: now also ДТ24. (П)
- net at ДТ7. (П): now also Стрелка15.; no longer Стрелка9.
- net at ДТ24. (П): no longer Стрелка9.
- net at ЯРМ29П.: now also ДТ19. (П), Стрелка16.4, Электротяга2.2
- net at Стрелка13.: now also Стрелка11.
- net at Стрелка11.: no longer Стрелка13.
- net at Путь2.: no longer ДТ14. (П)
- net at Стрелка9.: now also ДТ6. (П); no longer ДТ3. (П)
- net at ДТ6. (П): now also Стрелка12.; no longer Стрелка9.
- net at Стрелка12.: now also Стрелка12.
- net at Стрелка12.: no longer Стрелка12.
- net at К111111.: no longer Магистральный_кабель1. (привязка)
- net at К11111.: now also Магистральный_кабель1. (привязка)
- net at Магистральный_кабель1. (привязка): now also Магистральный_кабель1. (привязка); no longer К11111.
- net at Магистральный_кабель1. (привязка): now also Магистральный_2. (привязка); no longer К11111.
- net at К11.: now also Магистральный_7. (привязка)
- net at Магистральный_6. (привязка): now also Магистральный_5. (привязка); no longer К11.
- net at Магистральный_7. (привязка): no longer К11.
- net at Магистральный_5. (привязка): now also Магистральный_4. (привязка); no longer Магистральный_6. (привязка)
- net at Стрелка14.: now also ДТ9. (П); no longer ДТ16. (П)
- net at Магистральный_кабель1. (привязка): now also К1111.; no longer Магистральный_кабель1. (привязка) (x2)
- net at ДТ15. (П): now also Стрелка19.
- net at Стрелка19.: now also ДТ18. (П); no longer ДТ15. (П)
- net at Стрелка15.: no longer ДТ7. (П)
- net at К1111.: no longer Магистральный_кабель1. (привязка) (x2)
- net at ЯП19.: now also ДТ12. (П), Соединитель11.1, Соединитель12.2, Стрелка15.1, Стрелка16.2
- net at ДТ12. (П): now also Стрелка15.
- net at Стрелка11.: now also ДТ5. (П)
- net at ДТ5. (П): now also ДТ2. (П); no longer Стрелка11.
- net at Магистральный_4. (привязка): now also Магистральный_3. (привязка); no longer Магистральный_5. (привязка)
- net at ДТ18. (П): no longer Стрелка19.
- new net: Магистральный_кабель1. (привязка), Магистральный_кабель1. (привязка) (x2)
- new net: ДТ23. (П), Путь3.
- new net: К1., Магистральный_кабель1. (привязка)
- new net: ДТ22. (П), Стрелка15. (x2)
- new net: ДТ16. (П), Стрелка15. (x2)
- new net: ДТ23. (П), Стрелка15.
- new net: Магистральный_9. (привязка), Магистральный_кабель1. (привязка)
- new net: Стрелка13., Стрелка14. (x2)
- new net: ДТ14. (П), Стрелка13.
- new net: Стрелка10., Стрелка10. (x2)
- new net: ДТ4. (П), Стрелка10.
- new net: ДТ1. (П), ДТ3. (П) (x2)
- new net: ДТ8. (П), Стрелка10.
- new net: ДТ10. (П), Стрелка14.
- new net: Магистральный_1. (привязка), Магистральный_3. (привязка)
- new net: ДТ11. (П), Стрелка17. (x2)
- new net: ДТ13. (П), Стрелка17.
- new net: ДТ17. (П), Стрелка18. (x2)
- new net: ДТ17. (П), Путь4.
- new net: ДТ7. (П), Стрелка9. (x2)
- new net: ДТ24. (П), Стрелка9.
- new net: ДТ11. (П), Стрелка13.
- new net: Стрелка11., Стрелка13.
- new net: ДТ14. (П), Путь2.
- new net: ДТ3. (П), Стрелка9.
- new net: ДТ6. (П), Стрелка9.
- new net: ДТ10. (П), Стрелка12.
- new net: Стрелка12., Стрелка12.
- new net: К111111., Магистральный_кабель1. (привязка)
- new net: ДТ22. (П), Путь1.
- new net: К11111., Магистральный_кабель1. (привязка)
- new net: ДТ6. (П), Стрелка12.
- new net: К11., Магистральный_6. (привязка)
- new net: ДТ16. (П), Стрелка14.
- new net: ДТ15. (П), Стрелка19.
- new net: ДТ7. (П), Стрелка15.
- new net: К111111., Магистральный_2. (привязка)
- new net: ДТ12. (П), Стрелка15.
- new net: ДТ9. (П), Стрелка11. (x2)
- new net: ДТ5. (П), Стрелка11.
- new net: ДТ9. (П), Стрелка14.
- new net: ДТ18. (П), Стрелка19.
- new net: ДТ2. (П), ДТ5. (П)
- new net: ДТ8. (П), Стрелка11.
- new net: ДТ13. (П), Стрелка18.
- now unconnected: ДТ18. (П), ДТ18. (П), ДТ19. (П), ДТ24. (П), ДТ4. (П), К111111., Путь2., Путь4., Стрелка11., Стрелка11., Стрелка11., Стрелка12., Стрелка12., Стрелка12., Стрелка15., Стрелка15., Стрелка15., ЯР6П.
Other:
- added sheet Канализация (канализация.kicad_sch)
- note added: "Оборудование горловины станции устройсвами блочной маршрутно-релейной централизации (БМРЦ)"

Commit message: Наведен порядок в двухнитке
Parts:
- added Магистральный_кабель1 (x3): ~, symbol SCB:Магистральный_кабель
- Входной2: Литера НД -> Н
- ДТ4: Секция2 М5П -> М3П
- Изостыки2, Изостыки3, Изостыки4, Изостыки5, Изостыки6, Изостыки7, Изостыки8, Изостыки9: symbol SCB_Двухнитка:Изостыки_бок -> SCB_Двухнитка:Изостыки_без_контроля_отв
- Маневровый18: Литера М5 -> М3
- Маневровый19: Литера М3 -> М5
- Маневровый21: Литера М9 -> М11
- Маневровый22: Литера М11 -> М9
- Маневровый29: Литера М27 -> М25
- Маневровый30: Литера М25 -> М29
- Маневровый6: Литера М29 -> М27
- ЯРМ29П: Секция1 М29П -> М27П
Connections:
- net at ЯП37.: now also ДТ18. (П), Соединитель18.1, Соединитель19.2, Стрелка19.1, Стрелка20.2
- net at Магистральный_кабель1. (привязка): now also Магистральный_кабель1. (привязка); no longer Магистральный_кабель1. (привязка) (x8)
- net at Магистральный_кабель1. (привязка): now also К111.; no longer Магистральный_кабель1. (привязка)
- net at Путь3.: now also ДТ23. (П)
- net at ДТ23. (П): now also Стрелка15.; no longer Путь3.
- net at Магистральный_кабель1. (привязка): now also Магистральный_кабель1. (привязка); no longer К1.
- net at ДТ22. (П): now also Путь1.; no longer Стрелка15.
- net at ДТ16. (П): now also Стрелка14.; no longer Стрелка15.
- net at ДТ21. (П): now also Путь6.2, Стрелка20.6, Электротяга4.2, ЯР6П.
- net at Магистральный_кабель1. (привязка): now also Магистральный_кабель1. (привязка); no longer Магистральный_9. (привязка)
- net at Стрелка13.: now also ДТ14. (П)
- net at Стрелка14.: now also ДТ10. (П); no longer Стрелка13.
- net at ДТ14. (П): now also Путь2.; no longer Стрелка13.
- net at Стрелка10.: now also ДТ4. (П)
- net at Стрелка10.: now also ДТ8. (П); no longer Стрелка10.
- net at ДТ4. (П): no longer Стрелка10.
- net at ДТ1. (П): now also ДТ3. (П), Путь1.2, Соединитель1.2, Стрелка9.2
- net at ДТ3. (П): now also Стрелка9.; no longer ДТ1. (П)
- net at ДТ8. (П): now also Стрелка11.; no longer Стрелка10.
- net at ДТ10. (П): now also Стрелка12.; no longer Стрелка14.
- net at Магистральный_1. (привязка): now also Магистральный_кабель1. (привязка); no longer Магистральный_3. (привязка)
- net at Магистральный_кабель1. (привязка): now also Магистральный_8. (привязка); no longer Магистральный_1. (привязка)
- net at Стрелка17.: now also ДТ13. (П)
- net at ДТ11. (П): now also Стрелка13.; no longer Стрелка17.
- net at ДТ13. (П): now also Стрелка18.; no longer Стрелка17.
- net at К111.: now also Магистральный_кабель1. (привязка)
- net at Магистральный_кабель1. (привязка): now also Магистральный_кабель1. (привязка); no longer К111.
- net at ДТ17. (П): now also Путь4.; no longer Стрелка18.
- net at Путь4.: no longer ДТ17. (П)
- net at Стрелка9.: now also ДТ24. (П)
- net at ДТ7. (П): now also Стрелка15.; no longer Стрелка9.
- net at ДТ24. (П): no longer Стрелка9.
- net at ЯРМ29П.: now also ДТ19. (П), Стрелка16.4, Электротяга2.2
- net at Стрелка13.: now also Стрелка11.
- net at Стрелка11.: no longer Стрелка13.
- net at Путь2.: no longer ДТ14. (П)
- net at Стрелка9.: now also ДТ6. (П); no longer ДТ3. (П)
- net at ДТ6. (П): now also Стрелка12.; no longer Стрелка9.
- net at Стрелка12.: now also Стрелка12.
- net at Стрелка12.: no longer Стрелка12.
- net at К111111.: no longer Магистральный_кабель1. (привязка)
- net at К11111.: now also Магистральный_кабель1. (привязка)
- net at Магистральный_кабель1. (привязка): now also Магистральный_кабель1. (привязка); no longer К11111.
- net at Магистральный_кабель1. (привязка): now also Магистральный_2. (привязка); no longer К11111.
- net at К11.: now also Магистральный_7. (привязка)
- net at Магистральный_6. (привязка): now also Магистральный_5. (привязка); no longer К11.
- net at Магистральный_7. (привязка): no longer К11.
- net at Магистральный_5. (привязка): now also Магистральный_4. (привязка); no longer Магистральный_6. (привязка)
- net at Стрелка14.: now also ДТ9. (П); no longer ДТ16. (П)
- net at Магистральный_кабель1. (привязка): now also К1111.; no longer Магистральный_кабель1. (привязка) (x2)
- net at ДТ15. (П): now also Стрелка16.6, Стрелка19.5
- net at Стрелка19.: now also ДТ18. (П); no longer ДТ15. (П)
- net at Стрелка15.: no longer ДТ7. (П)
- net at К1111.: no longer Магистральный_кабель1. (привязка) (x2)
- net at ЯП19.: now also ДТ12. (П), Соединитель11.1, Соединитель12.2, Стрелка15.1, Стрелка16.2
- net at ДТ12. (П): now also Стрелка15.
- net at Стрелка11.: now also ДТ5. (П)
- net at ДТ5. (П): now also ДТ2. (П); no longer Стрелка11.
- net at Магистральный_4. (привязка): now also Магистральный_3. (привязка); no longer Магистральный_5. (привязка)
- net at ДТ18. (П): no longer Стрелка19.
- new net: Магистральный_кабель1. (привязка), Магистральный_кабель1. (привязка) (x4)
- new net: ДТ23. (П), Путь3.
- new net: К1., Магистральный_кабель1. (привязка)
- new net: ДТ22. (П), Стрелка15. (x2)
- new net: ДТ16. (П), Стрелка15. (x2)
- new net: ДТ23. (П), Стрелка15.
- new net: Магистральный_9. (привязка), Магистральный_кабель1. (привязка)
- new net: Стрелка13., Стрелка14. (x2)
- new net: ДТ14. (П), Стрелка13.
- new net: Стрелка10., Стрелка10. (x2)
- new net: ДТ4. (П), Стрелка10.
- new net: ДТ1. (П), ДТ3. (П) (x2)
- new net: ДТ8. (П), Стрелка10.
- new net: ДТ10. (П), Стрелка14.
- new net: Магистральный_1. (привязка), Магистральный_3. (привязка)
- new net: ДТ11. (П), Стрелка17. (x2)
- new net: ДТ13. (П), Стрелка17.
- new net: ДТ17. (П), Стрелка18. (x2)
- new net: ДТ17. (П), Путь4.
- new net: ДТ7. (П), Стрелка9. (x2)
- new net: ДТ24. (П), Стрелка9.
- new net: ДТ11. (П), Стрелка13.
- new net: Стрелка11., Стрелка13.
- new net: ДТ14. (П), Путь2.
- new net: ДТ3. (П), Стрелка9.
- new net: ДТ6. (П), Стрелка9.
- new net: ДТ10. (П), Стрелка12.
- new net: Стрелка12., Стрелка12.
- new net: К111111., Магистральный_кабель1. (привязка)
- new net: ДТ22. (П), Путь1.
- new net: К11111., Магистральный_кабель1. (привязка)
- new net: ДТ6. (П), Стрелка12.
- new net: К11., Магистральный_6. (привязка)
- new net: ДТ16. (П), Стрелка14.
- new net: ДТ15. (П), Стрелка19. (x2)
- new net: ДТ7. (П), Стрелка15.
- new net: К111111., Магистральный_2. (привязка)
- new net: ДТ12. (П), Стрелка15.
- new net: ДТ9. (П), Стрелка11. (x2)
- new net: ДТ5. (П), Стрелка11.
- new net: ДТ9. (П), Стрелка14.
- new net: ДТ18. (П), Стрелка19.
- new net: ДТ2. (П), ДТ5. (П)
- new net: ДТ8. (П), Стрелка11.
- new net: ДТ13. (П), Стрелка18.
- now unconnected: ДТ18. (П), ДТ18. (П), ДТ19. (П), ДТ24. (П), ДТ4. (П), К111111., Путь2., Путь4., Стрелка11., Стрелка11., Стрелка11., Стрелка12., Стрелка12., Стрелка12., Стрелка15., Стрелка15., Стрелка15., ЯР33., ЯР6П.
Other:
- note added: "М27П"
- note added: "М3П"
- note added: "Схема полной изоляции путей и стрелок с канализацией тягового тока"
- note removed: "М29П"
- note removed: "М5П"

Commit message: Исправлен пример БМРЦ
Parts:
- renumbered Входной2 to Входной1
Connections:
- net at ЯП37.: now also ДТ18., Соединитель18.1, Соединитель19.2, Стрелка19.1, Стрелка20.2
- net at Магистральный_кабель1. (привязка): now also Магистральный_кабель1. (привязка); no longer Магистральный_кабель1. (привязка) (x8)
- net at Магистральный_кабель1. (привязка): now also К111.; no longer Магистральный_кабель1. (привязка)
- net at Путь3.: now also ДТ23.
- net at ДТ23.: now also Стрелка15.; no longer Путь3.
- net at Магистральный_кабель1. (привязка): now also Магистральный_кабель1. (привязка); no longer К1.
- net at ДТ22.: now also Путь1.; no longer Стрелка15.
- net at ДТ16.: now also Стрелка14.; no longer Стрелка15.
- net at ДТ21.: now also Путь6.2, Стрелка20.6, Электротяга4.2, ЯР6П.
- net at Магистральный_кабель1. (привязка): now also Магистральный_кабель1. (привязка); no longer Магистральный_9. (привязка)
- net at Стрелка13.: now also ДТ14.
- net at Стрелка14.: now also ДТ10.; no longer Стрелка13.
- net at ДТ14.: now also Путь2.; no longer Стрелка13.
- net at Стрелка10.: now also ДТ4.
- net at Стрелка10.: now also ДТ8.; no longer Стрелка10.
- net at ДТ4.: no longer Стрелка10.
- net at ДТ1.: now also ДТ3., Путь1.2, Соединитель1.2, Стрелка9.2
- net at ДТ3.: now also Стрелка9.; no longer ДТ1. (П)
- net at ДТ8.: now also Стрелка11.; no longer Стрелка10.
- net at ДТ10.: now also Стрелка12.; no longer Стрелка14.
- net at Магистральный_1. (привязка): now also Магистральный_кабель1. (привязка); no longer Магистральный_3. (привязка)
- net at Магистральный_кабель1. (привязка): now also Магистральный_8. (привязка); no longer Магистральный_1. (привязка)
- net at Стрелка17.: now also ДТ13.
- net at ДТ11.: now also Стрелка13.; no longer Стрелка17.
- net at ДТ13.: now also Стрелка18.; no longer Стрелка17.
- net at К111.: now also Магистральный_кабель1. (привязка)
- net at Магистральный_кабель1. (привязка): now also Магистральный_кабель1. (привязка); no longer К111.
- net at ДТ17.: now also Путь4.; no longer Стрелка18.
- net at Путь4.: no longer ДТ17. (П)
- net at Стрелка9.: now also ДТ24.
- net at ДТ7.: now also Стрелка15.; no longer Стрелка9.
- net at ДТ24.: no longer Стрелка9.
- net at ЯРМ29П.: now also ДТ19., Стрелка16.4, Электротяга2.2
- net at Стрелка13.: now also Стрелка11.
- net at Стрелка11.: no longer Стрелка13.
- net at Путь2.: no longer ДТ14. (П)
- net at Стрелка9.: now also ДТ6.; no longer ДТ3. (П)
- net at ДТ6.: now also Стрелка12.; no longer Стрелка9.
- net at Стрелка12.: now also Стрелка12.
- net at Стрелка12.: no longer Стрелка12.
- net at К111111.: no longer Магистральный_кабель1. (привязка)
- net at К11111.: now also Магистральный_кабель1. (привязка)
- net at Магистральный_кабель1. (привязка): now also Магистральный_кабель1. (привязка); no longer К11111.
- net at Магистральный_кабель1. (привязка): now also Магистральный_2. (привязка); no longer К11111.
- net at К11.: now also Магистральный_7. (привязка)
- net at Магистральный_6. (привязка): now also Магистральный_5. (привязка); no longer К11.
- net at Магистральный_7. (привязка): no longer К11.
- net at Магистральный_5. (привязка): now also Магистральный_4. (привязка); no longer Магистральный_6. (привязка)
- net at Стрелка14.: now also ДТ9.; no longer ДТ16. (П)
- net at Магистральный_кабель1. (привязка): now also К1111.; no longer Магистральный_кабель1. (привязка) (x2)
- net at ДТ15.: now also Стрелка16.6, Стрелка19.5
- net at Стрелка19.: now also ДТ18.; no longer ДТ15. (П)
- net at Стрелка15.: no longer ДТ7. (П)
- net at К1111.: no longer Магистральный_кабель1. (привязка) (x2)
- net at ЯП19.: now also ДТ12., Соединитель11.1, Соединитель12.2, Стрелка15.1, Стрелка16.2
- net at ДТ12.: now also Стрелка15.
- net at Стрелка11.: now also ДТ5.
- net at ДТ5.: now also ДТ2.; no longer Стрелка11.
- net at Магистральный_4. (привязка): now also Магистральный_3. (привязка); no longer Магистральный_5. (привязка)
- net at ДТ18.: no longer Стрелка19.
- new net: Магистральный_кабель1. (привязка), Магистральный_кабель1. (привязка) (x3)
- new net: ДТ23., Путь3.
- new net: К1., Магистральный_кабель1. (привязка)
- new net: ДТ22., Стрелка15. (x2)
- new net: ДТ16., Стрелка15. (x2)
- new net: ДТ23., Стрелка15.
- new net: Магистральный_9. (привязка), Магистральный_кабель1. (привязка)
- new net: Стрелка13., Стрелка14. (x2)
- new net: ДТ14., Стрелка13.
- new net: Стрелка10., Стрелка10. (x2)
- new net: ДТ4., Стрелка10.
- new net: ДТ1., ДТ3. (x2)
- new net: ДТ8., Стрелка10.
- new net: ДТ10., Стрелка14.
- new net: Магистральный_1. (привязка), Магистральный_3. (привязка)
- new net: ДТ11., Стрелка17. (x2)
- new net: ДТ13., Стрелка17.
- new net: ДТ17., Стрелка18. (x2)
- new net: ДТ17., Путь4.
- new net: ДТ7., Стрелка9. (x2)
- new net: ДТ24., Стрелка9.
- new net: ДТ11., Стрелка13.
- new net: Стрелка11., Стрелка13.
- new net: ДТ14., Путь2.
- new net: ДТ3., Стрелка9.
- new net: ДТ6., Стрелка9.
- new net: ДТ10., Стрелка12.
- new net: Стрелка12., Стрелка12.
- new net: К111111., Магистральный_кабель1. (привязка)
- new net: ДТ22., Путь1.
- new net: К11111., Магистральный_кабель1. (привязка)
- new net: ДТ6., Стрелка12.
- new net: К11., Магистральный_6. (привязка)
- new net: ДТ16., Стрелка14.
- new net: ДТ15., Стрелка19. (x2)
- new net: ДТ7., Стрелка15.
- new net: К111111., Магистральный_2. (привязка)
- new net: ДТ12., Стрелка15.
- new net: ДТ9., Стрелка11. (x2)
- new net: ДТ5., Стрелка11.
- new net: ДТ9., Стрелка14.
- new net: ДТ18., Стрелка19.
- new net: ДТ2., ДТ5.
- new net: ДТ8., Стрелка11.
- new net: ДТ13., Стрелка18.
- now unconnected: ДТ18. (П), ДТ18. (П), ДТ19. (П), ДТ24. (П), ДТ4. (П), К111111., Путь2., Путь4., Стрелка11., Стрелка11., Стрелка11., Стрелка12., Стрелка12., Стрелка12., Стрелка15., Стрелка15., Стрелка15., ЯР6П.
