File: example/БМРЦ/Двухниточный/Двухниточный.kicad_sch (KiCad schematic)
At the start: 181 parts

Commit message: Обновление до 9 KiCad
Parts:
- Входной1, Входной2: now in the parts list
- renumbered Выходной8 to Выходной1, Выходной6 to Выходной2, Выходной5 to Выходной3, Выходной7 to Выходной4, ДТ19 to ДТ1, ДТ8 to ДТ10, ДТ13 to ДТ12, ДТ17 to ДТ13, ДТ1 to ДТ14, ДТ3 to ДТ15, ДТ6 to ДТ16, ДТ10 to ДТ17, ДТ14 to ДТ18, ДТ2 to ДТ19, ДТ20 to ДТ2, ДТ5 to ДТ20, ДТ9 to ДТ21, ДТ16 to ДТ22, ДТ22 to ДТ23, ДТ23 to ДТ24, ДТ24 to ДТ3, ДТ7 to ДТ4, ДТ12 to ДТ5, ДТ15 to ДТ6, ДТ18 to ДТ7, ДТ21 to ДТ8, ДТ4 to ДТ9, Изостыки3 to Изостыки1, Изостыки6 to Изостыки2, Изостыки9 to Изостыки3, Изостыки1 to Изостыки4, Изостыки2 to Изостыки5, Изостыки5 to Изостыки6, Изостыки4 to Изостыки8, Изостыки8 to Изостыки9, К11111 to К1, К1111 to К2, К1111 to К3, К111 to К4, К1 to К5, К1111 to К6, К111 to К7, К11 to К8, К111111 to К9, Магистральный_7 to Магистральный_1, Магистральный_6 to Магистральный_3, Магистральный_5 to Магистральный_4, Магистральный_9 to Магистральный_5, Магистральный_4 to Магистральный_6, Магистральный_3 to Магистральный_7, Магистральный_1 to Магистральный_8, Магистральный_8 to Магистральный_9, Магистральный_кабель1 to Магистральный_?, Магистральный_кабель1 to Магистральный_кабель10, Магистральный_кабель1 to Магистральный_кабель11, Магистральный_кабель1 to Магистральный_кабель12, Магистральный_кабель1 to Магистральный_кабель13, Магистральный_кабель1 to Магистральный_кабель14, Магистральный_кабель1 to Магистральный_кабель15, Магистральный_кабель1 to Магистральный_кабель16, Магистральный_кабель1 to Магистральный_кабель17, Магистральный_кабель1 to Магистральный_кабель18, Магистральный_кабель1 to Магистральный_кабель19, Магистральный_кабель1 to Магистральный_кабель2, Магистральный_кабель1 to Магистральный_кабель20, Магистральный_кабель1 to Магистральный_кабель3, Магистральный_кабель1 to Магистральный_кабель4, Магистральный_кабель1 to Магистральный_кабель5, Магистральный_кабель1 to Магистральный_кабель6, Магистральный_кабель1 to Магистральный_кабель7, Магистральный_кабель1 to Магистральный_кабель8, Магистральный_кабель1 to Магистральный_кабель9, Маневровый6 to Маневровый1, Маневровый18 to Маневровый10, Маневровый24 to Маневровый11, Маневровый29 to Маневровый12, Маневровый21 to Маневровый13, Маневровый17 to Маневровый14, Маневровый26 to Маневровый15, Маневровый25 to Маневровый16, Маневровый7 to Маневровый17, Маневровый20 to Маневровый18, Маневровый31 to Маневровый19, Маневровый8 to Маневровый2, Маневровый22 to Маневровый3, Маневровый30 to Маневровый4, Маневровый19 to Маневровый5, Маневровый28 to Маневровый6, Маневровый32 to Маневровый7, Маневровый23 to Маневровый8, Маневровый27 to Маневровый9, Путь6 to Путь1, Путь4 to Путь2, Путь1 to Путь3, Путь2 to Путь4, Путь2 to Путь5, Путь1 to Путь6, Путь3 to Путь7, СП2 to СП1, СП15 to СП10, СП3 to СП11, СП1 to СП12, СП7 to СП13, СП9 to СП14, СП11 to СП15, СП13 to СП16, СП5 to СП17, СП16 to СП18, СП18 to СП19, СП10 to СП2, СП12 to СП3, СП17 to СП4, СП19 to СП5, СП4 to СП6, СП6 to СП7, СП14 to СП9, Соединитель12 to Соединитель1, Соединитель6 to Соединитель10, Соединитель14 to Соединитель11, Соединитель1 to Соединитель12, Соединитель9 to Соединитель13, Соединитель10 to Соединитель14, Соединитель7 to Соединитель15, Соединитель13 to Соединитель16, Соединитель4 to Соединитель17, Соединитель16 to Соединитель18, Соединитель17 to Соединитель19, Соединитель19 to Соединитель2, Соединитель2 to Соединитель3, Соединитель11 to Соединитель4, Соединитель18 to Соединитель5, Соединитель5 to Соединитель6, Соединитель8 to Соединитель7, Соединитель15 to Соединитель8, Соединитель3 to Соединитель9, Стрелка9 to Стрелка1, Стрелка16 to Стрелка1, Стрелка14 to Стрелка10, Стрелка12 to Стрелка11, Стрелка11 to Стрелка12, Стрелка10 to Стрелка2, Стрелка20 to Стрелка2, Стрелка15 to Стрелка3, Стрелка11 to Стрелка3, Стрелка12 to Стрелка4, Стрелка19 to Стрелка4, Стрелка13 to Стрелка5, Стрелка14 to Стрелка6, Стрелка18 to Стрелка6, Стрелка15 to Стрелка7, Стрелка10 to Стрелка7, Стрелка17 to Стрелка8, ЭЦ11 to ЭЦ1, Электротяга2 to Электротяга1, Электротяга3 to Электротяга2, Электротяга4 to Электротяга3, Электротяга1 to Электротяга4, ЯП19 to ЯП2, ЯП37 to ЯП3, ЯП3-7 to ЯП3-1, ЯП23 to ЯП4, ЯП4П to ЯП4П1, ЯР19 to ЯР1, ЯР13-17 to ЯР13-1, ЯР33 to ЯР2, ЯР31 to ЯР3, ЯР3П to ЯР3П1, ЯР6П to ЯР6П1, ЯРМ29П to ЯРМ29П1, ЯРМ37П to ЯРМ37П1
Connections:
- net at ЯП3.: now also ДТ7., Соединитель2.2, Соединитель5.1, Стрелка2.2, Стрелка4.1
- net at Магистральный_кабель6. (привязка): now also Магистральный_кабель7. (привязка); no longer Магистральный_кабель5. (привязка)
- net at Магистральный_кабель7. (привязка): now also Магистральный_кабель8. (привязка); no longer Магистральный_кабель6. (привязка)
- net at Магистральный_?. (привязка): now also Магистральный_?. (привязка); no longer Магистральный_?. (привязка)
- net at Магистральный_?. (привязка): now also Магистральный_кабель11. (привязка); no longer Магистральный_?. (привязка)
- net at Магистральный_кабель8. (привязка): now also Магистральный_кабель9. (привязка); no longer Магистральный_кабель7. (привязка)
- net at Магистральный_кабель9. (привязка): now also К4.; no longer Магистральный_кабель8. (привязка)
- net at Путь7.: now also ДТ24.
- net at ДТ24.: now also Стрелка7.; no longer Путь7.
- net at Магистральный_кабель10. (привязка): now also Магистральный_кабель11. (привязка); no longer К5.
- net at ДТ23.: now also Путь6.; no longer Стрелка7.
- net at ДТ22.: now also Стрелка6.; no longer Стрелка7.
- net at ДТ8.: now also Путь1.2, Стрелка2.6, Электротяга3.2, ЯР6П1.
- net at Магистральный_кабель17. (привязка): now also Магистральный_кабель18. (привязка); no longer Магистральный_5. (привязка)
- net at Магистральный_кабель18. (привязка): now also Магистральный_кабель19. (привязка); no longer Магистральный_кабель17. (привязка)
- net at Стрелка5.: now also ДТ18.
- net at Стрелка10.: now also ДТ17.; no longer Стрелка5.
- net at ДТ18.: now also Путь4.; no longer Стрелка5.
- net at Стрелка7.: now also ДТ9.
- net at Стрелка2.: now also ДТ10.; no longer Стрелка7.
- net at ДТ9.: no longer Стрелка7.
- net at ДТ14.: now also ДТ15., Путь3.2, Соединитель12.2, Стрелка9.2
- net at ДТ15.: now also Стрелка9.; no longer ДТ14.
- net at ДТ10.: now also Стрелка3.; no longer Стрелка2.
- net at ДТ17.: now also Стрелка4.; no longer Стрелка10.
- net at Магистральный_8. (привязка): now also Магистральный_кабель20. (привязка); no longer Магистральный_7. (привязка)
- net at Магистральный_кабель20. (привязка): now also Магистральный_9. (привязка); no longer Магистральный_8. (привязка)
- net at Стрелка8.: now also ДТ12.
- net at ДТ11.: now also Стрелка5.; no longer Стрелка8.
- net at ДТ12.: now also Стрелка6.; no longer Стрелка8.
- net at К7.: now also Магистральный_кабель14. (привязка)
- net at Магистральный_кабель14. (привязка): now also Магистральный_кабель15. (привязка); no longer К7.
- net at ДТ13.: now also Путь2.; no longer Стрелка6.
- net at Путь2.: no longer ДТ13.
- net at Стрелка1.: now also ДТ3.
- net at ДТ4.: now also Стрелка3.; no longer Стрелка1.
- net at ДТ3.: no longer Стрелка1.
- net at ЯРМ29П1.: now also ДТ1., Стрелка1.4, Электротяга1.2
- net at Стрелка5.: now also Стрелка3.
- net at Стрелка3.: no longer Стрелка5.
- net at Магистральный_кабель15. (привязка): now also Магистральный_кабель16. (привязка); no longer Магистральный_кабель14. (привязка)
- net at Путь4.: no longer ДТ18.
- net at Стрелка9.: now also ДТ16.; no longer ДТ15.
- net at ДТ16.: now also Стрелка11.; no longer Стрелка9.
- net at Стрелка4.: now also Стрелка11.
- net at Стрелка11.: no longer Стрелка4.
- net at К9.: no longer Магистральный_кабель19. (привязка)
- net at К1.: now also Магистральный_кабель1. (привязка)
- net at Магистральный_кабель2. (привязка): now also Магистральный_кабель3. (привязка); no longer К1.
- net at Магистральный_кабель1. (привязка): now also Магистральный_2. (привязка); no longer К1.
- net at К8.: now also Магистральный_1. (привязка)
- net at Магистральный_3. (привязка): now also Магистральный_4. (привязка); no longer К8.
- net at Магистральный_1. (привязка): no longer К8.
- net at Магистральный_4. (привязка): now also Магистральный_6. (привязка); no longer Магистральный_3. (привязка)
- net at Магистральный_кабель3. (привязка): now also Магистральный_кабель4. (привязка); no longer Магистральный_кабель2. (привязка)
- net at Стрелка6.: now also ДТ21.; no longer ДТ22.
- net at Магистральный_кабель4. (привязка): now also К2.; no longer Магистральный_кабель3. (привязка)
- net at ДТ6.: now also Стрелка1.6, Стрелка4.5
- net at Стрелка4.: now also ДТ7.; no longer ДТ6.
- net at Стрелка3.: no longer ДТ4.
- net at Магистральный_кабель13. (привязка): now also К6.; no longer Магистральный_кабель12. (привязка)
- net at К6.: no longer Магистральный_кабель13. (привязка)
- net at ЯП2.: now also ДТ5., Соединитель1.2, Соединитель4.1, Стрелка1.2, Стрелка3.1
- net at ДТ5.: now also Стрелка3.
- net at К2.: no longer Магистральный_кабель4. (привязка)
- net at Стрелка12.: now also ДТ20.
- net at ДТ20.: now also ДТ19.; no longer Стрелка12.
- net at Магистральный_6. (привязка): now also Магистральный_7. (привязка); no longer Магистральный_4. (привязка)
- net at ДТ7.: no longer Стрелка4.
- new net: Магистральный_кабель5. (привязка), Магистральный_кабель6. (привязка)
- new net: Магистральный_?. (привязка), Магистральный_?. (привязка)
- new net: ДТ24., Путь7.
- new net: К5., Магистральный_кабель10. (привязка)
- new net: ДТ23., Стрелка7. (x2)
- new net: ДТ22., Стрелка7. (x2)
- new net: ДТ24., Стрелка7.
- new net: Магистральный_5. (привязка), Магистральный_кабель17. (привязка)
- new net: Стрелка10., Стрелка5. (x2)
- new net: ДТ18., Стрелка5.
- new net: Стрелка2., Стрелка7. (x2)
- new net: ДТ9., Стрелка7.
- new net: ДТ14., ДТ15. (x2)
- new net: ДТ10., Стрелка2.
- new net: ДТ17., Стрелка10.
- new net: Магистральный_7. (привязка), Магистральный_8. (привязка)
- new net: ДТ11., Стрелка8. (x2)
- new net: ДТ12., Стрелка8.
- new net: ДТ13., Стрелка6. (x2)
- new net: ДТ13., Путь2.
- new net: ДТ4., Стрелка1. (x2)
- new net: ДТ3., Стрелка1.
- new net: ДТ11., Стрелка5.
- new net: Стрелка3., Стрелка5.
- new net: ДТ18., Путь4.
- new net: ДТ15., Стрелка9.
- new net: ДТ16., Стрелка9.
- new net: ДТ17., Стрелка4.
- new net: Стрелка11., Стрелка4.
- new net: К9., Магистральный_кабель19. (привязка)
- new net: ДТ23., Путь6.
- new net: К1., Магистральный_кабель2. (привязка)
- new net: ДТ16., Стрелка11.
- new net: К8., Магистральный_3. (привязка)
- new net: ДТ22., Стрелка6.
- new net: ДТ6., Стрелка4. (x2)
- new net: ДТ4., Стрелка3.
- new net: Магистральный_кабель12. (привязка), Магистральный_кабель13. (привязка)
- new net: К9., Магистральный_2. (привязка)
- new net: ДТ5., Стрелка3.
- new net: ДТ21., Стрелка12. (x2)
- new net: ДТ20., Стрелка12.
- new net: ДТ21., Стрелка6.
- new net: ДТ7., Стрелка4.
- new net: ДТ19., ДТ20.
- new net: ДТ10., Стрелка3.
- new net: ДТ12., Стрелка6.
- now unconnected: ДТ1., ДТ3., ДТ7., ДТ7., ДТ9., К9., Путь2., Путь4., Стрелка11., Стрелка11., Стрелка11., Стрелка3., Стрелка3., Стрелка3., Стрелка3., Стрелка3., Стрелка3., ЯР6П1.

Commit message: Embed рамки
Connections:
- net at ЯП3.: now also ДТ7., Соединитель2.2, Соединитель5.1, Стрелка2.2, Стрелка4.1
- net at Магистральный_кабель6. (привязка): now also Магистральный_кабель7. (привязка); no longer Магистральный_кабель5. (привязка)
- net at Магистральный_кабель7. (привязка): now also Магистральный_кабель8. (привязка); no longer Магистральный_кабель6. (привязка)
- net at Магистральный_?. (привязка): now also Магистральный_?. (привязка); no longer Магистральный_?. (привязка)
- net at Магистральный_?. (привязка): now also Магистральный_кабель11. (привязка); no longer Магистральный_?. (привязка)
- net at Магистральный_кабель8. (привязка): now also Магистральный_кабель9. (привязка); no longer Магистральный_кабель7. (привязка)
- net at Магистральный_кабель9. (привязка): now also К4.; no longer Магистральный_кабель8. (привязка)
- net at Путь7.: now also ДТ24.
- net at ДТ24.: now also Стрелка7.; no longer Путь7.
- net at Магистральный_кабель10. (привязка): now also Магистральный_кабель11. (привязка); no longer К5.
- net at ДТ23.: now also Путь6.; no longer Стрелка7.
- net at ДТ22.: now also Стрелка6.; no longer Стрелка7.
- net at ДТ8.: now also Путь1.2, Стрелка2.6, Электротяга3.2, ЯР6П1.
- net at Магистральный_кабель17. (привязка): now also Магистральный_кабель18. (привязка); no longer Магистральный_5. (привязка)
- net at Магистральный_кабель18. (привязка): now also Магистральный_кабель19. (привязка); no longer Магистральный_кабель17. (привязка)
- net at Стрелка5.: now also ДТ18.
- net at Стрелка10.: now also ДТ17.; no longer Стрелка5.
- net at ДТ18.: now also Путь4.; no longer Стрелка5.
- net at Стрелка7.: now also ДТ9.
- net at Стрелка2.: now also ДТ10.; no longer Стрелка7.
- net at ДТ9.: no longer Стрелка7.
- net at ДТ14.: now also ДТ15., Путь3.2, Соединитель12.2, Стрелка9.2
- net at ДТ15.: now also Стрелка9.; no longer ДТ14.
- net at ДТ10.: now also Стрелка3.; no longer Стрелка2.
- net at ДТ17.: now also Стрелка4.; no longer Стрелка10.
- net at Магистральный_8. (привязка): now also Магистральный_кабель20. (привязка); no longer Магистральный_7. (привязка)
- net at Магистральный_кабель20. (привязка): now also Магистральный_9. (привязка); no longer Магистральный_8. (привязка)
- net at Стрелка8.: now also ДТ12.
- net at ДТ11.: now also Стрелка5.; no longer Стрелка8.
- net at ДТ12.: now also Стрелка6.; no longer Стрелка8.
- net at К7.: now also Магистральный_кабель14. (привязка)
- net at Магистральный_кабель14. (привязка): now also Магистральный_кабель15. (привязка); no longer К7.
- net at ДТ13.: now also Путь2.; no longer Стрелка6.
- net at Путь2.: no longer ДТ13.
- net at Стрелка1.: now also ДТ3.
- net at ДТ4.: now also Стрелка3.; no longer Стрелка1.
- net at ДТ3.: no longer Стрелка1.
- net at ЯРМ29П1.: now also ДТ1., Стрелка1.4, Электротяга1.2
- net at Стрелка5.: now also Стрелка3.
- net at Стрелка3.: no longer Стрелка5.
- net at Магистральный_кабель15. (привязка): now also Магистральный_кабель16. (привязка); no longer Магистральный_кабель14. (привязка)
- net at Путь4.: no longer ДТ18.
- net at Стрелка9.: now also ДТ16.; no longer ДТ15.
- net at ДТ16.: now also Стрелка11.; no longer Стрелка9.
- net at Стрелка4.: now also Стрелка11.
- net at Стрелка11.: no longer Стрелка4.
- net at К9.: no longer Магистральный_кабель19. (привязка)
- net at К1.: now also Магистральный_кабель1. (привязка)
- net at Магистральный_кабель2. (привязка): now also Магистральный_кабель3. (привязка); no longer К1.
- net at Магистральный_кабель1. (привязка): now also Магистральный_2. (привязка); no longer К1.
- net at К8.: now also Магистральный_1. (привязка)
- net at Магистральный_3. (привязка): now also Магистральный_4. (привязка); no longer К8.
- net at Магистральный_1. (привязка): no longer К8.
- net at Магистральный_4. (привязка): now also Магистральный_6. (привязка); no longer Магистральный_3. (привязка)
- net at Магистральный_кабель3. (привязка): now also Магистральный_кабель4. (привязка); no longer Магистральный_кабель2. (привязка)
- net at Стрелка6.: now also ДТ21.; no longer ДТ22.
- net at Магистральный_кабель4. (привязка): now also К2.; no longer Магистральный_кабель3. (привязка)
- net at ДТ6.: now also Стрелка1.6, Стрелка4.5
- net at Стрелка4.: now also ДТ7.; no longer ДТ6.
- net at Стрелка3.: no longer ДТ4.
- net at Магистральный_кабель13. (привязка): now also К6.; no longer Магистральный_кабель12. (привязка)
- net at К6.: no longer Магистральный_кабель13. (привязка)
- net at ЯП2.: now also ДТ5., Соединитель1.2, Соединитель4.1, Стрелка1.2, Стрелка3.1
- net at ДТ5.: now also Стрелка3.
- net at К2.: no longer Магистральный_кабель4. (привязка)
- net at Стрелка12.: now also ДТ20.
- net at ДТ20.: now also ДТ19.; no longer Стрелка12.
- net at Магистральный_6. (привязка): now also Магистральный_7. (привязка); no longer Магистральный_4. (привязка)
- net at ДТ7.: no longer Стрелка4.
- new net: Магистральный_кабель5. (привязка), Магистральный_кабель6. (привязка)
- new net: Магистральный_?. (привязка), Магистральный_?. (привязка)
- new net: ДТ24., Путь7.
- new net: К5., Магистральный_кабель10. (привязка)
- new net: ДТ23., Стрелка7. (x2)
- new net: ДТ22., Стрелка7. (x2)
- new net: ДТ24., Стрелка7.
- new net: Магистральный_5. (привязка), Магистральный_кабель17. (привязка)
- new net: Стрелка10., Стрелка5. (x2)
- new net: ДТ18., Стрелка5.
- new net: Стрелка2., Стрелка7. (x2)
- new net: ДТ9., Стрелка7.
- new net: ДТ14., ДТ15. (x2)
- new net: ДТ10., Стрелка2.
- new net: ДТ17., Стрелка10.
- new net: Магистральный_7. (привязка), Магистральный_8. (привязка)
- new net: ДТ11., Стрелка8. (x2)
- new net: ДТ12., Стрелка8.
- new net: ДТ13., Стрелка6. (x2)
- new net: ДТ13., Путь2.
- new net: ДТ4., Стрелка1. (x2)
- new net: ДТ3., Стрелка1.
- new net: ДТ11., Стрелка5.
- new net: Стрелка3., Стрелка5.
- new net: ДТ18., Путь4.
- new net: ДТ15., Стрелка9.
- new net: ДТ16., Стрелка9.
- new net: ДТ17., Стрелка4.
- new net: Стрелка11., Стрелка4.
- new net: К9., Магистральный_кабель19. (привязка)
- new net: ДТ23., Путь6.
- new net: К1., Магистральный_кабель2. (привязка)
- new net: ДТ16., Стрелка11.
- new net: К8., Магистральный_3. (привязка)
- new net: ДТ22., Стрелка6.
- new net: ДТ6., Стрелка4. (x2)
- new net: ДТ4., Стрелка3.
- new net: Магистральный_кабель12. (привязка), Магистральный_кабель13. (привязка)
- new net: К9., Магистральный_2. (привязка)
- new net: ДТ5., Стрелка3.
- new net: ДТ21., Стрелка12. (x2)
- new net: ДТ20., Стрелка12.
- new net: ДТ21., Стрелка6.
- new net: ДТ7., Стрелка4.
- new net: ДТ19., ДТ20.
- new net: ДТ10., Стрелка3.
- new net: ДТ12., Стрелка6.
- now unconnected: ДТ1., ДТ3., ДТ7., ДТ7., ДТ9., К9., Путь2., Путь4., Стрелка11., Стрелка11., Стрелка11., Стрелка3., Стрелка3., Стрелка3., Стрелка3., Стрелка3., Стрелка3., ЯР6П1.
Changed lines of the file:
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@@
 	)
 	(embedded_fonts no)
+	(embedded_files
+		(file
+			(name "КП_МКТ.kicad_wks")
+			(type worksheet)
+			(data |KLUv/WBoIM0nAIZtizBAdTpUIcw/MEEl5UD9vvRxVUaTt7Tdim1NsQHCcIaa6NdKKWWSMk3Fl5PY
+				Ge6GSwSJAG0AhwD9ludlJRB0aTRPj2bLyztxzWxeGSaSIC2v99IsRE8fKpoOBP3ZWQpdVDSzEkYp
+				JmHCaMXIyuJe1igLlSIoxXRQq3gr6ISlMS+LBPrKd3JYJ4qaVKDT8Zgw6DxxFT8Rnwyj1sSMIJk+
+				m2E0lM1rjgQ6HlDs7ubse2HWKZsZAh3P6UIjYiIksi4EArDjY/dOthYZ9rOLcbmxtwuj2PXd7fUy
+				N34NRl+WkSG7993L/v7O9cC35W+wBxblzR3F7LLZmbmS//9a+3bs9qNrGyFs8cHn75zr5rxBurCe
+				o5CJmjBedubqf2WUleyWHt81fN+NTHRZbWlomjwrU7fCSXlnmwpTa6oMTt2PFExNkbGljjzYICwV
+				BTb3qhB33futwQ5JgaRk6om3fMGBMtLUlpf61dtrklChUsdn8t6uhqRYagnLnTREsaxyuK1yqTZV
+				prLUmEpSPZv0mqLdoLDoCcOi8rZfve89YSaKmg8E/alqqkhqpt7Ul8qSs/BZippUgsIekAfU8YDe
+				vXNf5ph5fJWvdLF6sSU/99gebP92zq5V7b4OX0t3/Ptw/8FvZ/4Kuv3XDwsHCq6jc+se7vtDLBQ0
+				KDAYcNtZIbvbto6HXhhF9G3RHSQ8IDw46dyEUdmxmwcAQEfAyobOsgJfjIqL7/KRSnGwdYPu2l9q
+				gUuoIUmqZkaSgqSSNgNRESGMWKeuDnJwGINQCMJwDENSKAcZZwhhxAgKMkRkZEi0A8hZg3bWYlb2
+				h4YoYKGFmekygghKPx7M15IDD7IYd0WZcR9+6xUxAWj38yoXAmC92oZMMfSB1X7rMp20tBrmEBIe
+				hJakM3LW1t3YaQqxwLlbgpwXnM4OLhkcj+VMBQPN2YfN4GDyKLQvgbLaFMHD7rsVHUKT0f1CBDFP
+				XSbe2VB8O79sP6vXCAAfQsfS9FmMsucETSZlwUkkPcQNppQ7TSRxPLsSCN3qj6BnCn09e0/ycEVX
+				3g7wv0CN+KgnLnaDw8y9wQhha3BdLY2v2im89zFrK+VXxtKex5HrauhBrs/tfKi6CNhwPzqzFi3z
+				9U9Sfevn18nGhVF6A8vogOXyMhBb5VwDaXeWAKXYKMLnvwFgs6HSKajyFcrFafcXwJdaG1hIPkiI
+				V/sxYh7nQd22wwlq3PVReFUKBL6a2LzD6KYLdqFI5QQgIR7waZWh9JSLVhZEctJdcwR7A21bB4Hz
+				YfEHf73jPKpiFEOcdpvT9+AQ+tz+oKOKfBl8eLO27y8VJRblwQT7135UnaHRYO7Y2aumWmyLln0M
+				EkEDoZrYI3+aWzQDyapNeKGVQYAECUSWgbsKzB1f7vHwQoUlWbzELbjETzjux+sduNZypQe0pMC3
+				27OXquavENrbkZwas/aMKEFFfiCsrJGJaiGom2yCQx+xet8JSY59VXzJJZZqANQJJJLQ10mk4+Zo
+				KFq0lCRIAwvRiSaVy+NmH7CuRcJ8H5tzH5nMFpPSW2OVDZxoTeXn3khhg88GFYDHgwvheKwMphGy
+				pUNF15jqOumO8hmv3H0Kp2Kv648A3/nhJFgFVZKCoNKJ80sYuikSwx16AEgHvf+okhOf8aBlIYg9
+				C5pjkJDYaAirz+RKmgVKCmny3vo9qWmdnfGSrgI=|
+			)
+			(checksum "3FBF103777E8EE01081CA18737155A0D")
+		)
+	)
 )
