File: example/БМРЦ/Двухниточный/канализация.kicad_sch (KiCad schematic)
At the start: 0 parts

Commit message: Наведен порядок в двухнитке
Other:
- note added: "М27П"
- note added: "М3П"
- note removed: "М29П"
- note removed: "М5П"
Changed lines of the file:
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@@
 	(title_block
 		(company "АТ-451")
+		(comment 1 "КП27.02.03.10.000 ГЧ")
 		(comment 2 "Михайлов А.К.")
 		(comment 3 "Ворона В.К.")
@@
 		)
 	)
-	(text "М29П"
+	(text "М27П"
 		(exclude_from_sim no)
 		(at 360 75 0)
@@
 		)
 	)
-	(text "М5П"
+	(text "М3П"
 		(exclude_from_sim no)
 		(at 100 135 0)
