File: example/БМРЦ/Однониточный/Однониточный.kicad_sch (KiCad schematic)
At the start: 59 parts

Commit message: Новое дерево для КП 01.01
Connections:
- new net: Изостык11. (привязка), Стрелка5.1, Стрелка6.1
- new net: Изостык14. (привязка), Стрелка6.1, Стрелка7.1
- new net: Изостык9. (привязка), Стрелка3.1, Стрелка5.1
- new net: Изостык12. (привязка), Стрелка4.1, Стрелка6.1
- new net: Изостык7. (привязка), Стрелка3.1, Стрелка4.1
- new net: Изостык8. (привязка), Стрелка1.1, Стрелка2.1
- new net: Изостык10. (привязка), Стрелка2.1, Стрелка8.1
Other:
- removed sheet Двухниточный_план_станции
- removed sheet Канализация_тягового_тока
Changed lines of the file:
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@@
 	)
 	(symbol
-		(lib_name "SCB:Изостык")
 		(lib_id "SCB:Изостык")
 		(at 330 160 0)
@@
 	)
 	(symbol
-		(lib_name "SCB:Изостык")
 		(lib_id "SCB:Изостык")
 		(at 208 190 0)
@@
 	)
 	(symbol
-		(lib_name "SCB:Стрелка_спаренная")
 		(lib_id "SCB:Стрелка_спаренная")
 		(at 284 175 0)
@@
 	)
 	(symbol
-		(lib_name "SCB:Изостык")
 		(lib_id "SCB:Изостык")
 		(at 157 175 0)
@@
 	)
 	(symbol
-		(lib_name "SCB:Изостык")
 		(lib_id "SCB:Изостык")
 		(at 334 130 0)
@@
 	)
 	(symbol
-		(lib_name "SCB:Изостык")
 		(lib_id "SCB:Изостык")
 		(at 226 175 0)
@@
 	)
 	(symbol
-		(lib_name "SCB:Изостык")
 		(lib_id "SCB:Изостык")
 		(at 350 220 0)
@@
 	)
 	(symbol
-		(lib_name "SCB:Изостык")
 		(lib_id "SCB:Изостык")
 		(at 86 160 0)
@@
 	)
 	(symbol
-		(lib_name "SCB:Изостык")
 		(lib_id "SCB:Изостык")
 		(at 279 175 0)
@@
 	)
 	(symbol
-		(lib_name "SCB:Стрелка_спаренная_15")
 		(lib_id "SCB:Стрелка_спаренная_15")
 		(at 148 175 0)
@@
 	)
 	(symbol
-		(lib_name "SCB:Изостык")
 		(lib_id "SCB:Изостык")
 		(at 313 175 0)
@@
 	)
 	(symbol
-		(lib_name "SCB:Стрелка_спаренная_15")
 		(lib_id "SCB:Стрелка_спаренная_15")
 		(at 127 205 0)
@@
 	)
 	(symbol
-		(lib_name "SCB:Изостык")
 		(lib_id "SCB:Изостык")
 		(at 74 190 0)
@@
 	)
 	(symbol
-		(lib_name "SCB:Изостык")
 		(lib_id "SCB:Изостык")
 		(at 249 160 0)
@@
 	)
 	(symbol
-		(lib_name "SCB:Изостык")
 		(lib_id "SCB:Изостык")
 		(at 132 190 0)
@@
 	)
 	(symbol
-		(lib_name "SCB:Изостык")
 		(lib_id "SCB:Изостык")
 		(at 167 205 0)
@@
 	)
 	(symbol
-		(lib_name "SCB:Изостык")
 		(lib_id "SCB:Изостык")
 		(at 350 205 0)
@@
 	)
 	(symbol
-		(lib_name "SCB:Изостык")
 		(lib_id "SCB:Изостык")
 		(at 40 190 0)
@@
 	)
 	(symbol
-		(lib_name "SCB:Изостык")
 		(lib_id "SCB:Изостык")
 		(at 40 205 0)
@@
 	)
 	(symbol
-		(lib_name "SCB:Стрелка_спаренная_15")
 		(lib_id "SCB:Стрелка_спаренная_15")
 		(at 294 205 0)
@@
 	)
 	(symbol
-		(lib_name "SCB:Изостык")
 		(lib_id "SCB:Изостык")
 		(at 375 160 0)
@@
 	)
 	(symbol
-		(lib_name "SCB:Изостык")
 		(lib_id "SCB:Изостык")
 		(at 82 175 0)
@@
 	)
 	(symbol
-		(lib_name "SCB:Стрелка_спаренная_15")
 		(lib_id "SCB:Стрелка_спаренная_15")
 		(at 190 175 0)
@@
 	)
 	(symbol
-		(lib_name "SCB:Стрелка_спаренная_15")
 		(lib_id "SCB:Стрелка_спаренная_15")
 		(at 79 190 0)
@@
 	)
 	(symbol
-		(lib_name "SCB:Изостык")
 		(lib_id "SCB:Изостык")
 		(at 123 205 0)
@@
 	)
 	(symbol
-		(lib_name "SCB:Изостык")
 		(lib_id "SCB:Изостык")
 		(at 307 205 0)
@@
 	)
 	(symbol
-		(lib_name "SCB:Изостык")
 		(lib_id "SCB:Изостык")
 		(at 128 160 0)
@@
 	)
 	(symbol
-		(lib_name "SCB:Изостык")
 		(lib_id "SCB:Изостык")
 		(at 286 190 0)
@@
 	)
 	(symbol
-		(lib_name "SCB:Изостык")
 		(lib_id "SCB:Изостык")
 		(at 290 160 0)
@@
 				)
 			)
-		)
-	)
-	(sheet
-		(at 430 270)
-		(size 13 4)
-		(fields_autoplaced yes)
-		(stroke
-			(width 0.1524)
-			(type solid)
-		)
-		(fill
-			(color 0 0 0 0.0000)
-		)
-		(property "Sheetname" "Двухниточный_план_станции"
-			(at 430 269.2884 0)
-			(effects
-				(font
-					(size 1.27 1.27)
-				)
-				(justify left bottom)
-			)
-		)
-		(property "Sheetfile" "двухниточный.kicad_sch"
-			(at 430 274.5846 0)
-			(effects
-				(font
-					(size 1.27 1.27)
-				)
-				(justify left top)
-			)
-		)
-		(instances
-			(project "БМРЦ"
-				(path "/59e30762-dbae-41fa-856e-a9035e08cb51"
-					(page "2")
-				)
-			)
-		)
-	)
-	(sheet
-		(at 430 280)
-		(size 13 4)
-		(fields_autoplaced yes)
-		(stroke
-			(width 0.1524)
-			(type solid)
-		)
-		(fill
-			(color 0 0 0 0.0000)
-		)
-		(property "Sheetname" "Канализация_тягового_тока"
-			(at 430 279.2884 0)
-			(effects
-				(font
-					(size 1.27 1.27)
-				)
-				(justify left bottom)
-			)
-		)
-		(property "Sheetfile" "канализация.kicad_sch"
-			(at 430 284.5846 0)
-			(effects
-				(font
-					(size 1.27 1.27)
-				)
-				(justify left top)
-			)
-		)
-		(instances
-			(project "БМРЦ"
-				(path "/59e30762-dbae-41fa-856e-a9035e08cb51"
-					(page "3")
-				)
-			)

Commit message: Наведен порядок в двухнитке
Parts:
- removed unit 2 of Маневровый2
- added Маневровый613: ~, symbol SCB:Маневровый_к
- Маневровый1: Литера М5 -> М3
- Маневровый13: Литера М27 -> М25
- Маневровый14: Литера М25 -> М29
- Маневровый2: Литера М29 -> М27
- Маневровый3: Литера М3 -> М5
- Маневровый5: Литера М11 -> М9
- Маневровый6: Литера М9 -> М11
Connections:
- net at Изостык17. (привязка), Стрелка8.1: now also C2.1
- new net: Изостык11. (привязка), Стрелка5.1, Стрелка6.1
- new net: Изостык14. (привязка), Стрелка6.1, Стрелка7.1
- new net: Изостык9. (привязка), Стрелка3.1, Стрелка5.1
- new net: Изостык12. (привязка), Стрелка4.1, Стрелка6.1
- new net: Изостык7. (привязка), Стрелка3.1, Стрелка4.1
- new net: Изостык8. (привязка), Стрелка1.1, Стрелка2.1
- new net: Изостык10. (привязка), Стрелка2.1, Стрелка8.1
Other:
- note added: "Оборудование горловины станции устройсвами блочной маршрутно-релейной централизации (БМРЦ)"
- note added: "Схематический план станции с осигнализованием"
- note added: "Ч2,М27"
- note removed: "М27"
- note removed: "Ч2"

Commit message: Обновление до 9 KiCad
Parts:
- Входной1: now in the parts list
- Входной2: renamed from Входной1; now in the parts list
Connections:
- new net: Изостык11. (привязка), Стрелка5.1, Стрелка6.1
- new net: Изостык14. (привязка), Стрелка6.1, Стрелка7.1
- new net: Изостык9. (привязка), Стрелка3.1, Стрелка5.1
- new net: Изостык12. (привязка), Стрелка4.1, Стрелка6.1
- new net: Изостык7. (привязка), Стрелка3.1, Стрелка4.1
- new net: Изостык8. (привязка), Стрелка1.1, Стрелка2.1
- new net: Изостык10. (привязка), Стрелка2.1, Стрелка8.1

Commit message: Embed рамки
Connections:
- new net: Изостык11. (привязка), Стрелка5.1, Стрелка6.1
- new net: Изостык14. (привязка), Стрелка6.1, Стрелка7.1
- new net: Изостык9. (привязка), Стрелка3.1, Стрелка5.1
- new net: Изостык12. (привязка), Стрелка4.1, Стрелка6.1
- new net: Изостык7. (привязка), Стрелка3.1, Стрелка4.1
- new net: Изостык8. (привязка), Стрелка1.1, Стрелка2.1
- new net: Изостык10. (привязка), Стрелка2.1, Стрелка8.1
Changed lines of the file:
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@@
 	)
 	(embedded_fonts no)
+	(embedded_files
+		(file
+			(name "КП_МКТ.kicad_wks")
+			(type worksheet)
+			(data |KLUv/WBoIM0nAIZtizBAdTpUIcw/MEEl5UD9vvRxVUaTt7Tdim1NsQHCcIaa6NdKKWWSMk3Fl5PY
+				Ge6GSwSJAG0AhwD9ludlJRB0aTRPj2bLyztxzWxeGSaSIC2v99IsRE8fKpoOBP3ZWQpdVDSzEkYp
+				JmHCaMXIyuJe1igLlSIoxXRQq3gr6ISlMS+LBPrKd3JYJ4qaVKDT8Zgw6DxxFT8Rnwyj1sSMIJk+
+				m2E0lM1rjgQ6HlDs7ubse2HWKZsZAh3P6UIjYiIksi4EArDjY/dOthYZ9rOLcbmxtwuj2PXd7fUy
+				N34NRl+WkSG7993L/v7O9cC35W+wBxblzR3F7LLZmbmS//9a+3bs9qNrGyFs8cHn75zr5rxBurCe
+				o5CJmjBedubqf2WUleyWHt81fN+NTHRZbWlomjwrU7fCSXlnmwpTa6oMTt2PFExNkbGljjzYICwV
+				BTb3qhB33futwQ5JgaRk6om3fMGBMtLUlpf61dtrklChUsdn8t6uhqRYagnLnTREsaxyuK1yqTZV
+				prLUmEpSPZv0mqLdoLDoCcOi8rZfve89YSaKmg8E/alqqkhqpt7Ul8qSs/BZippUgsIekAfU8YDe
+				vXNf5ph5fJWvdLF6sSU/99gebP92zq5V7b4OX0t3/Ptw/8FvZ/4Kuv3XDwsHCq6jc+se7vtDLBQ0
+				KDAYcNtZIbvbto6HXhhF9G3RHSQ8IDw46dyEUdmxmwcAQEfAyobOsgJfjIqL7/KRSnGwdYPu2l9q
+				gUuoIUmqZkaSgqSSNgNRESGMWKeuDnJwGINQCMJwDENSKAcZZwhhxAgKMkRkZEi0A8hZg3bWYlb2
+				h4YoYKGFmekygghKPx7M15IDD7IYd0WZcR9+6xUxAWj38yoXAmC92oZMMfSB1X7rMp20tBrmEBIe
+				hJakM3LW1t3YaQqxwLlbgpwXnM4OLhkcj+VMBQPN2YfN4GDyKLQvgbLaFMHD7rsVHUKT0f1CBDFP
+				XSbe2VB8O79sP6vXCAAfQsfS9FmMsucETSZlwUkkPcQNppQ7TSRxPLsSCN3qj6BnCn09e0/ycEVX
+				3g7wv0CN+KgnLnaDw8y9wQhha3BdLY2v2im89zFrK+VXxtKex5HrauhBrs/tfKi6CNhwPzqzFi3z
+				9U9Sfevn18nGhVF6A8vogOXyMhBb5VwDaXeWAKXYKMLnvwFgs6HSKajyFcrFafcXwJdaG1hIPkiI
+				V/sxYh7nQd22wwlq3PVReFUKBL6a2LzD6KYLdqFI5QQgIR7waZWh9JSLVhZEctJdcwR7A21bB4Hz
+				YfEHf73jPKpiFEOcdpvT9+AQ+tz+oKOKfBl8eLO27y8VJRblwQT7135UnaHRYO7Y2aumWmyLln0M
+				EkEDoZrYI3+aWzQDyapNeKGVQYAECUSWgbsKzB1f7vHwQoUlWbzELbjETzjux+sduNZypQe0pMC3
+				27OXquavENrbkZwas/aMKEFFfiCsrJGJaiGom2yCQx+xet8JSY59VXzJJZZqANQJJJLQ10mk4+Zo
+				KFq0lCRIAwvRiSaVy+NmH7CuRcJ8H5tzH5nMFpPSW2OVDZxoTeXn3khhg88GFYDHgwvheKwMphGy
+				pUNF15jqOumO8hmv3H0Kp2Kv648A3/nhJFgFVZKCoNKJ80sYuikSwx16AEgHvf+okhOf8aBlIYg9
+				C5pjkJDYaAirz+RKmgVKCmny3vo9qWmdnfGSrgI=|
+			)
+			(checksum "3FBF103777E8EE01081CA18737155A0D")
+		)
+	)
 )
